File: pcbs/DALU/AddSub.kicad_sch (KiCad schematic)
At the start: 5 parts, among them U201 74HC86, U202 74HC86, U203 74LS283, U204 74LS283, U205 74HC86

Commit message: Trying to figure out the hierarchical buses
Connections:
- net RESULT0 renamed AS0
- net RESULT1 renamed AS1
- net RESULT2 renamed AS2
- net RESULT3 renamed AS3
- net RESULT4 renamed AS4
- net RESULT5 renamed AS5
- net RESULT6 renamed AS6
- net RESULT7 renamed AS7

Commit message: Trying to get everything together
Connections:
- net GND: now also U201.7 (GND), U202.7 (GND), U203.8 (GND), U204.8 (GND), U205.7 (GND)
- net +5V: now reaches U203.16 (VCC)
- net +5V: now also U201.14 (VCC), U202.14 (VCC), U204.16 (VCC), U205.14 (VCC)
Changed lines of the file:
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@@
+    (stroke (width 0) (type default) (color 0 0 0 0))
+  )
+  (wire (pts (xy 269.24 154.94) (xy 269.24 157.48))
     (stroke (width 0) (type default) (color 0 0 0 0))
   )
@@
     (stroke (width 0) (type default) (color 0 0 0 0))
   )
+  (wire (pts (xy 29.21 189.23) (xy 29.21 193.04))
+    (stroke (width 0) (type default) (color 0 0 0 0))
+  )
   (wire (pts (xy 77.47 104.14) (xy 60.96 104.14))
     (stroke (width 0) (type default) (color 0 0 0 0))
@@
     (stroke (width 0) (type default) (color 0 0 0 0))
   )
+  (wire (pts (xy 163.83 87.63) (xy 168.91 87.63))
+    (stroke (width 0) (type default) (color 0 0 0 0))
+  )
+  (wire (pts (xy 57.15 189.23) (xy 57.15 193.04))
+    (stroke (width 0) (type default) (color 0 0 0 0))
+  )
   (wire (pts (xy 146.05 107.95) (xy 156.21 107.95))
     (stroke (width 0) (type default) (color 0 0 0 0))
   )
+  (wire (pts (xy 57.15 160.02) (xy 57.15 163.83))
+    (stroke (width 0) (type default) (color 0 0 0 0))
+  )
+  (wire (pts (xy 163.83 78.74) (xy 168.91 78.74))
+    (stroke (width 0) (type default) (color 0 0 0 0))
+  )
   (wire (pts (xy 137.16 63.5) (xy 156.21 63.5))
     (stroke (width 0) (type default) (color 0 0 0 0))
@@
     (stroke (width 0) (type default) (color 0 0 0 0))
   )
+  (wire (pts (xy 67.31 36.83) (xy 77.47 36.83))
+    (stroke (width 0) (type default) (color 0 0 0 0))
+  )
   (bus (pts (xy 200.66 45.72) (xy 200.66 43.18))
     (stroke (width 0) (type default) (color 0 0 0 0))
@@
     (stroke (width 0) (type default) (color 0 0 0 0))
   )
+  (wire (pts (xy 168.91 35.56) (xy 168.91 38.1))
+    (stroke (width 0) (type default) (color 0 0 0 0))
+  )
   (wire (pts (xy 181.61 100.33) (xy 198.12 100.33))
     (stroke (width 0) (type default) (color 0 0 0 0))
@@
     (stroke (width 0) (type default) (color 0 0 0 0))
   )
+  (wire (pts (xy 29.21 160.02) (xy 29.21 163.83))
+    (stroke (width 0) (type default) (color 0 0 0 0))
+  )
   (wire (pts (xy 146.05 55.88) (xy 156.21 55.88))
     (stroke (width 0) (type default) (color 0 0 0 0))
@@
     (stroke (width 0) (type default) (color 0 0 0 0))
   )
+  (wire (pts (xy 168.91 128.27) (xy 168.91 130.81))
+    (stroke (width 0) (type default) (color 0 0 0 0))
+  )
   (bus (pts (xy 64.77 49.53) (xy 64.77 64.77))
     (stroke (width 0) (type default) (color 0 0 0 0))
@@
     (stroke (width 0) (type default) (color 0 0 0 0))
   )
-  (wire (pts (xy 67.31 36.83) (xy 77.47 36.83))
-    (stroke (width 0) (type default) (color 0 0 0 0))
-  )
   (wire (pts (xy 92.71 85.09) (xy 97.79 85.09))
     (stroke (width 0) (type default) (color 0 0 0 0))
@@
   )
   (wire (pts (xy 60.96 57.15) (xy 60.96 41.91))
+    (stroke (width 0) (type default) (color 0 0 0 0))
+  )
+  (wire (pts (xy 269.24 127) (xy 269.24 129.54))
     (stroke (width 0) (type default) (color 0 0 0 0))
   )
@@
     (pin "8")
     (pin "9")
+  )
+  (symbol (lib_id "power:+5V") (at 168.91 35.56 0) (unit 1)
+    (in_bom yes) (on_board yes) (fields_autoplaced)
+    (property "Reference" "#PWR0207" (id 0) (at 168.91 39.37 0)
+      (effects (font (size 1.27 1.27)) hide)
+    )
+    (property "Value" "+5V" (id 1) (at 168.91 30.48 0))
+    (property "Footprint" "" (id 2) (at 168.91 35.56 0)
+      (effects (font (size 1.27 1.27)) hide)
+    )
+    (property "Datasheet" "" (id 3) (at 168.91 35.56 0)
+      (effects (font (size 1.27 1.27)) hide)
+    )
+    (pin "1")
+  )
+  (symbol (lib_id "power:GND") (at 163.83 78.74 270) (unit 1)
+    (in_bom yes) (on_board yes) (fields_autoplaced)
+    (property "Reference" "#PWR0205" (id 0) (at 157.48 78.74 0)
+      (effects (font (size 1.27 1.27)) hide)
+    )
+    (property "Value" "GND" (id 1) (at 160.02 78.7399 90)
+      (effects (font (size 1.27 1.27)) (justify right))
+    )
+    (property "Footprint" "" (id 2) (at 163.83 78.74 0)
+      (effects (font (size 1.27 1.27)) hide)
+    )
+    (property "Datasheet" "" (id 3) (at 163.83 78.74 0)
+      (effects (font (size 1.27 1.27)) hide)
+    )
+    (pin "1")
+  )
+  (symbol (lib_id "power:GND") (at 269.24 157.48 0) (unit 1)
+    (in_bom yes) (on_board yes) (fields_autoplaced)
+    (property "Reference" "#PWR0211" (id 0) (at 269.24 163.83 0)
+      (effects (font (size 1.27 1.27)) hide)
+    )
+    (property "Value" "GND" (id 1) (at 269.24 162.56 0))
+    (property "Footprint" "" (id 2) (at 269.24 157.48 0)
+      (effects (font (size 1.27 1.27)) hide)
+    )
+    (property "Datasheet" "" (id 3) (at 269.24 157.48 0)
+      (effects (font (size 1.27 1.27)) hide)
+    )
+    (pin "1")
   )
   (symbol (lib_id "74xx:74HC86") (at 269.24 142.24 0) (unit 5)
@@
     (pin "7")
   )
+  (symbol (lib_id "power:+5V") (at 163.83 87.63 90) (unit 1)
+    (in_bom yes) (on_board yes) (fields_autoplaced)
+    (property "Reference" "#PWR0206" (id 0) (at 167.64 87.63 0)
+      (effects (font (size 1.27 1.27)) hide)
+    )
+    (property "Value" "+5V" (id 1) (at 160.02 87.6299 90)
+      (effects (font (size 1.27 1.27)) (justify left))
+    )
+    (property "Footprint" "" (id 2) (at 163.83 87.63 0)
+      (effects (font (size 1.27 1.27)) hide)
+    )
+    (property "Datasheet" "" (id 3) (at 163.83 87.63 0)
+      (effects (font (size 1.27 1.27)) hide)
+    )
+    (pin "1")
+  )
   (symbol (lib_id "74xx:74HC86") (at 85.09 69.85 0) (unit 3)
     (in_bom yes) (on_board yes) (fields_autoplaced)
@@
     (pin "7")
   )
+  (symbol (lib_id "power:+5V") (at 29.21 160.02 0) (unit 1)
+    (in_bom yes) (on_board yes) (fields_autoplaced)
+    (property "Reference" "#PWR0201" (id 0) (at 29.21 163.83 0)
+      (effects (font (size 1.27 1.27)) hide)
+    )
+    (property "Value" "+5V" (id 1) (at 29.21 154.94 0))
+    (property "Footprint" "" (id 2) (at 29.21 160.02 0)
+      (effects (font (size 1.27 1.27)) hide)
+    )
+    (property "Datasheet" "" (id 3) (at 29.21 160.02 0)
+      (effects (font (size 1.27 1.27)) hide)
+    )
+    (pin "1")
+  )
   (symbol (lib_id "74xx:74HC86") (at 273.05 82.55 0) (unit 2)
     (in_bom yes) (on_board yes) (fields_autoplaced)
@@
   (symbol (lib_id "power:GND") (at 261.62 118.11 0) (unit 1)
     (in_bom yes) (on_board yes) (fields_autoplaced)
-    (property "Reference" "#PWR0201" (id 0) (at 261.62 124.46 0)
+    (property "Reference" "#PWR0209" (id 0) (at 261.62 124.46 0)
       (effects (font (size 1.27 1.27)) hide)
     )
@@
     (pin "7")
   )
+  (symbol (lib_id "power:+5V") (at 57.15 160.02 0) (unit 1)
+    (in_bom yes) (on_board yes) (fields_autoplaced)
+    (property "Reference" "#PWR0203" (id 0) (at 57.15 163.83 0)
+      (effects (font (size 1.27 1.27)) hide)
+    )
+    (property "Value" "+5V" (id 1) (at 57.15 154.94 0))
+    (property "Footprint" "" (id 2) (at 57.15 160.02 0)
+      (effects (font (size 1.27 1.27)) hide)
+    )
+    (property "Datasheet" "" (id 3) (at 57.15 160.02 0)
+      (effects (font (size 1.27 1.27)) hide)
+    )
+    (pin "1")
+  )
   (symbol (lib_id "74xx:74HC86") (at 85.09 147.32 0) (unit 4)
     (in_bom yes) (on_board yes) (fields_autoplaced)
@@
     (pin "7")
   )
+  (symbol (lib_id "power:GND") (at 29.21 193.04 0) (unit 1)
+    (in_bom yes) (on_board yes) (fields_autoplaced)
+    (property "Reference" "#PWR0202" (id 0) (at 29.21 199.39 0)
+      (effects (font (size 1.27 1.27)) hide)
+    )
+    (property "Value" "GND" (id 1) (at 29.21 198.12 0))
+    (property "Footprint" "" (id 2) (at 29.21 193.04 0)
+      (effects (font (size 1.27 1.27)) hide)
+    )
+    (property "Datasheet" "" (id 3) (at 29.21 193.04 0)
+      (effects (font (size 1.27 1.27)) hide)
+    )
+    (pin "1")
+  )
+  (symbol (lib_id "power:GND") (at 57.15 193.04 0) (unit 1)
+    (in_bom yes) (on_board yes) (fields_autoplaced)
+    (property "Reference" "#PWR0204" (id 0) (at 57.15 199.39 0)
+      (effects (font (size 1.27 1.27)) hide)
+    )
+    (property "Value" "GND" (id 1) (at 57.15 198.12 0))
+    (property "Footprint" "" (id 2) (at 57.15 193.04 0)
+      (effects (font (size 1.27 1.27)) hide)
+    )
+    (property "Datasheet" "" (id 3) (at 57.15 193.04 0)
+      (effects (font (size 1.27 1.27)) hide)
+    )
+    (pin "1")
+  )
+  (symbol (lib_id "power:GND") (at 168.91 130.81 0) (unit 1)
+    (in_bom yes) (on_board yes) (fields_autoplaced)
+    (property "Reference" "#PWR0208" (id 0) (at 168.91 137.16 0)
+      (effects (font (size 1.27 1.27)) hide)
+    )
+    (property "Value" "GND" (id 1) (at 168.91 135.89 0))
+    (property "Footprint" "" (id 2) (at 168.91 130.81 0)
+      (effects (font (size 1.27 1.27)) hide)
+    )
+    (property "Datasheet" "" (id 3) (at 168.91 130.81 0)
+      (effects (font (size 1.27 1.27)) hide)
+    )
+    (pin "1")
+  )
   (symbol (lib_id "74xx:74HC86") (at 57.15 176.53 0) (unit 5)
     (in_bom yes) (on_board yes) (fields_autoplaced)
@@
     (pin "7")
   )
+  (symbol (lib_id "power:+5V") (at 269.24 127 0) (unit 1)
+    (in_bom yes) (on_board yes) (fields_autoplaced)
+    (property "Reference" "#PWR0210" (id 0) (at 269.24 130.81 0)
+      (effects (font (size 1.27 1.27)) hide)
+    )
+    (property "Value" "+5V" (id 1) (at 269.24 121.92 0))
+    (property "Footprint" "" (id 2) (at 269.24 127 0)
+      (effects (font (size 1.27 1.27)) hide)
+    )
+    (property "Datasheet" "" (id 3) (at 269.24 127 0)
+      (effects (font (size 1.27 1.27)) hide)
+    )
+    (pin "1")
+  )
   (symbol (lib_id "74xx:74HC86") (at 217.17 110.49 0) (unit 1)

Commit message: Rethinking some design
Parts:
- added U204: 74HC125, Package_DIP:DIP-14_W7.62mm_Socket, symbol 74xx:74LS125
- added U207: 74HCT541, Package_DIP:DIP-20_W7.62mm_Socket, symbol 74xx:74HCT541
- renumbered U205 to U203, U203 to U205, U204 to U206
Connections:
- net +5V: now also U204.14 (VCC), U207.20 (VCC)
- net FLAG: now also U204.3; no longer U203.3
- net GND: now also U204.10, U204.12, U204.13, U204.4, U204.5, U204.7 (GND), U204.9, U207.10 (GND)
- net AS0: no longer names the net of U205.4 (S1)
- net AS0: now also U207.2 (A0)
- net AS1: no longer names the net of U205.1 (S2)
- net AS1: now also U207.3 (A1)
- net AS2: no longer names the net of U205.13 (S3)
- net AS2: now also U207.4 (A2)
- net AS3: no longer names the net of U205.10 (S4)
- net AS3: now also U207.5 (A3)
- net AS4: no longer names the net of U206.4 (S1)
- net AS4: now also U207.6 (A4)
- net AS5: no longer names the net of U206.1 (S2)
- net AS5: now also U207.7 (A5)
- net AS6: no longer names the net of U206.13 (S3)
- net AS6: now also U207.8 (A6)
- net AS7: no longer names the net of U206.10 (S4)
- net AS7: now also U207.9 (A7)
- new net: U203.3, U204.2
- new net ~{ENABLE_{AS}}: U204.1, U207.1 (G1), U207.19 (G2)
Other:
- moved on the sheet: U203B, U203C, U203D, U203E

Commit message: Thinking about some of the control logic
Parts:
- added R201: 100k, Resistor_THT:R_Axial_DIN0207_L6.3mm_D2.5mm_P7.62mm_Horizontal, symbol Device:R
- U201: footprint (none) -> Package_DIP:DIP-14_W7.62mm_Socket
- U203: renamed from U202; footprint (none) -> Package_DIP:DIP-14_W7.62mm_Socket
- U204: renamed from U203; footprint (none) -> Package_DIP:DIP-14_W7.62mm_Socket
- U205, U206: value 74LS283 -> 74HC283
- renumbered U204 to U202, U202 to U203, U203 to U204
Connections:
- net +5V: now also U204.10, R201.1
- net GND: no longer U202.12, U202.4, U202.5, U202.9, U204.10, U204.13, U204.4, U204.5, U204.9
- net ~{ADD}/SUBTRACT: now also U202.12, U202.9, U204.11; no longer U201.10, U201.13, U201.2, U201.5, U203.10, U203.13, U203.2, U203.5
- net ~{ENABLE_{AS}}: now also U202.6, R201.2
- net at U202.11: now also U203.10, U203.13, U203.2, U203.5
- net at U202.8: now also U201.10, U201.13, U201.2, U201.5
- net at U204.6: now also U204.9
- net at U204.8: now also U202.5
- new net ~{ENABLE_{ADD}}: U204.13, U204.4
- new net ~{ENABLE_{DALU}}: U202.4
- new net ~{ENABLE_{SUBTRACT}}: U204.5
Other:
- note added: "Note that ~{ENABLE_{ADD}} or ~{ENABLE_{SUBTRACT}} can both be high, but it is not possible for both to be low at the same time."
- moved on the sheet: U202B, U202C, U202D, U204B, U204C, U204D

Commit message: Thinking about SMD assembly. Will be rethinking
Parts:
- U201: footprint Package_DIP:DIP-14_W7.62mm_Socket -> Package_SO:TSSOP-14_4.4x5mm_P0.65mm; LCSC (none) -> C113209
- U205: footprint Package_DIP:DIP-16_W7.62mm_Socket -> Package_SO:SOIC-16_3.9x9.9mm_P1.27mm; LCSC (none) -> C1523472
Changed lines of the file:
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@@
       (effects (font (size 1.27 1.27)) (justify left))
     )
-    (property "Footprint" "Package_DIP:DIP-16_W7.62mm_Socket" (id 2) (at 168.91 58.42 0)
+    (property "Footprint" "Package_SO:SOIC-16_3.9x9.9mm_P1.27mm" (id 2) (at 168.91 58.42 0)
       (effects (font (size 1.27 1.27)) hide)
     )
     (property "Datasheet" "http://www.ti.com/lit/gpn/sn74LS283" (id 3) (at 168.91 58.42 0)
+      (effects (font (size 1.27 1.27)) hide)
+    )
+    (property "LCSC" "C1523472" (id 4) (at 168.91 58.42 0)
       (effects (font (size 1.27 1.27)) hide)
     )
@@
     (property "Reference" "U201" (id 0) (at 84.7852 60.96 0))
     (property "Value" "74HC86" (id 1) (at 84.7852 63.5 0))
-    (property "Footprint" "Package_DIP:DIP-14_W7.62mm_Socket" (id 2) (at 85.09 69.85 0)
+    (property "Footprint" "Package_SO:TSSOP-14_4.4x5mm_P0.65mm" (id 2) (at 85.09 69.85 0)
       (effects (font (size 1.27 1.27)) hide)
     )
     (property "Datasheet" "http://www.ti.com/lit/gpn/sn74HC86" (id 3) (at 85.09 69.85 0)
+      (effects (font (size 1.27 1.27)) hide)
+    )
+    (property "LCSC" "C113209" (id 4) (at 85.09 69.85 0)
       (effects (font (size 1.27 1.27)) hide)
     )
@@
       (effects (font (size 1.27 1.27)) (justify left))
     )
-    (property "Footprint" "Package_DIP:DIP-14_W7.62mm_Socket" (id 2) (at 29.21 176.53 0)
+    (property "Footprint" "Package_SO:TSSOP-14_4.4x5mm_P0.65mm" (id 2) (at 29.21 176.53 0)
       (effects (font (size 1.27 1.27)) hide)
     )
     (property "Datasheet" "http://www.ti.com/lit/gpn/sn74HC86" (id 3) (at 29.21 176.53 0)
+      (effects (font (size 1.27 1.27)) hide)
+    )
+    (property "LCSC" "C113209" (id 4) (at 29.21 176.53 0)
       (effects (font (size 1.27 1.27)) hide)
     )
@@
     (property "Reference" "U201" (id 0) (at 84.7852 45.72 0))
     (property "Value" "74HC86" (id 1) (at 84.7852 48.26 0))
-    (property "Footprint" "Package_DIP:DIP-14_W7.62mm_Socket" (id 2) (at 85.09 54.61 0)
+    (property "Footprint" "Package_SO:TSSOP-14_4.4x5mm_P0.65mm" (id 2) (at 85.09 54.61 0)
       (effects (font (size 1.27 1.27)) hide)
     )
     (property "Datasheet" "http://www.ti.com/lit/gpn/sn74HC86" (id 3) (at 85.09 54.61 0)
+      (effects (font (size 1.27 1.27)) hide)
+    )
+    (property "LCSC" "C113209" (id 4) (at 85.09 54.61 0)
       (effects (font (size 1.27 1.27)) hide)
     )
@@
     (property "Reference" "U201" (id 0) (at 84.7852 30.48 0))
     (property "Value" "74HC86" (id 1) (at 84.7852 33.02 0))
-    (property "Footprint" "Package_DIP:DIP-14_W7.62mm_Socket" (id 2) (at 85.09 39.37 0)
+    (property "Footprint" "Package_SO:TSSOP-14_4.4x5mm_P0.65mm" (id 2) (at 85.09 39.37 0)
       (effects (font (size 1.27 1.27)) hide)
     )
     (property "Datasheet" "http://www.ti.com/lit/gpn/sn74HC86" (id 3) (at 85.09 39.37 0)
+      (effects (font (size 1.27 1.27)) hide)
+    )
+    (property "LCSC" "C113209" (id 4) (at 85.09 39.37 0)
       (effects (font (size 1.27 1.27)) hide)
     )
@@
     (property "Reference" "U201" (id 0) (at 84.7852 76.2 0))
     (property "Value" "74HC86" (id 1) (at 84.7852 78.74 0))
-    (property "Footprint" "Package_DIP:DIP-14_W7.62mm_Socket" (id 2) (at 85.09 85.09 0)
+    (property "Footprint" "Package_SO:TSSOP-14_4.4x5mm_P0.65mm" (id 2) (at 85.09 85.09 0)
       (effects (font (size 1.27 1.27)) hide)
     )
@@
       (effects (font (size 1.27 1.27)) hide)
     )
+    (property "LCSC" "C113209" (id 4) (at 85.09 85.09 0)
+      (effects (font (size 1.27 1.27)) hide)
+    )

Commit message: Doing some rethinking
Parts:
- removed U207: 74HCT541, Package_DIP:DIP-20_W7.62mm_Socket, symbol 74xx:74HCT541
- added U307: 74HC245, Package_SO:SOIC-20W_7.5x12.8mm_P1.27mm, symbol 74xx:74HC245
- U301: renamed from U201; footprint Package_SO:TSSOP-14_4.4x5mm_P0.65mm -> Package_DIP:DIP-14_W7.62mm_Socket; LCSC C113209 -> (none)
- U305: renamed from U205; footprint Package_SO:SOIC-16_3.9x9.9mm_P1.27mm -> Package_DIP:DIP-16_W7.62mm_Socket; LCSC C1523472 -> (none)
- renumbered R201 to R301, U202 to U302, U203 to U303, U204 to U304, U206 to U306
Connections:
- net +5V: now also U307.20 (VCC)
- net GND: now also U307.10 (GND)
- net ~{ENABLE_{AS}}: now also U307.1 (A->B), U307.19 (CE)
- net at U305.1 (S2): now also U307.3 (A1)
- net at U305.10 (S4): now also U307.5 (A3)
- net at U305.13 (S3): now also U307.4 (A2)
- net at U305.4 (S1): now also U307.2 (A0)
- net at U306.4 (S1): now also U307.6 (A4)
- net at U306.1 (S2): now also U307.7 (A5)
- net at U306.13 (S3): now also U307.8 (A6)
- net at U306.10 (S4): now also U307.9 (A7)

Commit message: Starting to think about decoding etc.
Parts:
- removed R301: 100k, Resistor_THT:R_Axial_DIN0207_L6.3mm_D2.5mm_P7.62mm_Horizontal, symbol Device:R
- removed U302: 74HC125, Package_DIP:DIP-14_W7.62mm_Socket, symbol 74xx:74LS125
- removed unit 3 of U304
- renumbered U301 to U401, U303 to U402, U304 to U403, U305 to U404, U306 to U405, U307 to U406
Connections:
- net ~{ENABLE_{ADD}}: no longer names the net of U403.13, U403.4
- net ~{ENABLE_{SUBTRACT}}: no longer names the net of U403.5
Other:
- note removed: "Note that ~{ENABLE_{ADD}} or ~{ENABLE_{SUBTRACT}} can both be high, but it is not possible for both to be low at the same time."
