File: pcbs/DALU/AddSub.kicad_sch (KiCad schematic)
At the start: 16 parts, among them U401 74HC86, U402 74HC08, U403 74HC86, U404 74HC86, U405 74HC283, U406 74HC283, U407 74HC245, U408 74HC245

Commit message: Sending for production
Parts:
- U401, U403, U404, U405, U406: now left out of the parts list
- U402: LCSC (none) -> C5593
Changed lines of the file:
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@@
   )
   (symbol (lib_id "74xx:74LS283") (at 168.91 58.42 0) (unit 1)
-    (in_bom yes) (on_board yes) (fields_autoplaced)
+    (in_bom no) (on_board yes) (fields_autoplaced)
     (property "Reference" "U405" (id 0) (at 170.9294 38.1 0)
       (effects (font (size 1.27 1.27)) (justify left))
@@
   )
   (symbol (lib_id "74xx:74HC86") (at 87.63 176.53 0) (unit 5)
-    (in_bom yes) (on_board yes) (fields_autoplaced)
+    (in_bom no) (on_board yes) (fields_autoplaced)
     (property "Reference" "U404" (id 0) (at 93.98 175.2599 0)
       (effects (font (size 1.27 1.27)) (justify left))
@@
   )
   (symbol (lib_id "74xx:74HC86") (at 170.18 222.25 0) (unit 4)
-    (in_bom yes) (on_board yes) (fields_autoplaced)
+    (in_bom no) (on_board yes) (fields_autoplaced)
     (property "Reference" "U404" (id 0) (at 169.8752 213.36 0))
     (property "Value" "74HC86" (id 1) (at 169.8752 215.9 0))
@@
   )
   (symbol (lib_id "74xx:74HC86") (at 142.24 219.075 0) (unit 3)
-    (in_bom yes) (on_board yes) (fields_autoplaced)
+    (in_bom no) (on_board yes) (fields_autoplaced)
     (property "Reference" "U404" (id 0) (at 141.9352 210.185 0))
     (property "Value" "74HC86" (id 1) (at 141.9352 212.725 0))
@@
   )
   (symbol (lib_id "74xx:74HC86") (at 85.09 69.85 0) (unit 3)
-    (in_bom yes) (on_board yes) (fields_autoplaced)
+    (in_bom no) (on_board yes) (fields_autoplaced)
     (property "Reference" "U401" (id 0) (at 84.7852 60.96 0))
     (property "Value" "74HC86" (id 1) (at 84.7852 63.5 0))
@@
   )
   (symbol (lib_id "74xx:74HC86") (at 217.17 105.41 0) (unit 2)
-    (in_bom yes) (on_board yes) (fields_autoplaced)
+    (in_bom no) (on_board yes) (fields_autoplaced)
     (property "Reference" "U404" (id 0) (at 216.8652 96.52 0))
     (property "Value" "74HC86" (id 1) (at 216.8652 99.06 0))
@@
   )
   (symbol (lib_id "74xx:74LS283") (at 168.91 107.95 0) (unit 1)
-    (in_bom yes) (on_board yes) (fields_autoplaced)
+    (in_bom no) (on_board yes) (fields_autoplaced)
     (property "Reference" "U406" (id 0) (at 170.9294 87.63 0)
       (effects (font (size 1.27 1.27)) (justify left))
@@
   )
   (symbol (lib_id "74xx:74HC86") (at 85.09 132.08 0) (unit 3)
-    (in_bom yes) (on_board yes) (fields_autoplaced)
+    (in_bom no) (on_board yes) (fields_autoplaced)
     (property "Reference" "U403" (id 0) (at 84.7852 123.19 0))
     (property "Value" "74HC86" (id 1) (at 84.7852 125.73 0))
@@
   )
   (symbol (lib_id "74xx:74HC86") (at 29.21 176.53 0) (unit 5)
-    (in_bom yes) (on_board yes) (fields_autoplaced)
+    (in_bom no) (on_board yes) (fields_autoplaced)
     (property "Reference" "U401" (id 0) (at 35.56 175.2599 0)
       (effects (font (size 1.27 1.27)) (justify left))
@@
   )
   (symbol (lib_id "74xx:74HC86") (at 85.09 147.32 0) (unit 4)
-    (in_bom yes) (on_board yes) (fields_autoplaced)
+    (in_bom no) (on_board yes) (fields_autoplaced)
     (property "Reference" "U403" (id 0) (at 84.7852 138.43 0))
     (property "Value" "74HC86" (id 1) (at 84.7852 140.97 0))
@@
       (effects (font (size 1.27 1.27)) hide)
     )
+    (property "LCSC" "C5593" (id 4) (at 133.35 147.955 0)
+      (effects (font (size 1.27 1.27)) hide)
+    )
     (pin "1")
     (pin "2")
@@
   )
   (symbol (lib_id "74xx:74HC86") (at 85.09 101.6 0) (unit 1)
-    (in_bom yes) (on_board yes) (fields_autoplaced)
+    (in_bom no) (on_board yes) (fields_autoplaced)
     (property "Reference" "U403" (id 0) (at 84.7852 92.71 0))
     (property "Value" "74HC86" (id 1) (at 84.7852 95.25 0))
@@
   )
   (symbol (lib_id "74xx:74HC86") (at 57.15 176.53 0) (unit 5)
-    (in_bom yes) (on_board yes) (fields_autoplaced)
+    (in_bom no) (on_board yes) (fields_autoplaced)
     (property "Reference" "U403" (id 0) (at 63.5 175.2599 0)
       (effects (font (size 1.27 1.27)) (justify left))
@@
   )
   (symbol (lib_id "74xx:74HC86") (at 85.09 54.61 0) (unit 2)
-    (in_bom yes) (on_board yes) (fields_autoplaced)
+    (in_bom no) (on_board yes) (fields_autoplaced)
     (property "Reference" "U401" (id 0) (at 84.7852 45.72 0))
     (property "Value" "74HC86" (id 1) (at 84.7852 48.26 0))
@@
   )
   (symbol (lib_id "74xx:74HC86") (at 85.09 39.37 0) (unit 1)
-    (in_bom yes) (on_board yes) (fields_autoplaced)
+    (in_bom no) (on_board yes) (fields_autoplaced)
     (property "Reference" "U401" (id 0) (at 84.7852 30.48 0))
     (property "Value" "74HC86" (id 1) (at 84.7852 33.02 0))
@@
   )
   (symbol (lib_id "74xx:74HC86") (at 85.09 85.09 0) (unit 4)
-    (in_bom yes) (on_board yes) (fields_autoplaced)
+    (in_bom no) (on_board yes) (fields_autoplaced)
     (property "Reference" "U401" (id 0) (at 84.7852 76.2 0))
     (property "Value" "74HC86" (id 1) (at 84.7852 78.74 0))
@@
   )
   (symbol (lib_id "74xx:74HC86") (at 99.695 216.535 0) (unit 1)
-    (in_bom yes) (on_board yes) (fields_autoplaced)
+    (in_bom no) (on_board yes) (fields_autoplaced)
     (property "Reference" "U404" (id 0) (at 99.3902 207.645 0))
     (property "Value" "74HC86" (id 1) (at 99.3902 210.185 0))
@@
   )
   (symbol (lib_id "74xx:74HC86") (at 85.09 116.84 0) (unit 2)
-    (in_bom yes) (on_board yes) (fields_autoplaced)
+    (in_bom no) (on_board yes) (fields_autoplaced)
     (property "Reference" "U403" (id 0) (at 84.7852 107.95 0))
     (property "Value" "74HC86" (id 1) (at 84.7852 110.49 0))
