File: pcbs/DALU/DALU.kicad_pcb (KiCad board)
At the start: 2 copper layers, 6 parts, among them J101 Conn_02x20_Odd_Even, U201 74HC86, U202 74HC86, U203 74LS283, U204 74LS283, U205 74HC86

Commit message: Last of the compute stages
Parts:
- added D501: 1N4148, Diode_THT:D_DO-35_SOD27_P7.62mm_Horizontal, F.Cu at (165.1, 87.6)
- added D502: 1N4148, Diode_THT:D_DO-35_SOD27_P7.62mm_Horizontal, F.Cu at (165.1, 91.4)
- added D503: 1N4148, Diode_THT:D_DO-35_SOD27_P7.62mm_Horizontal, F.Cu at (165.1, 95.2)
- added D504: 1N4148, Diode_THT:D_DO-35_SOD27_P7.62mm_Horizontal, F.Cu at (165.1, 99.1)
- added D505: 1N4148, Diode_THT:D_DO-35_SOD27_P7.62mm_Horizontal, F.Cu at (165.1, 102.9)
- added D506: 1N4148, Diode_THT:D_DO-35_SOD27_P7.62mm_Horizontal, F.Cu at (165.1, 106.7)
- added D507: 1N4148, Diode_THT:D_DO-35_SOD27_P7.62mm_Horizontal, F.Cu at (165.1, 110.5)
- added D508: 1N4148, Diode_THT:D_DO-35_SOD27_P7.62mm_Horizontal, F.Cu at (165.1, 114.3)
- added D509: 1N4148, Diode_THT:D_DO-35_SOD27_P7.62mm_Horizontal, F.Cu at (165.1, 118.1)
- added D510: 1N4148, Diode_THT:D_DO-35_SOD27_P7.62mm_Horizontal, F.Cu at (165.1, 121.9)
- added D511: 1N4148, Diode_THT:D_DO-35_SOD27_P7.62mm_Horizontal, F.Cu at (165.1, 125.7)
- added D512: 1N4148, Diode_THT:D_DO-35_SOD27_P7.62mm_Horizontal, F.Cu at (165.1, 129.5)
- added D513: 1N4148, Diode_THT:D_DO-35_SOD27_P7.62mm_Horizontal, F.Cu at (165.1, 133.3)
- added D514: 1N4148, Diode_THT:D_DO-35_SOD27_P7.62mm_Horizontal, F.Cu at (165.1, 137.2)
- added D515: 1N4148, Diode_THT:D_DO-35_SOD27_P7.62mm_Horizontal, F.Cu at (165.1, 141.0)
- added D516: 1N4148, Diode_THT:D_DO-35_SOD27_P7.62mm_Horizontal, F.Cu at (165.1, 144.8)
- added R501: 100k, Resistor_THT:R_Axial_DIN0207_L6.3mm_D2.5mm_P7.62mm_Horizontal, F.Cu at (168.9, 87.6)
- added R502: 100k, Resistor_THT:R_Axial_DIN0207_L6.3mm_D2.5mm_P7.62mm_Horizontal, F.Cu at (168.9, 95.2)
- added R503: 100k, Resistor_THT:R_Axial_DIN0207_L6.3mm_D2.5mm_P7.62mm_Horizontal, F.Cu at (168.9, 102.9)
- added R504: 100k, Resistor_THT:R_Axial_DIN0207_L6.3mm_D2.5mm_P7.62mm_Horizontal, F.Cu at (168.9, 110.5)
- added R505: 100k, Resistor_THT:R_Axial_DIN0207_L6.3mm_D2.5mm_P7.62mm_Horizontal, F.Cu at (168.9, 118.1)
- added R506: 100k, Resistor_THT:R_Axial_DIN0207_L6.3mm_D2.5mm_P7.62mm_Horizontal, F.Cu at (168.9, 125.7)
- added R507: 100k, Resistor_THT:R_Axial_DIN0207_L6.3mm_D2.5mm_P7.62mm_Horizontal, F.Cu at (168.9, 133.3)
- added R508: 100k, Resistor_THT:R_Axial_DIN0207_L6.3mm_D2.5mm_P7.62mm_Horizontal, F.Cu at (168.9, 141.0)
- added U301: 74HC00, Package_DIP:DIP-14_W7.62mm_Socket, F.Cu at (102.9, 101.6)
- added U302: 74HC00, Package_DIP:DIP-14_W7.62mm_Socket, F.Cu at (102.9, 125.7)
- added U401: 74HC86, Package_DIP:DIP-14_W7.62mm_Socket, F.Cu at (168.9, 34.3)
- added U402: 74HC86, Package_DIP:DIP-14_W7.62mm_Socket, F.Cu at (168.9, 57.1)
- moved U201 27.5 mm to (71.1, 36.8)
- moved U202 2.84 mm to (71.1, 57.1)
- moved U203 2.54 mm to (96.5, 34.3)

Commit message: Trying to figure out the hierarchical buses
Parts:
- added U601: 74HCT541, Package_DIP:DIP-20_W7.62mm_Socket, F.Cu at (132.1, 39.4)
- added U602: 74HCT541, Package_DIP:DIP-20_W7.62mm_Socket, F.Cu at (125.7, 99.1)
- added U603: 74LS540, Package_DIP:DIP-20_W7.62mm_Socket, F.Cu at (125.7, 130.8)
- added U604: 74HCT541, Package_DIP:DIP-20_W7.62mm_Socket, F.Cu at (198.1, 99.1)
- added U605: 74HCT541, Package_DIP:DIP-20_W7.62mm_Socket, F.Cu at (198.1, 38.1)
- moved U202 1.28 mm to (71.1, 58.4)
Connections:
- net /OR/RESULT0 renamed /OR/OR0
- net /OR/RESULT1 renamed /OR/OR1
- net /OR/RESULT2 renamed /OR/OR2
- net /OR/RESULT3 renamed /OR/OR3
- net /OR/RESULT4 renamed /OR/OR4
- net /OR/RESULT5 renamed /OR/OR5
- net /OR/RESULT6 renamed /OR/OR6
- net /OR/RESULT7 renamed /OR/OR7
- J101 pad 11: unconnected-(J101-Pad11) -> /C3
- J101 pad 13: unconnected-(J101-Pad13) -> /C2
- J101 pad 15: unconnected-(J101-Pad15) -> /C1
- J101 pad 17: unconnected-(J101-Pad17) -> /C0
- J101 pad 3: unconnected-(J101-Pad3) -> /C7
- J101 pad 5: unconnected-(J101-Pad5) -> /C6
- J101 pad 7: unconnected-(J101-Pad7) -> /C5
- J101 pad 9: unconnected-(J101-Pad9) -> /C4
- U203 pad 1: /Adder-Subtractor/RESULT1 -> /Adder-Subtractor/AS1
- U203 pad 10: /Adder-Subtractor/RESULT3 -> /Adder-Subtractor/AS3
- U203 pad 13: /Adder-Subtractor/RESULT2 -> /Adder-Subtractor/AS2
- U203 pad 4: /Adder-Subtractor/RESULT0 -> /Adder-Subtractor/AS0
- U204 pad 1: /Adder-Subtractor/RESULT5 -> /Adder-Subtractor/AS5
- U204 pad 10: /Adder-Subtractor/RESULT7 -> /Adder-Subtractor/AS7
- U204 pad 13: /Adder-Subtractor/RESULT6 -> /Adder-Subtractor/AS6
- U204 pad 4: /Adder-Subtractor/RESULT4 -> /Adder-Subtractor/AS4
- U301 pad 11: /AND-NAND/RESULT2 -> /AND-NAND/NAND2
- U301 pad 3: /AND-NAND/RESULT0 -> /AND-NAND/NAND0
- U301 pad 6: unconnected-(U301-Pad6) -> /AND-NAND/NAND1
- U301 pad 8: /AND-NAND/RESULT3 -> /AND-NAND/NAND3
- U302 pad 11: /AND-NAND/RESULT6 -> /AND-NAND/NAND6
- U302 pad 3: /AND-NAND/RESULT4 -> /AND-NAND/NAND4
- U302 pad 6: /AND-NAND/RESULT5 -> /AND-NAND/NAND5
- U302 pad 8: /AND-NAND/RESULT7 -> /AND-NAND/NAND7
- U401 pad 11: /XOR/RESULT2 -> /Output Stage/XOR2
- U401 pad 3: /XOR/RESULT0 -> /Output Stage/XOR0
- U401 pad 6: /XOR/RESULT1 -> /Output Stage/XOR1
- U401 pad 8: /XOR/RESULT3 -> /Output Stage/XOR3
- U402 pad 11: /XOR/RESULT6 -> /Output Stage/XOR6
- U402 pad 3: /XOR/RESULT4 -> /Output Stage/XOR4
- U402 pad 6: /XOR/RESULT5 -> /Output Stage/XOR5
- U402 pad 8: /XOR/RESULT7 -> /Output Stage/XOR7

Commit message: Rethinking some design
Parts:
- removed U603: 74LS540, Package_DIP:DIP-20_W7.62mm_Socket
- removed U604, U605: 74HCT541, Package_DIP:DIP-20_W7.62mm_Socket
- added R601: 10k, Resistor_THT:R_Axial_DIN0207_L6.3mm_D2.5mm_P7.62mm_Horizontal, F.Cu at (256.5, 54.6)
- added RN601: R_Network08, Resistor_THT:R_Array_SIP9, F.Cu at (256.5, 40.6)
- added U204: 74HC125, Package_DIP:DIP-14_W7.62mm_Socket, F.Cu at (134.6, 61.0)
- added U207: 74HCT541, Package_DIP:DIP-20_W7.62mm_Socket, F.Cu at (133.4, 30.5)
- added U303: 74HCT541, Package_DIP:DIP-20_W7.62mm_Socket, F.Cu at (127.0, 100.3)
- added U304: 74LS540, Package_DIP:DIP-20_W7.62mm_Socket, F.Cu at (127.0, 129.5)
- added U403: 74HCT541, Package_DIP:DIP-20_W7.62mm_Socket, F.Cu at (201.9, 34.3)
- added U501: 74HCT541, Package_DIP:DIP-20_W7.62mm_Socket, F.Cu at (190.5, 99.1)
- U601: value 74HCT541 -> 74HC74; footprint Package_DIP:DIP-20_W7.62mm_Socket -> Package_DIP:DIP-14_W7.62mm_Socket
- U602: value 74HCT541 -> 74LS573
- moved U602 159.4 mm to (262.9, 17.8)
- moved U601 131.4 mm to (262.9, 52.1)
- moved D501 11.5 mm to (166.4, 99.1)
- moved D502 11.5 mm to (166.4, 102.9)
- moved D503 11.5 mm to (166.4, 106.7)
- moved D507 11.5 mm to (166.4, 121.9)
- moved D508 11.5 mm to (166.4, 125.7)
- moved D512 11.5 mm to (166.4, 141.0)
- moved D513 11.5 mm to (166.4, 144.8)
- moved D514 11.5 mm to (166.4, 148.6)
- moved D515 11.5 mm to (166.4, 152.4)
- moved D516 11.5 mm to (166.4, 156.2)
- moved R501 11.5 mm to (170.2, 99.1)
- moved R502 11.5 mm to (170.2, 106.7)
- moved R504 11.5 mm to (170.2, 121.9)
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- renumbered U205 to U203, U203 to U205, U204 to U206
Connections:
- net /Adder-Subtractor/B'0 renamed /AdderSubtractor/B'0
- net /Adder-Subtractor/B'1 renamed /AdderSubtractor/B'1
- net /Adder-Subtractor/B'2 renamed /AdderSubtractor/B'2
- net /Adder-Subtractor/B'3 renamed /AdderSubtractor/B'3
- net /Adder-Subtractor/B'4 renamed /AdderSubtractor/B'4
- net /Adder-Subtractor/B'5 renamed /AdderSubtractor/B'5
- net /Adder-Subtractor/B'6 renamed /AdderSubtractor/B'6
- net /Adder-Subtractor/B'7 renamed /AdderSubtractor/B'7
- net /Adder-Subtractor/~{ADD}/SUBTRACT renamed /AdderSubtractor/~{ADD}/SUBTRACT
- net /B0 renamed /AND-NAND/B0
- net /B1 renamed /AND-NAND/B1
- net /B2 renamed /AND-NAND/B2
- net /B3 renamed /AND-NAND/B3
- net /B4 renamed /AND-NAND/B4
- net /B5 renamed /AND-NAND/B5
- net /B6 renamed /AND-NAND/B6
- net /B7 renamed /AND-NAND/B7
- net /OR/OR0 renamed Net-(D501-Pad1)
- net /OR/OR1 renamed Net-(D503-Pad1)
- net /OR/OR2 renamed Net-(D505-Pad1)
- net /OR/OR3 renamed Net-(D507-Pad1)
- net /OR/OR4 renamed Net-(D509-Pad1)
- net /OR/OR5 renamed Net-(D511-Pad1)
- net /OR/OR6 renamed Net-(D513-Pad1)
- net /OR/OR7 renamed Net-(D515-Pad1)
- D501 pad 2: /A0 -> /AND-NAND/A0
- D503 pad 2: /A1 -> /AND-NAND/A1
- D505 pad 2: /A2 -> /AND-NAND/A2
- D507 pad 2: /A3 -> /AND-NAND/A3
- D509 pad 2: /A4 -> /AND-NAND/A4
- D511 pad 2: /A5 -> /AND-NAND/A5
- D513 pad 2: /A6 -> /AND-NAND/A6
- D515 pad 2: /A7 -> /AND-NAND/A7
- J101 pad 10: /A4 -> unconnected-(J101-Pad10)
- J101 pad 11: /C3 -> unconnected-(J101-Pad11)
- J101 pad 12: /A3 -> unconnected-(J101-Pad12)
- J101 pad 13: /C2 -> unconnected-(J101-Pad13)
- J101 pad 14: /A2 -> unconnected-(J101-Pad14)
- J101 pad 15: /C1 -> unconnected-(J101-Pad15)
- J101 pad 16: /A1 -> unconnected-(J101-Pad16)
- J101 pad 17: /C0 -> unconnected-(J101-Pad17)
- J101 pad 18: /A0 -> unconnected-(J101-Pad18)
- J101 pad 3: /C7 -> /C_{bus}0
- J101 pad 4: /A7 -> /A.A7
- J101 pad 5: /C6 -> unconnected-(J101-Pad5)
- J101 pad 6: /A6 -> unconnected-(J101-Pad6)
- J101 pad 7: /C5 -> unconnected-(J101-Pad7)
- J101 pad 8: /A5 -> unconnected-(J101-Pad8)
- J101 pad 9: /C4 -> unconnected-(J101-Pad9)
- U201 pad 14: unconnected-(U201-Pad14) -> +5V
- U201 pad 7: unconnected-(U201-Pad7) -> GND
- U202 pad 14: unconnected-(U202-Pad14) -> +5V
- U202 pad 7: unconnected-(U202-Pad7) -> GND
- U203 pad 14: unconnected-(U205-Pad14) -> +5V
- U203 pad 3: /Adder-Subtractor/FLAG -> Net-(U203-Pad3)
- U203 pad 7: unconnected-(U205-Pad7) -> GND
- U205 pad 1: /Adder-Subtractor/AS1 -> Net-(U205-Pad1)
- U205 pad 10: /Adder-Subtractor/AS3 -> Net-(U205-Pad10)
- U205 pad 12: /A3 -> /AdderSubtractor/A3
- U205 pad 13: /Adder-Subtractor/AS2 -> Net-(U205-Pad13)
- U205 pad 14: /A2 -> /AdderSubtractor/A2
- U205 pad 16: unconnected-(U203-Pad16) -> +5V
- U205 pad 3: /A1 -> /AdderSubtractor/A1
- U205 pad 4: /Adder-Subtractor/AS0 -> Net-(U205-Pad4)
- U205 pad 5: /A0 -> /AdderSubtractor/A0
- U205 pad 8: unconnected-(U203-Pad8) (its old number) -> GND
- U206 pad 1: /Adder-Subtractor/AS5 -> Net-(U206-Pad1)
- U206 pad 10: /Adder-Subtractor/AS7 -> Net-(U206-Pad10)
- U206 pad 12: /A7 -> /AdderSubtractor/A7
- U206 pad 13: /Adder-Subtractor/AS6 -> Net-(U206-Pad13)
- U206 pad 14: /A6 -> /AdderSubtractor/A6
- U206 pad 16: unconnected-(U204-Pad16) -> +5V
- U206 pad 3: /A5 -> /AdderSubtractor/A5
- U206 pad 4: /Adder-Subtractor/AS4 -> Net-(U206-Pad4)
- U206 pad 5: /A4 -> /AdderSubtractor/A4
- U206 pad 8: unconnected-(U204-Pad8) -> GND
- U301 pad 1: /A0 -> /AND-NAND/A0
- U301 pad 12: /A2 -> /AND-NAND/A2
- U301 pad 14: unconnected-(U301-Pad14) -> +5V
- U301 pad 4: /A1 -> /AND-NAND/A1
- U301 pad 7: unconnected-(U301-Pad7) -> GND
- U301 pad 9: /A3 -> /AND-NAND/A3
- U302 pad 1: /A4 -> /AND-NAND/A4
- U302 pad 12: /A6 -> /AND-NAND/A6
- U302 pad 14: unconnected-(U302-Pad14) -> +5V
- U302 pad 4: /A5 -> /AND-NAND/A5
- U302 pad 7: unconnected-(U302-Pad7) -> GND
- U302 pad 9: /A7 -> /AND-NAND/A7
- U401 pad 1: /A0 -> /AND-NAND/A0
- U401 pad 11: /Output Stage/XOR2 -> Net-(U401-Pad11)
- U401 pad 12: /A2 -> /AND-NAND/A2
- U401 pad 14: unconnected-(U401-Pad14) -> +5V
- U401 pad 3: /Output Stage/XOR0 -> Net-(U401-Pad3)
- U401 pad 4: /A1 -> /AND-NAND/A1
- U401 pad 6: /Output Stage/XOR1 -> Net-(U401-Pad6)
- U401 pad 7: unconnected-(U401-Pad7) -> GND
- U401 pad 8: /Output Stage/XOR3 -> Net-(U401-Pad8)
- U401 pad 9: /A3 -> /AND-NAND/A3
- U402 pad 1: /A4 -> /AND-NAND/A4
- U402 pad 11: /Output Stage/XOR6 -> Net-(U402-Pad11)
- U402 pad 12: /A6 -> /AND-NAND/A6
- U402 pad 14: unconnected-(U402-Pad14) -> +5V
- U402 pad 3: /Output Stage/XOR4 -> Net-(U402-Pad3)
- U402 pad 4: /A5 -> /AND-NAND/A5
- U402 pad 6: /Output Stage/XOR5 -> Net-(U402-Pad6)
- U402 pad 7: unconnected-(U402-Pad7) -> GND
- U402 pad 8: /Output Stage/XOR7 -> Net-(U402-Pad8)
- U402 pad 9: /A7 -> /AND-NAND/A7
- U601 pad 1: unconnected-(U601-Pad1) -> +5V
- U601 pad 10: unconnected-(U601-Pad10) -> +5V
- U601 pad 11: /C7 -> GND
- U601 pad 12: /C6 -> GND
- U601 pad 13: /C5 -> +5V
- U601 pad 14: /C4 -> +5V
- U601 pad 2: /Adder-Subtractor/AS0 -> /Output Stage/FLAG
- U601 pad 3: /Adder-Subtractor/AS1 -> Net-(U601-Pad3)
- U601 pad 4: /Adder-Subtractor/AS2 -> +5V
- U601 pad 5: /Adder-Subtractor/AS3 -> /Output Stage/DALUFLAG
- U601 pad 6: /Adder-Subtractor/AS4 -> unconnected-(U601-Pad6)
- U601 pad 7: /Adder-Subtractor/AS5 -> GND
- U601 pad 8: /Adder-Subtractor/AS6 -> unconnected-(U601-Pad8)
- U601 pad 9: /Adder-Subtractor/AS7 -> unconnected-(U601-Pad9)
- U602 pad 10: unconnected-(U602-Pad10) -> GND
- U602 pad 11: /C7 -> Net-(U601-Pad3)
- U602 pad 12: /C6 -> unconnected-(U602-Pad12)
- U602 pad 13: /C5 -> unconnected-(U602-Pad13)
- U602 pad 14: /C4 -> unconnected-(U602-Pad14)
- U602 pad 15: /C3 -> unconnected-(U602-Pad15)
- U602 pad 16: /C2 -> unconnected-(U602-Pad16)
- U602 pad 17: /C1 -> unconnected-(U602-Pad17)
- U602 pad 18: /C0 -> unconnected-(U602-Pad18)
- U602 pad 2: /AND-NAND/NAND0 -> Net-(U602-Pad2)
- U602 pad 20: unconnected-(U602-Pad20) -> +5V
- U602 pad 3: /AND-NAND/NAND1 -> Net-(U602-Pad3)
- U602 pad 4: /AND-NAND/NAND2 -> Net-(U602-Pad4)
- U602 pad 5: /AND-NAND/NAND3 -> Net-(U602-Pad5)
- U602 pad 6: /AND-NAND/NAND4 -> Net-(U602-Pad6)
- U602 pad 7: /AND-NAND/NAND5 -> Net-(U602-Pad7)
- U602 pad 8: /AND-NAND/NAND6 -> Net-(U602-Pad8)
- U602 pad 9: /AND-NAND/NAND7 -> Net-(U602-Pad9)

Commit message: Thinking about some of the control logic
Parts:
- added D601: 1N4148, Diode_THT:D_DO-35_SOD27_P7.62mm_Horizontal, F.Cu at (262.9, 20.3)
- added D602: 1N4148, Diode_THT:D_DO-35_SOD27_P7.62mm_Horizontal, F.Cu at (262.9, 25.4)
- added R201: 100k, Resistor_THT:R_Axial_DIN0207_L6.3mm_D2.5mm_P7.62mm_Horizontal, F.Cu at (125.7, 38.1)
- added R601: 100k, Resistor_THT:R_Axial_DIN0207_L6.3mm_D2.5mm_P7.62mm_Horizontal, F.Cu at (265.4, 20.3)
- added R602: 10k, Resistor_THT:R_Axial_DIN0207_L6.3mm_D2.5mm_P7.62mm_Horizontal, F.Cu at (293.4, 47.0)
- added R603: 100k, Resistor_THT:R_Axial_DIN0207_L6.3mm_D2.5mm_P7.62mm_Horizontal, F.Cu at (262.9, 30.5)
- added R604: 100k, Resistor_THT:R_Axial_DIN0207_L6.3mm_D2.5mm_P7.62mm_Horizontal, F.Cu at (275.6, 35.6)
- added U602: 74HC125, Package_DIP:DIP-14_W7.62mm_Socket, F.Cu at (275.6, 15.2)
- U205, U206: value 74LS283 -> 74HC283
- moved U202 56.2 mm to (83.8, 36.8)
- moved R605 39.0 mm to (293.4, 41.9), turned to 180 degrees
- moved U601 36.2 mm to (297.2, 40.6)
- moved U603 36.2 mm to (297.2, 6.34)
- moved RN601 36.2 mm to (290.8, 29.2)
- moved U204 30.5 mm to (83.8, 58.4)
- moved U207 25.1 mm to (111.8, 43.2)
- renumbered R601 to R605, U204 to U202, U202 to U203, U203 to U204, U602 to U603
Connections:
- net Net-(U601-Pad3) renamed /Output Stage/CLK
- U201 pad 10: /AdderSubtractor/~{ADD}/SUBTRACT -> Net-(U201-Pad10)
- U201 pad 13: /AdderSubtractor/~{ADD}/SUBTRACT -> Net-(U201-Pad10)
- U201 pad 2: /AdderSubtractor/~{ADD}/SUBTRACT -> Net-(U201-Pad10)
- U201 pad 5: /AdderSubtractor/~{ADD}/SUBTRACT -> Net-(U201-Pad10)
- U202 pad 11: unconnected-(U204-Pad11) -> Net-(U203-Pad10)
- U202 pad 12: GND -> /AdderSubtractor/~{ADD}/SUBTRACT
- U202 pad 4: GND -> /AdderSubtractor/~{ENABLE_{DALU}}
- U202 pad 5: GND -> Net-(U202-Pad5)
- U202 pad 6: unconnected-(U204-Pad6) -> /AdderSubtractor/~{ENABLE_{AS}}
- U202 pad 8: unconnected-(U204-Pad8) -> Net-(U201-Pad10)
- U202 pad 9: GND -> /AdderSubtractor/~{ADD}/SUBTRACT
- U203 pad 10: /AdderSubtractor/~{ADD}/SUBTRACT -> Net-(U203-Pad10)
- U203 pad 13: /AdderSubtractor/~{ADD}/SUBTRACT -> Net-(U203-Pad10)
- U203 pad 2: /AdderSubtractor/~{ADD}/SUBTRACT -> Net-(U203-Pad10)
- U203 pad 5: /AdderSubtractor/~{ADD}/SUBTRACT -> Net-(U203-Pad10)
- U204 pad 10: GND -> +5V
- U204 pad 11: unconnected-(U203-Pad11) -> /AdderSubtractor/~{ADD}/SUBTRACT
- U204 pad 13: GND -> /AdderSubtractor/~{ENABLE_{ADD}}
- U204 pad 4: GND -> /AdderSubtractor/~{ENABLE_{ADD}}
- U204 pad 5: GND -> /AdderSubtractor/~{ENABLE_{SUBTRACT}}
- U204 pad 6: unconnected-(U203-Pad6) -> Net-(U204-Pad6)
- U204 pad 8: unconnected-(U203-Pad8) -> Net-(U202-Pad5)
- U204 pad 9: GND -> Net-(U204-Pad6)
- U603 pad 1: unconnected-(U602-Pad1) -> Net-(U603-Pad1)

Commit message: Thinking about SMD assembly. Will be rethinking
Parts:
- added U101: 74HC245, Package_SO:SOIC-20W_7.5x12.8mm_P1.27mm, F.Cu at (63.5, 108.0)
- added U102: 74HC245, Package_SO:SOIC-20W_7.5x12.8mm_P1.27mm, F.Cu at (63.5, 125.7)
- U201: footprint Package_DIP:DIP-14_W7.62mm_Socket -> Package_SO:TSSOP-14_4.4x5mm_P0.65mm
- U205: footprint Package_DIP:DIP-16_W7.62mm_Socket -> Package_SO:SOIC-16_3.9x9.9mm_P1.27mm
- U603: value 74LS573 -> 74HCT574; footprint Package_DIP:DIP-20_W7.62mm_Socket -> Package_SO:SOIC-20W_7.5x12.8mm_P1.27mm
- moved J101 62.4 mm to (44.5, 95.2)
- moved U603 14.5 mm to (301.0, 20.3)
- moved U205 11.4 mm to (101.6, 44.5)
- moved U201 10.9 mm to (74.9, 47.0)
Connections:
- J101 pad 10: unconnected-(J101-Pad10) -> Net-(J101-Pad10)
- J101 pad 12: unconnected-(J101-Pad12) -> Net-(J101-Pad12)
- J101 pad 14: unconnected-(J101-Pad14) -> Net-(J101-Pad14)
- J101 pad 16: unconnected-(J101-Pad16) -> Net-(J101-Pad16)
- J101 pad 18: unconnected-(J101-Pad18) -> Net-(J101-Pad18)
- J101 pad 24: /AND-NAND/B7 -> Net-(J101-Pad24)
- J101 pad 26: /AND-NAND/B6 -> Net-(J101-Pad26)
- J101 pad 28: /AND-NAND/B5 -> Net-(J101-Pad28)
- J101 pad 3: /C_{bus}0 -> unconnected-(J101-Pad3)
- J101 pad 30: /AND-NAND/B4 -> Net-(J101-Pad30)
- J101 pad 32: /AND-NAND/B3 -> Net-(J101-Pad32)
- J101 pad 34: /AND-NAND/B2 -> Net-(J101-Pad34)
- J101 pad 36: /AND-NAND/B1 -> Net-(J101-Pad36)
- J101 pad 38: /AND-NAND/B0 -> Net-(J101-Pad38)
- J101 pad 4: /A.A7 -> Net-(J101-Pad4)
- J101 pad 6: unconnected-(J101-Pad6) -> Net-(J101-Pad6)
- J101 pad 8: unconnected-(J101-Pad8) -> Net-(J101-Pad8)

Commit message: Doing some rethinking
Parts:
- removed J101: Conn_02x20_Odd_Even, Connector_PinHeader_2.54mm:PinHeader_2x20_P2.54mm_Vertical
- removed U101, U102: 74HC245, Package_SO:SOIC-20W_7.5x12.8mm_P1.27mm
- removed U207: 74HCT541, Package_DIP:DIP-20_W7.62mm_Socket
- removed the U303 at (127.0, 100.3)
- removed the U304 at (127.0, 129.5)
- removed the U501 at (190.5, 99.1)
- added J201: Conn_02x20_Odd_Even, Connector_PinHeader_2.54mm:PinHeader_2x20_P2.54mm_Vertical, F.Cu at (34.3, 99.1)
- added U201: 74HC245, Package_SO:SOIC-20W_7.5x12.8mm_P1.27mm, F.Cu at (58.4, 143.5)
- added U202: 74HC245, Package_SO:SOIC-20W_7.5x12.8mm_P1.27mm, F.Cu at (58.4, 104.1)
- added U203: 74HC245, Package_SO:SOIC-20W_7.5x12.8mm_P1.27mm, F.Cu at (58.4, 123.2)
- added U307: 74HC245, Package_SO:SOIC-20W_7.5x12.8mm_P1.27mm, F.Cu at (124.5, 58.4)
- added U404: 74HC245, Package_SO:SOIC-20W_7.5x12.8mm_P1.27mm, F.Cu at (135.9, 137.2)
- added U503: 74HC245, Package_SO:SOIC-20W_7.5x12.8mm_P1.27mm, F.Cu at (196.8, 40.6)
- added U601: 74HC245, Package_SO:SOIC-20W_7.5x12.8mm_P1.27mm, F.Cu at (195.6, 106.7)
- U301: renamed from U201; footprint Package_SO:TSSOP-14_4.4x5mm_P0.65mm -> Package_DIP:DIP-14_W7.62mm_Socket
- U305: renamed from U205; footprint Package_SO:SOIC-16_3.9x9.9mm_P1.27mm -> Package_DIP:DIP-16_W7.62mm_Socket
- U403: value 74HCT541 -> 74HC245; footprint Package_DIP:DIP-20_W7.62mm_Socket -> Package_SO:SOIC-20W_7.5x12.8mm_P1.27mm
- U703: renamed from U603; footprint Package_SO:SOIC-20W_7.5x12.8mm_P1.27mm -> Package_DIP:DIP-20_W7.62mm_Socket
- moved U403 104.6 mm to (134.6, 114.3)
- moved U301 10.9 mm to (71.1, 36.8)
- moved U305 10.2 mm to (96.5, 35.5)
- renumbered D501 to D601, D502 to D602, D503 to D603, D504 to D604, D505 to D605, D506 to D606, D507 to D607, D508 to D608, D509 to D609, D510 to D610, D511 to D611, D512 to D612, D513 to D613, D514 to D614, D515 to D615, D516 to D616, D601 to D701, D602 to D702, R201 to R301, R501 to R601, R502 to R602, R503 to R603, R504 to R604, R505 to R605, R506 to R606, R507 to R607, R508 to R608, R601 to R701, R602 to R702, R603 to R703, R604 to R704, R605 to R705, RN601 to RN701, U202 to U302, U203 to U303, U204 to U304, U206 to U306, U301 to U401, U302 to U402, U401 to U501, U402 to U502, U601 to U701, U602 to U702
Connections:
- U403 pad 1: /XOR/~{ENABLE_{XOR}} -> unconnected-(U403-Pad1)
- U403 pad 19: /XOR/~{ENABLE_{XOR}} -> unconnected-(U403-Pad19)
- U403 pad 2: Net-(U401-Pad3) -> /AND-NAND/NAND0
- U403 pad 3: Net-(U401-Pad6) -> /AND-NAND/NAND1
- U403 pad 4: Net-(U401-Pad11) -> /AND-NAND/NAND2
- U403 pad 5: Net-(U401-Pad8) -> /AND-NAND/NAND3
- U403 pad 6: Net-(U402-Pad3) -> /AND-NAND/NAND4
- U403 pad 7: Net-(U402-Pad6) -> /AND-NAND/NAND5
- U403 pad 8: Net-(U402-Pad11) -> /AND-NAND/NAND6
- U403 pad 9: Net-(U402-Pad8) -> /AND-NAND/NAND7
- U501 pad 11: Net-(U401-Pad11) -> Net-(U501-Pad11)
- U501 pad 3: Net-(U401-Pad3) -> Net-(U501-Pad3)
- U501 pad 6: Net-(U401-Pad6) -> Net-(U501-Pad6)
- U501 pad 8: Net-(U401-Pad8) -> Net-(U501-Pad8)
- U502 pad 11: Net-(U402-Pad11) -> Net-(U502-Pad11)
- U502 pad 3: Net-(U402-Pad3) -> Net-(U502-Pad3)
- U502 pad 6: Net-(U402-Pad6) -> Net-(U502-Pad6)
- U502 pad 8: Net-(U402-Pad8) -> Net-(U502-Pad8)
