File: pcbs/DALU/xor.kicad_sch (KiCad schematic)
At the start: 2 parts, among them U401 74HC86, U402 74HC86

Commit message: Last of the compute stages
Connections:
- net RESULT5: now reaches U402.6
- net RESULT7: now reaches U402.8
- net RESULT3: now reaches U401.8
- net RESULT6: now reaches U402.11
- net RESULT4: now reaches U402.3
- net RESULT2: now reaches U401.11
- net RESULT1: now reaches U401.6
Changed lines of the file:
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@@
+    (stroke (width 0) (type default) (color 0 0 0 0))
+  )
+  (bus_entry (at 142.24 55.88) (size -2.54 2.54)
     (stroke (width 0) (type default) (color 0 0 0 0))
   )
@@
     (stroke (width 0) (type default) (color 0 0 0 0))
   )
+  (bus_entry (at 142.24 69.85) (size -2.54 2.54)
+    (stroke (width 0) (type default) (color 0 0 0 0))
+  )
+  (bus_entry (at 142.24 83.82) (size -2.54 2.54)
+    (stroke (width 0) (type default) (color 0 0 0 0))
+  )
   (bus_entry (at 88.9 53.34) (size 2.54 2.54)
     (stroke (width 0) (type default) (color 0 0 0 0))
   )
+  (bus_entry (at 142.24 113.03) (size -2.54 2.54)
+    (stroke (width 0) (type default) (color 0 0 0 0))
+  )
   (bus_entry (at 83.82 143.51) (size 2.54 2.54)
     (stroke (width 0) (type default) (color 0 0 0 0))
   )
+  (bus_entry (at 142.24 99.06) (size -2.54 2.54)
+    (stroke (width 0) (type default) (color 0 0 0 0))
+  )
   (bus_entry (at 88.9 96.52) (size 2.54 2.54)
     (stroke (width 0) (type default) (color 0 0 0 0))
   )
+  (bus_entry (at 142.24 127) (size -2.54 2.54)
+    (stroke (width 0) (type default) (color 0 0 0 0))
+  )
   (bus_entry (at 88.9 81.28) (size 2.54 2.54)
     (stroke (width 0) (type default) (color 0 0 0 0))
@@
     (stroke (width 0) (type default) (color 0 0 0 0))
   )
+  (bus_entry (at 142.24 140.97) (size -2.54 2.54)
+    (stroke (width 0) (type default) (color 0 0 0 0))
+  )
   (bus_entry (at 88.9 39.37) (size 2.54 2.54)
     (stroke (width 0) (type default) (color 0 0 0 0))
@@
     (stroke (width 0) (type default) (color 0 0 0 0))
   )
+  (wire (pts (xy 116.84 101.6) (xy 139.7 101.6))
+    (stroke (width 0) (type default) (color 0 0 0 0))
+  )
   (bus (pts (xy 38.1 25.4) (xy 88.9 25.4))
     (stroke (width 0) (type default) (color 0 0 0 0))
@@
     (stroke (width 0) (type default) (color 0 0 0 0))
   )
+  (bus (pts (xy 142.24 55.88) (xy 142.24 69.85))
+    (stroke (width 0) (type default) (color 0 0 0 0))
+  )
   (bus (pts (xy 88.9 53.34) (xy 88.9 67.31))
     (stroke (width 0) (type default) (color 0 0 0 0))
@@
     (stroke (width 0) (type default) (color 0 0 0 0))
   )
-  (bus (pts (xy 142.24 41.91) (xy 142.24 140.97))
+  (bus (pts (xy 142.24 83.82) (xy 142.24 99.06))
+    (stroke (width 0) (type default) (color 0 0 0 0))
+  )
+  (bus (pts (xy 142.24 41.91) (xy 142.24 55.88))
     (stroke (width 0) (type default) (color 0 0 0 0))
   )
@@
     (stroke (width 0) (type default) (color 0 0 0 0))
   )
+  (wire (pts (xy 116.84 58.42) (xy 139.7 58.42))
+    (stroke (width 0) (type default) (color 0 0 0 0))
+  )
+  (wire (pts (xy 116.84 115.57) (xy 139.7 115.57))
+    (stroke (width 0) (type default) (color 0 0 0 0))
+  )
+  (bus (pts (xy 142.24 127) (xy 142.24 140.97))
+    (stroke (width 0) (type default) (color 0 0 0 0))
+  )
   (wire (pts (xy 86.36 132.08) (xy 101.6 132.08))
     (stroke (width 0) (type default) (color 0 0 0 0))
@@
     (stroke (width 0) (type default) (color 0 0 0 0))
   )
+  (wire (pts (xy 116.84 129.54) (xy 139.7 129.54))
+    (stroke (width 0) (type default) (color 0 0 0 0))
+  )
   (wire (pts (xy 86.36 46.99) (xy 101.6 46.99))
     (stroke (width 0) (type default) (color 0 0 0 0))
@@
     (stroke (width 0) (type default) (color 0 0 0 0))
   )
+  (wire (pts (xy 116.84 143.51) (xy 139.7 143.51))
+    (stroke (width 0) (type default) (color 0 0 0 0))
+  )
   (wire (pts (xy 86.36 74.93) (xy 101.6 74.93))
     (stroke (width 0) (type default) (color 0 0 0 0))
@@
     (stroke (width 0) (type default) (color 0 0 0 0))
   )
+  (wire (pts (xy 116.84 86.36) (xy 139.7 86.36))
+    (stroke (width 0) (type default) (color 0 0 0 0))
+  )
+  (bus (pts (xy 142.24 113.03) (xy 142.24 127))
+    (stroke (width 0) (type default) (color 0 0 0 0))
+  )
   (wire (pts (xy 86.36 88.9) (xy 101.6 88.9))
     (stroke (width 0) (type default) (color 0 0 0 0))
@@
     (stroke (width 0) (type default) (color 0 0 0 0))
   )
+  (bus (pts (xy 142.24 69.85) (xy 142.24 83.82))
+    (stroke (width 0) (type default) (color 0 0 0 0))
+  )
   (bus (pts (xy 83.82 129.54) (xy 83.82 143.51))
     (stroke (width 0) (type default) (color 0 0 0 0))
@@
     (stroke (width 0) (type default) (color 0 0 0 0))
   )
+  (wire (pts (xy 116.84 72.39) (xy 139.7 72.39))
+    (stroke (width 0) (type default) (color 0 0 0 0))
+  )
+  (bus (pts (xy 142.24 99.06) (xy 142.24 113.03))
+    (stroke (width 0) (type default) (color 0 0 0 0))
+  )
+  (label "RESULT7" (at 116.84 143.51 0)
+    (effects (font (size 1.27 1.27)) (justify left bottom))
+  )
   (label "A[0..7]" (at 60.96 25.4 0)
     (effects (font (size 1.27 1.27)) (justify left bottom))
@@
     (effects (font (size 1.27 1.27)) (justify left bottom))
   )
+  (label "RESULT6" (at 116.84 129.54 0)
+    (effects (font (size 1.27 1.27)) (justify left bottom))
+  )
   (label "A4" (at 91.44 99.06 0)
     (effects (font (size 1.27 1.27)) (justify left bottom))
@@
     (effects (font (size 1.27 1.27)) (justify left bottom))
   )
+  (label "RESULT5" (at 116.84 115.57 0)
+    (effects (font (size 1.27 1.27)) (justify left bottom))
+  )
   (label "B0" (at 91.44 46.99 0)
     (effects (font (size 1.27 1.27)) (justify left bottom))
   )
+  (label "RESULT3" (at 116.84 86.36 0)
+    (effects (font (size 1.27 1.27)) (justify left bottom))
+  )
+  (label "RESULT4" (at 116.84 101.6 0)
+    (effects (font (size 1.27 1.27)) (justify left bottom))
+  )
+  (label "RESULT2" (at 116.84 72.39 0)
+    (effects (font (size 1.27 1.27)) (justify left bottom))
+  )
   (label "A1" (at 91.44 55.88 0)
     (effects (font (size 1.27 1.27)) (justify left bottom))
@@
     (effects (font (size 1.27 1.27)) (justify left bottom))
   )
+  (label "RESULT1" (at 116.84 58.42 0)
+    (effects (font (size 1.27 1.27)) (justify left bottom))
+  )

Commit message: Trying to figure out the hierarchical buses
Connections:
- net RESULT0 renamed XOR0
- net RESULT1 renamed XOR1
- net RESULT2 renamed XOR2
- net RESULT3 renamed XOR3
- net RESULT4 renamed XOR4
- net RESULT5 renamed XOR5
- net RESULT6 renamed XOR6
- net RESULT7 renamed XOR7
Changed lines of the file:
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@@
     (stroke (width 0) (type default) (color 0 0 0 0))
   )
-  (label "RESULT7" (at 116.84 143.51 0)
-    (effects (font (size 1.27 1.27)) (justify left bottom))
-  )
-  (label "A[0..7]" (at 60.96 25.4 0)
+  (label "XOR7" (at 116.84 143.51 0)
     (effects (font (size 1.27 1.27)) (justify left bottom))
   )
@@
     (effects (font (size 1.27 1.27)) (justify left bottom))
   )
-  (label "RESULT6" (at 116.84 129.54 0)
+  (label "XOR6" (at 116.84 129.54 0)
     (effects (font (size 1.27 1.27)) (justify left bottom))
   )
   (label "A4" (at 91.44 99.06 0)
-    (effects (font (size 1.27 1.27)) (justify left bottom))
-  )
-  (label "B[0..7]" (at 60.96 30.48 0)
     (effects (font (size 1.27 1.27)) (justify left bottom))
   )
@@
     (effects (font (size 1.27 1.27)) (justify left bottom))
   )
-  (label "RESULT5" (at 116.84 115.57 0)
+  (label "XOR5" (at 116.84 115.57 0)
     (effects (font (size 1.27 1.27)) (justify left bottom))
   )
@@
     (effects (font (size 1.27 1.27)) (justify left bottom))
   )
-  (label "RESULT3" (at 116.84 86.36 0)
+  (label "XOR3" (at 116.84 86.36 0)
     (effects (font (size 1.27 1.27)) (justify left bottom))
   )
-  (label "RESULT4" (at 116.84 101.6 0)
+  (label "XOR4" (at 116.84 101.6 0)
     (effects (font (size 1.27 1.27)) (justify left bottom))
   )
-  (label "RESULT2" (at 116.84 72.39 0)
+  (label "XOR2" (at 116.84 72.39 0)
     (effects (font (size 1.27 1.27)) (justify left bottom))
   )
@@
     (effects (font (size 1.27 1.27)) (justify left bottom))
   )
-  (label "RESULT[0..7]" (at 143.51 27.94 0)
+  (label "XOR1" (at 116.84 58.42 0)
     (effects (font (size 1.27 1.27)) (justify left bottom))
   )
-  (label "RESULT1" (at 116.84 58.42 0)
-    (effects (font (size 1.27 1.27)) (justify left bottom))
-  )
-  (label "RESULT0" (at 116.84 44.45 0)
+  (label "XOR0" (at 116.84 44.45 0)
     (effects (font (size 1.27 1.27)) (justify left bottom))
   )
@@
     (effects (font (size 1.27 1.27)) (justify left bottom))
   )
-  (hierarchical_label "A_{bus}" (shape input) (at 38.1 25.4 180)
+  (hierarchical_label "A[0..7]" (shape input) (at 38.1 25.4 180)
     (effects (font (size 1.27 1.27)) (justify right))
   )
-  (hierarchical_label "XOR_{bus}" (shape output) (at 163.83 27.94 0)
+  (hierarchical_label "XOR[0..7]" (shape output) (at 163.83 27.94 0)
     (effects (font (size 1.27 1.27)) (justify left))
   )
-  (hierarchical_label "B_{bus}" (shape input) (at 38.1 30.48 180)
+  (hierarchical_label "B[0..7]" (shape input) (at 38.1 30.48 180)
     (effects (font (size 1.27 1.27)) (justify right))
   )

Commit message: Trying to get everything together
Connections:
- net +5V: now reaches U402.14 (VCC)
- net +5V: now also U401.14 (VCC)
- net GND: now reaches U402.7 (GND)
- net GND: now also U401.7 (GND)
Changed lines of the file:
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@@
+    (stroke (width 0) (type default) (color 0 0 0 0))
+  )
+  (wire (pts (xy 29.21 156.21) (xy 29.21 158.75))
     (stroke (width 0) (type default) (color 0 0 0 0))
   )
@@
     (stroke (width 0) (type default) (color 0 0 0 0))
   )
+  (wire (pts (xy 29.21 184.15) (xy 29.21 186.69))
+    (stroke (width 0) (type default) (color 0 0 0 0))
+  )
   (wire (pts (xy 116.84 44.45) (xy 139.7 44.45))
     (stroke (width 0) (type default) (color 0 0 0 0))
   )
+  (wire (pts (xy 57.15 184.15) (xy 57.15 186.69))
+    (stroke (width 0) (type default) (color 0 0 0 0))
+  )
   (wire (pts (xy 86.36 60.96) (xy 101.6 60.96))
     (stroke (width 0) (type default) (color 0 0 0 0))
@@
   )
   (bus (pts (xy 83.82 30.48) (xy 83.82 44.45))
+    (stroke (width 0) (type default) (color 0 0 0 0))
+  )
+  (wire (pts (xy 57.15 156.21) (xy 57.15 158.75))
     (stroke (width 0) (type default) (color 0 0 0 0))
   )
@@
     (pin "7")
   )
+  (symbol (lib_id "power:GND") (at 57.15 186.69 0) (unit 1)
+    (in_bom yes) (on_board yes) (fields_autoplaced)
+    (property "Reference" "#PWR0404" (id 0) (at 57.15 193.04 0)
+      (effects (font (size 1.27 1.27)) hide)
+    )
+    (property "Value" "GND" (id 1) (at 57.15 191.77 0))
+    (property "Footprint" "" (id 2) (at 57.15 186.69 0)
+      (effects (font (size 1.27 1.27)) hide)
+    )
+    (property "Datasheet" "" (id 3) (at 57.15 186.69 0)
+      (effects (font (size 1.27 1.27)) hide)
+    )
+    (pin "1")
+  )
+  (symbol (lib_id "power:GND") (at 29.21 186.69 0) (unit 1)
+    (in_bom yes) (on_board yes) (fields_autoplaced)
+    (property "Reference" "#PWR0402" (id 0) (at 29.21 193.04 0)
+      (effects (font (size 1.27 1.27)) hide)
+    )
+    (property "Value" "GND" (id 1) (at 29.21 191.77 0))
+    (property "Footprint" "" (id 2) (at 29.21 186.69 0)
+      (effects (font (size 1.27 1.27)) hide)
+    )
+    (property "Datasheet" "" (id 3) (at 29.21 186.69 0)
+      (effects (font (size 1.27 1.27)) hide)
+    )
+    (pin "1")
+  )
+  (symbol (lib_id "power:+5V") (at 29.21 156.21 0) (unit 1)
+    (in_bom yes) (on_board yes) (fields_autoplaced)
+    (property "Reference" "#PWR0401" (id 0) (at 29.21 160.02 0)
+      (effects (font (size 1.27 1.27)) hide)
+    )
+    (property "Value" "+5V" (id 1) (at 29.21 151.13 0))
+    (property "Footprint" "" (id 2) (at 29.21 156.21 0)
+      (effects (font (size 1.27 1.27)) hide)
+    )
+    (property "Datasheet" "" (id 3) (at 29.21 156.21 0)
+      (effects (font (size 1.27 1.27)) hide)
+    )
+    (pin "1")
+  )
   (symbol (lib_id "74xx:74HC86") (at 109.22 129.54 0) (unit 4)
     (in_bom yes) (on_board yes) (fields_autoplaced)
@@
     (pin "7")
   )
+  (symbol (lib_id "power:+5V") (at 57.15 156.21 0) (unit 1)
+    (in_bom yes) (on_board yes) (fields_autoplaced)
+    (property "Reference" "#PWR0403" (id 0) (at 57.15 160.02 0)
+      (effects (font (size 1.27 1.27)) hide)
+    )
+    (property "Value" "+5V" (id 1) (at 57.15 151.13 0))
+    (property "Footprint" "" (id 2) (at 57.15 156.21 0)
+      (effects (font (size 1.27 1.27)) hide)
+    )
+    (property "Datasheet" "" (id 3) (at 57.15 156.21 0)
+      (effects (font (size 1.27 1.27)) hide)
+    )
+    (pin "1")
+  )
 )

Commit message: Rethinking some design
Parts:
- added U403: 74HCT541, Package_DIP:DIP-20_W7.62mm_Socket, symbol 74xx:74HCT541
Connections:
- net +5V: now also U403.20 (VCC)
- net GND: now also U403.10 (GND)
- net XOR0: no longer names the net of U401.3
- net XOR0: now also U403.2 (A0)
- net XOR1: no longer names the net of U401.6
- net XOR1: now also U403.3 (A1)
- net XOR2: no longer names the net of U401.11
- net XOR2: now also U403.4 (A2)
- net XOR3: no longer names the net of U401.8
- net XOR3: now also U403.5 (A3)
- net XOR4: no longer names the net of U402.3
- net XOR4: now also U403.6 (A4)
- net XOR5: no longer names the net of U402.6
- net XOR5: now also U403.7 (A5)
- net XOR6: no longer names the net of U402.11
- net XOR6: now also U403.8 (A6)
- net XOR7: no longer names the net of U402.8
- net XOR7: now also U403.9 (A7)
- new net ~{ENABLE_{XOR}}: U403.1 (G1), U403.19 (G2)

Commit message: Thinking about some of the control logic
Parts:
- U401, U402: footprint (none) -> Package_DIP:DIP-14_W7.62mm_Socket
Changed lines of the file:
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@@
       (effects (font (size 1.27 1.27)) (justify left))
     )
-    (property "Footprint" "" (id 2) (at 57.15 171.45 0)
+    (property "Footprint" "Package_DIP:DIP-14_W7.62mm_Socket" (id 2) (at 57.15 171.45 0)
       (effects (font (size 1.27 1.27)) hide)
     )
@@
     (property "Reference" "U401" (id 0) (at 108.9152 35.56 0))
     (property "Value" "74HC86" (id 1) (at 108.9152 38.1 0))
-    (property "Footprint" "" (id 2) (at 109.22 44.45 0)
+    (property "Footprint" "Package_DIP:DIP-14_W7.62mm_Socket" (id 2) (at 109.22 44.45 0)
       (effects (font (size 1.27 1.27)) hide)
     )
@@
     (property "Reference" "U402" (id 0) (at 108.9152 106.68 0))
     (property "Value" "74HC86" (id 1) (at 108.9152 109.22 0))
-    (property "Footprint" "" (id 2) (at 109.22 115.57 0)
+    (property "Footprint" "Package_DIP:DIP-14_W7.62mm_Socket" (id 2) (at 109.22 115.57 0)
       (effects (font (size 1.27 1.27)) hide)
     )
@@
     (property "Reference" "U402" (id 0) (at 108.9152 120.65 0))
     (property "Value" "74HC86" (id 1) (at 108.9152 123.19 0))
-    (property "Footprint" "" (id 2) (at 109.22 129.54 0)
+    (property "Footprint" "Package_DIP:DIP-14_W7.62mm_Socket" (id 2) (at 109.22 129.54 0)
       (effects (font (size 1.27 1.27)) hide)
     )
@@
     (property "Reference" "U402" (id 0) (at 108.9152 92.71 0))
     (property "Value" "74HC86" (id 1) (at 108.9152 95.25 0))
-    (property "Footprint" "" (id 2) (at 109.22 101.6 0)
+    (property "Footprint" "Package_DIP:DIP-14_W7.62mm_Socket" (id 2) (at 109.22 101.6 0)
       (effects (font (size 1.27 1.27)) hide)
     )
@@
     (property "Reference" "U401" (id 0) (at 108.9152 63.5 0))
     (property "Value" "74HC86" (id 1) (at 108.9152 66.04 0))
-    (property "Footprint" "" (id 2) (at 109.22 72.39 0)
+    (property "Footprint" "Package_DIP:DIP-14_W7.62mm_Socket" (id 2) (at 109.22 72.39 0)
       (effects (font (size 1.27 1.27)) hide)
     )
@@
       (effects (font (size 1.27 1.27)) (justify left))
     )
-    (property "Footprint" "" (id 2) (at 29.21 171.45 0)
+    (property "Footprint" "Package_DIP:DIP-14_W7.62mm_Socket" (id 2) (at 29.21 171.45 0)
       (effects (font (size 1.27 1.27)) hide)
     )
@@
     (property "Reference" "U401" (id 0) (at 108.9152 49.53 0))
     (property "Value" "74HC86" (id 1) (at 108.9152 52.07 0))
-    (property "Footprint" "" (id 2) (at 109.22 58.42 0)
-      (effects (font (size 1.27 1.27)) hide)
-    )
+    (property "Footprint" "Package_DIP:DIP-14_W7.62mm_Socket" (id 2) (at 109.22 58.42 0)
+      (effects (font (size 1.27 1.27)) hide)
+    )

Commit message: Doing some rethinking
Parts:
- removed U403: 74HCT541, Package_DIP:DIP-20_W7.62mm_Socket, symbol 74xx:74HCT541
- added U503: 74HC245, Package_SO:SOIC-20W_7.5x12.8mm_P1.27mm, symbol 74xx:74HC245
- renumbered U401 to U501, U402 to U502
Connections:
- net +5V: now also U503.20 (VCC)
- net GND: now also U503.10 (GND)
- net at U501.3: now also U503.2 (A0)
- net at U502.6: now also U503.7 (A5)
- net at U502.8: now also U503.9 (A7)
- net at U501.8: now also U503.5 (A3)
- net at U502.11: now also U503.8 (A6)
- net at U502.3: now also U503.6 (A4)
- net at U501.6: now also U503.3 (A1)
- net at U501.11: now also U503.4 (A2)

Commit message: Starting to think about decoding etc.
Parts:
- renumbered U501 to U601, U502 to U602, U503 to U603
Changed lines of the file:
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@@
   (symbol (lib_id "power:+5V") (at 215.9 25.4 0) (unit 1)
     (in_bom yes) (on_board yes) (fields_autoplaced)
-    (property "Reference" "#PWR0505" (id 0) (at 215.9 29.21 0)
+    (property "Reference" "#PWR0605" (id 0) (at 215.9 29.21 0)
       (effects (font (size 1.27 1.27)) hide)
     )
@@
   (symbol (lib_id "74xx:74HC86") (at 57.15 171.45 0) (unit 5)
     (in_bom yes) (on_board yes) (fields_autoplaced)
-    (property "Reference" "U502" (id 0) (at 63.5 170.1799 0)
+    (property "Reference" "U602" (id 0) (at 63.5 170.1799 0)
       (effects (font (size 1.27 1.27)) (justify left))
     )
@@
   (symbol (lib_id "power:GND") (at 215.9 88.9 0) (unit 1)
     (in_bom yes) (on_board yes) (fields_autoplaced)
-    (property "Reference" "#PWR0506" (id 0) (at 215.9 95.25 0)
+    (property "Reference" "#PWR0606" (id 0) (at 215.9 95.25 0)
       (effects (font (size 1.27 1.27)) hide)
     )
@@
   (symbol (lib_id "74xx:74HC86") (at 109.22 44.45 0) (unit 1)
     (in_bom yes) (on_board yes) (fields_autoplaced)
-    (property "Reference" "U501" (id 0) (at 108.9152 35.56 0))
+    (property "Reference" "U601" (id 0) (at 108.9152 35.56 0))
     (property "Value" "74HC86" (id 1) (at 108.9152 38.1 0))
     (property "Footprint" "Package_DIP:DIP-14_W7.62mm_Socket" (id 2) (at 109.22 44.45 0)
@@
   (symbol (lib_id "74xx:74HC86") (at 109.22 115.57 0) (unit 2)
     (in_bom yes) (on_board yes) (fields_autoplaced)
-    (property "Reference" "U502" (id 0) (at 108.9152 106.68 0))
+    (property "Reference" "U602" (id 0) (at 108.9152 106.68 0))
     (property "Value" "74HC86" (id 1) (at 108.9152 109.22 0))
     (property "Footprint" "Package_DIP:DIP-14_W7.62mm_Socket" (id 2) (at 109.22 115.57 0)
@@
   (symbol (lib_id "74xx:74HC86") (at 109.22 143.51 0) (unit 3)
     (in_bom yes) (on_board yes) (fields_autoplaced)
-    (property "Reference" "U502" (id 0) (at 108.9152 134.62 0))
+    (property "Reference" "U602" (id 0) (at 108.9152 134.62 0))
     (property "Value" "74HC86" (id 1) (at 108.9152 137.16 0))
     (property "Footprint" "Package_DIP:DIP-14_W7.62mm_Socket" (id 2) (at 109.22 143.51 0)
@@
   (symbol (lib_id "74xx:74HC86") (at 109.22 86.36 0) (unit 3)
     (in_bom yes) (on_board yes) (fields_autoplaced)
-    (property "Reference" "U501" (id 0) (at 108.9152 77.47 0))
+    (property "Reference" "U601" (id 0) (at 108.9152 77.47 0))
     (property "Value" "74HC86" (id 1) (at 108.9152 80.01 0))
     (property "Footprint" "Package_DIP:DIP-14_W7.62mm_Socket" (id 2) (at 109.22 86.36 0)
@@
   (symbol (lib_id "power:GND") (at 57.15 186.69 0) (unit 1)
     (in_bom yes) (on_board yes) (fields_autoplaced)
-    (property "Reference" "#PWR0504" (id 0) (at 57.15 193.04 0)
+    (property "Reference" "#PWR0604" (id 0) (at 57.15 193.04 0)
       (effects (font (size 1.27 1.27)) hide)
     )
@@
   (symbol (lib_id "power:GND") (at 29.21 186.69 0) (unit 1)
     (in_bom yes) (on_board yes) (fields_autoplaced)
-    (property "Reference" "#PWR0502" (id 0) (at 29.21 193.04 0)
+    (property "Reference" "#PWR0602" (id 0) (at 29.21 193.04 0)
       (effects (font (size 1.27 1.27)) hide)
     )
@@
   (symbol (lib_id "power:+5V") (at 29.21 156.21 0) (unit 1)
     (in_bom yes) (on_board yes) (fields_autoplaced)
-    (property "Reference" "#PWR0501" (id 0) (at 29.21 160.02 0)
+    (property "Reference" "#PWR0601" (id 0) (at 29.21 160.02 0)
       (effects (font (size 1.27 1.27)) hide)
     )
@@
   (symbol (lib_id "74xx:74HC86") (at 109.22 129.54 0) (unit 4)
     (in_bom yes) (on_board yes) (fields_autoplaced)
-    (property "Reference" "U502" (id 0) (at 108.9152 120.65 0))
+    (property "Reference" "U602" (id 0) (at 108.9152 120.65 0))
     (property "Value" "74HC86" (id 1) (at 108.9152 123.19 0))
     (property "Footprint" "Package_DIP:DIP-14_W7.62mm_Socket" (id 2) (at 109.22 129.54 0)
@@
   (symbol (lib_id "74xx:74HC86") (at 109.22 101.6 0) (unit 1)
     (in_bom yes) (on_board yes) (fields_autoplaced)
-    (property "Reference" "U502" (id 0) (at 108.9152 92.71 0))
+    (property "Reference" "U602" (id 0) (at 108.9152 92.71 0))
     (property "Value" "74HC86" (id 1) (at 108.9152 95.25 0))
     (property "Footprint" "Package_DIP:DIP-14_W7.62mm_Socket" (id 2) (at 109.22 101.6 0)
@@
   (symbol (lib_id "74xx:74HC86") (at 109.22 72.39 0) (unit 4)
     (in_bom yes) (on_board yes) (fields_autoplaced)
-    (property "Reference" "U501" (id 0) (at 108.9152 63.5 0))
+    (property "Reference" "U601" (id 0) (at 108.9152 63.5 0))
     (property "Value" "74HC86" (id 1) (at 108.9152 66.04 0))
     (property "Footprint" "Package_DIP:DIP-14_W7.62mm_Socket" (id 2) (at 109.22 72.39 0)
@@
   (symbol (lib_id "74xx:74HC86") (at 29.21 171.45 0) (unit 5)
     (in_bom yes) (on_board yes) (fields_autoplaced)
-    (property "Reference" "U501" (id 0) (at 35.56 170.1799 0)
+    (property "Reference" "U601" (id 0) (at 35.56 170.1799 0)
       (effects (font (size 1.27 1.27)) (justify left))
     )
@@
   (symbol (lib_id "74xx:74HC86") (at 109.22 58.42 0) (unit 2)
     (in_bom yes) (on_board yes) (fields_autoplaced)
-    (property "Reference" "U501" (id 0) (at 108.9152 49.53 0))
+    (property "Reference" "U601" (id 0) (at 108.9152 49.53 0))
     (property "Value" "74HC86" (id 1) (at 108.9152 52.07 0))
     (property "Footprint" "Package_DIP:DIP-14_W7.62mm_Socket" (id 2) (at 109.22 58.42 0)
@@
   (symbol (lib_id "74xx:74HC245") (at 215.9 57.15 0) (unit 1)
     (in_bom yes) (on_board yes) (fields_autoplaced)
-    (property "Reference" "U503" (id 0) (at 217.9194 36.83 0)
+    (property "Reference" "U603" (id 0) (at 217.9194 36.83 0)
       (effects (font (size 1.27 1.27)) (justify left))
     )
@@
   (symbol (lib_id "power:+5V") (at 57.15 156.21 0) (unit 1)
     (in_bom yes) (on_board yes) (fields_autoplaced)
-    (property "Reference" "#PWR0503" (id 0) (at 57.15 160.02 0)
-      (effects (font (size 1.27 1.27)) hide)
-    )
+    (property "Reference" "#PWR0603" (id 0) (at 57.15 160.02 0)
+      (effects (font (size 1.27 1.27)) hide)
+    )
