File: pcbs/Tester/Tester.kicad_pcb (KiCad board)
At the start: 2 copper layers, 88.9 x 139.7 mm, 110 parts, among them J201 Raspberry_Pi_2_3, J202 Conn_01x04, J301 Conn_02x20_Odd_Even, J401 Conn_02x20_Odd_Even, U201 SN74LVC4245APWR, U202 SN74LVC4245APWR, U203 SN74LVC4245APWR, U301 74HC595, U302 74HC595, U303 74HC595, U304 74HC595, U305 74HC595, U401 74HC165, U402 74HC165, U403 74HC165, U404 74HC165, U405 74HC165

Commit message: Finish routing
Parts:
- added J203: Conn_01x10, Connector_PinHeader_2.54mm:PinHeader_1x10_P2.54mm_Vertical, F.Cu at (114.3, 101.6)
- moved J201 2.54 mm to (96.5, 68.6)
Connections:
- J201 pad 10: unconnected-(J201-Pad10) -> /Pi Input/GPIO15
- J201 pad 11: /Pi Input/~{SPI1_{LOAD}} -> unconnected-(J201-Pad11)
- J201 pad 13: unconnected-(J201-Pad13) -> /Pi Input/~{SPI0_{OE2}}
- J201 pad 15: unconnected-(J201-Pad15) -> /Pi Input/~{SPI0_{OE1}}
- J201 pad 18: unconnected-(J201-Pad18) -> /Pi Input/GPIO24
- J201 pad 22: unconnected-(J201-Pad22) -> /Pi Input/GPIO25
- J201 pad 27: unconnected-(J201-Pad27) -> /Pi Input/GPIO0
- J201 pad 28: unconnected-(J201-Pad28) -> /Pi Input/GPIO1
- J201 pad 29: unconnected-(J201-Pad29) -> /Pi Input/GPIO5
- J201 pad 3: unconnected-(J201-Pad3) -> /Pi Input/~{SPI0_{OE5}}
- J201 pad 31: unconnected-(J201-Pad31) -> /Pi Input/GPIO6
- J201 pad 32: unconnected-(J201-Pad32) -> /Pi Input/GPIO12
- J201 pad 33: unconnected-(J201-Pad33) -> /Pi Input/GPIO13
- J201 pad 37: unconnected-(J201-Pad37) -> /Pi Input/~{SPI1_{LOAD}}
- J201 pad 5: unconnected-(J201-Pad5) -> /Pi Input/~{SPI0_{OE4}}
- J201 pad 7: unconnected-(J201-Pad7) -> /Pi Input/~{SPI0_{OE3}}
- J201 pad 8: unconnected-(J201-Pad8) -> /Pi Input/GPIO14
- U202 pad 14: unconnected-(U202-Pad14) -> GND
- U202 pad 15: unconnected-(U202-Pad15) -> GND
- U202 pad 16: unconnected-(U202-Pad16) -> GND
- U202 pad 17: unconnected-(U202-Pad17) -> GND
- U202 pad 19: unconnected-(U202-Pad19) -> GND
- U202 pad 20: unconnected-(U202-Pad20) -> GND
- U202 pad 21: unconnected-(U202-Pad21) -> GND
- U203 pad 14: unconnected-(U203-Pad14) -> GND
- U203 pad 18: unconnected-(U203-Pad18) -> GND
- U203 pad 19: unconnected-(U203-Pad19) -> GND
- U203 pad 20: unconnected-(U203-Pad20) -> GND
- U203 pad 21: unconnected-(U203-Pad21) -> GND
Routing:
- net +3V3: track 0.65 -> 132.3 mm, vias 0 -> 2
- net /Pi Input/SPI0_{CLK}: track 0.00 -> 65.0 mm
- net GND: track 0.00 -> 63.1 mm, vias 0 -> 8
- net /Pi Input/SPI0_{COPI}: track 0.00 -> 57.3 mm
- net /Pi Input/~{SPI0_{OE1}}: track 0.00 -> 50.7 mm
- net /Pi Input/~{SPI0_{SELECT}}: track 0.00 -> 50.1 mm, vias 0 -> 2
- net /Pi Input/SPI1_{CIPO}: track 0.00 -> 49.9 mm
- net /Pi Input/GPIO13: track 0.00 -> 46.8 mm
- net /Pi Input/~{SPI1_{SELECT}}: track 0.00 -> 46.8 mm, vias 0 -> 1
- net /Pi Input/~{SPI0_{OE2}}: track 0.00 -> 46.7 mm
- net /Pi Input/GPIO12: track 0.00 -> 38.3 mm
- net /Pi Input/~{SPI0_{OE3}}: track 0.00 -> 37.6 mm
- net /Pi Input/GPIO6: track 0.00 -> 37.1 mm
- net /Pi Input/GPIO5: track 0.00 -> 33.8 mm
- net /Pi Input/~{SPI0_{OE4}}: track 0.00 -> 33.6 mm
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- added copper zone on F.Cu, net GND
- removed copper zone on F.Cu, net /In Registers/In_{3}
Other:
- board size 88.9 x 139.7 mm -> 73.7 x 129.5 mm
- board text added: "+5V"
- board text added: "0"
- board text added: "1"
- board text added: "12"
- board text added: "13"
- board text added: "16"
- board text added: "17"
- board text added: "20"
- board text added: "21"
- board text added: "24"
- board text added: "25"
- board text added: "28"
- board text added: "29"
- board text added: "32"
- board text added: "33"
- board text added: "36"
- board text added: "37"
- board text added: "3V3"
- board text added: "4"
- board text added: "5"
- board text added: "8"
- board text added: "9"
- board text added: "GND"
- board text added: "GPIO0"
- board text added: "GPIO1"
- board text added: "GPIO12"
- board text added: "GPIO13"
- board text added: "GPIO14"
- board text added: "GPIO15"
- board text added: "GPIO24"
- board text added: "GPIO25"
- board text added: "GPIO5"
- board text added: "GPIO6"
- board text added: "In"
- board text added: "JLCJLCJLCJLC"
- board text added: "Out"
- board text added: "Pi"
- board text added: "RGE2023"
- board text added: "Tester"
