File: pcbs/Tester/Tester.kicad_pcb (KiCad board)
At the start: 2 copper layers, 73.7 x 129.5 mm, 111 parts, among them J201 Raspberry_Pi_2_3, J202 Conn_01x04, J203 Conn_01x10, J301 Conn_02x20_Odd_Even, J401 Conn_02x20_Odd_Even, U201 SN74LVC4245APWR, U202 SN74LVC4245APWR, U203 SN74LVC4245APWR, U301 74HC595, U302 74HC595, U303 74HC595, U304 74HC595, U305 74HC595, U401 74HC165, U402 74HC165, U403 74HC165, U404 74HC165, U405 74HC165

Commit message: Fix U202
Connections:
- U202 pad 10: unconnected-(U202-Pad10) -> GND
- U202 pad 14: GND -> unconnected-(U202-Pad14)
- U202 pad 15: GND -> unconnected-(U202-Pad15)
- U202 pad 16: GND -> unconnected-(U202-Pad16)
- U202 pad 17: GND -> unconnected-(U202-Pad17)
- U202 pad 19: GND -> unconnected-(U202-Pad19)
- U202 pad 20: GND -> unconnected-(U202-Pad20)
- U202 pad 21: GND -> unconnected-(U202-Pad21)
- U202 pad 3: unconnected-(U202-Pad3) -> GND
- U202 pad 4: unconnected-(U202-Pad4) -> GND
- U202 pad 5: unconnected-(U202-Pad5) -> GND
- U202 pad 7: unconnected-(U202-Pad7) -> GND
- U202 pad 8: unconnected-(U202-Pad8) -> GND
- U202 pad 9: unconnected-(U202-Pad9) -> GND
Other:
- board text added: "r${REVISION}"
Changed lines of the file:
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@@
   )
   (paper "A4")
+  (title_block
+    (rev "2")
+  )
   (layers
     (0 "F.Cu" signal)
@@
   (net 126 "/In Registers/In_{36}")
   (net 127 "/In Registers/In_{38}")
-  (net 128 "unconnected-(U202-Pad3)")
-  (net 129 "unconnected-(U202-Pad4)")
-  (net 130 "unconnected-(U202-Pad5)")
-  (net 131 "unconnected-(U202-Pad7)")
-  (net 132 "unconnected-(U202-Pad8)")
-  (net 133 "unconnected-(U202-Pad9)")
-  (net 134 "unconnected-(U202-Pad10)")
+  (net 128 "unconnected-(U202-Pad14)")
+  (net 129 "unconnected-(U202-Pad15)")
+  (net 130 "unconnected-(U202-Pad16)")
+  (net 131 "unconnected-(U202-Pad17)")
+  (net 132 "unconnected-(U202-Pad19)")
+  (net 133 "unconnected-(U202-Pad20)")
+  (net 134 "unconnected-(U202-Pad21)")
   (net 135 "/Pi Input/~{SPI0_{OE2}}")
   (net 136 "/Pi Input/~{SPI0_{OE3}}")
@@
       (net 2 "+5V") (pinfunction "DIR") (pintype "input"))
     (pad "3" smd roundrect (at -2.8625 -2.275 180) (size 1.475 0.4) (layers "F.Cu" "F.Paste" "F.Mask") (roundrect_rratio 0.25)
-      (net 128 "unconnected-(U202-Pad3)") (pinfunction "A1") (pintype "bidirectional+no_connect"))
+      (net 3 "GND") (pinfunction "A1") (pintype "bidirectional"))
     (pad "4" smd roundrect (at -2.8625 -1.625 180) (size 1.475 0.4) (layers "F.Cu" "F.Paste" "F.Mask") (roundrect_rratio 0.25)
-      (net 129 "unconnected-(U202-Pad4)") (pinfunction "A2") (pintype "bidirectional+no_connect"))
+      (net 3 "GND") (pinfunction "A2") (pintype "bidirectional"))
     (pad "5" smd roundrect (at -2.8625 -0.975 180) (size 1.475 0.4) (layers "F.Cu" "F.Paste" "F.Mask") (roundrect_rratio 0.25)
-      (net 130 "unconnected-(U202-Pad5)") (pinfunction "A3") (pintype "bidirectional+no_connect"))
+      (net 3 "GND") (pinfunction "A3") (pintype "bidirectional"))
     (pad "6" smd roundrect (at -2.8625 -0.325 180) (size 1.475 0.4) (layers "F.Cu" "F.Paste" "F.Mask") (roundrect_rratio 0.25)
       (net 39 "/In Registers/IN_{DATA}") (pinfunction "A4") (pintype "bidirectional"))
     (pad "7" smd roundrect (at -2.8625 0.325 180) (size 1.475 0.4) (layers "F.Cu" "F.Paste" "F.Mask") (roundrect_rratio 0.25)
-      (net 131 "unconnected-(U202-Pad7)") (pinfunction "A5") (pintype "bidirectional+no_connect"))
+      (net 3 "GND") (pinfunction "A5") (pintype "bidirectional"))
     (pad "8" smd roundrect (at -2.8625 0.975 180) (size 1.475 0.4) (layers "F.Cu" "F.Paste" "F.Mask") (roundrect_rratio 0.25)
-      (net 132 "unconnected-(U202-Pad8)") (pinfunction "A6") (pintype "bidirectional+no_connect"))
+      (net 3 "GND") (pinfunction "A6") (pintype "bidirectional"))
     (pad "9" smd roundrect (at -2.8625 1.625 180) (size 1.475 0.4) (layers "F.Cu" "F.Paste" "F.Mask") (roundrect_rratio 0.25)
-      (net 133 "unconnected-(U202-Pad9)") (pinfunction "A7") (pintype "bidirectional+no_connect"))
+      (net 3 "GND") (pinfunction "A7") (pintype "bidirectional"))
     (pad "10" smd roundrect (at -2.8625 2.275 180) (size 1.475 0.4) (layers "F.Cu" "F.Paste" "F.Mask") (roundrect_rratio 0.25)
-      (net 134 "unconnected-(U202-Pad10)") (pinfunction "A8") (pintype "bidirectional+no_connect"))
+      (net 3 "GND") (pinfunction "A8") (pintype "bidirectional"))
     (pad "11" smd roundrect (at -2.8625 2.925 180) (size 1.475 0.4) (layers "F.Cu" "F.Paste" "F.Mask") (roundrect_rratio 0.25)
       (net 3 "GND") (pinfunction "GND") (pintype "power_in"))
@@
       (net 3 "GND") (pinfunction "GND") (pintype "power_in"))
     (pad "14" smd roundrect (at 2.8625 2.925 180) (size 1.475 0.4) (layers "F.Cu" "F.Paste" "F.Mask") (roundrect_rratio 0.25)
-      (net 3 "GND") (pinfunction "B8") (pintype "bidirectional"))
+      (net 128 "unconnected-(U202-Pad14)") (pinfunction "B8") (pintype "bidirectional+no_connect"))
     (pad "15" smd roundrect (at 2.8625 2.275 180) (size 1.475 0.4) (layers "F.Cu" "F.Paste" "F.Mask") (roundrect_rratio 0.25)
-      (net 3 "GND") (pinfunction "B7") (pintype "bidirectional"))
+      (net 129 "unconnected-(U202-Pad15)") (pinfunction "B7") (pintype "bidirectional+no_connect"))
     (pad "16" smd roundrect (at 2.8625 1.625 180) (size 1.475 0.4) (layers "F.Cu" "F.Paste" "F.Mask") (roundrect_rratio 0.25)
-      (net 3 "GND") (pinfunction "B6") (pintype "bidirectional"))
+      (net 130 "unconnected-(U202-Pad16)") (pinfunction "B6") (pintype "bidirectional+no_connect"))
     (pad "17" smd roundrect (at 2.8625 0.975 180) (size 1.475 0.4) (layers "F.Cu" "F.Paste" "F.Mask") (roundrect_rratio 0.25)
-      (net 3 "GND") (pinfunction "B5") (pintype "bidirectional"))
+      (net 131 "unconnected-(U202-Pad17)") (pinfunction "B5") (pintype "bidirectional+no_connect"))
     (pad "18" smd roundrect (at 2.8625 0.325 180) (size 1.475 0.4) (layers "F.Cu" "F.Paste" "F.Mask") (roundrect_rratio 0.25)
       (net 12 "/Pi Input/SPI1_{CIPO}") (pinfunction "B4") (pintype "bidirectional"))
     (pad "19" smd roundrect (at 2.8625 -0.325 180) (size 1.475 0.4) (layers "F.Cu" "F.Paste" "F.Mask") (roundrect_rratio 0.25)
-      (net 3 "GND") (pinfunction "B3") (pintype "bidirectional"))
+      (net 132 "unconnected-(U202-Pad19)") (pinfunction "B3") (pintype "bidirectional+no_connect"))
     (pad "20" smd roundrect (at 2.8625 -0.975 180) (size 1.475 0.4) (layers "F.Cu" "F.Paste" "F.Mask") (roundrect_rratio 0.25)
-      (net 3 "GND") (pinfunction "B2") (pintype "bidirectional"))
+      (net 133 "unconnected-(U202-Pad20)") (pinfunction "B2") (pintype "bidirectional+no_connect"))
     (pad "21" smd roundrect (at 2.8625 -1.625 180) (size 1.475 0.4) (layers "F.Cu" "F.Paste" "F.Mask") (roundrect_rratio 0.25)
-      (net 3 "GND") (pinfunction "B1") (pintype "bidirectional"))
+      (net 134 "unconnected-(U202-Pad21)") (pinfunction "B1") (pintype "bidirectional+no_connect"))
     (pad "22" smd roundrect (at 2.8625 -2.275 180) (size 1.475 0.4) (layers "F.Cu" "F.Paste" "F.Mask") (roundrect_rratio 0.25)
       (net 3 "GND") (pinfunction "~{OE}") (pintype "input"))
@@
     (effects (font (size 1 1) (thickness 0.15)) (justify right))
   )
+  (gr_text "r${REVISION}" (at 100.33 34.29 90) (layer "F.SilkS")
+    (effects (font (size 1.6256 1.6256) (thickness 0.2032)) (justify left))
+  )
   (gr_text "GND" (at 101.6 73.66) (layer "F.SilkS")
