File: pcbs/Tester/pi_input.kicad_sch (KiCad schematic)
At the start: 8 parts, among them J201 Raspberry_Pi_2_3, J202 Conn_01x04, U201 SN74LVC4245APWR, U202 SN74LVC4245APWR, U203 SN74LVC4245APWR

Commit message: Finish routing
Parts:
- added J203: Conn_01x10, symbol Connector_Generic:Conn_01x10
- J202: footprint (none) -> Connector_PinHeader_2.54mm:PinHeader_1x04_P2.54mm_Vertical
Connections:
- net GND: now also U202.14 (B8), U202.15 (B7), U202.16 (B6), U202.17 (B5), U202.19 (B3), U202.20 (B2), U202.21 (B1), U203.14 (B8), U203.18 (B4), U203.19 (B3), U203.20 (B2), U203.21 (B1)
- net ~{SPI0_{OE1}}: now also J201.15 (GPIO22)
- net ~{SPI0_{OE2}}: now also J201.13 (GPIO27)
- net ~{SPI0_{OE3}}: now also J201.7 (GCLK0/GPIO4)
- net ~{SPI0_{OE4}}: now also J201.5 (SCL/GPIO3)
- net ~{SPI0_{OE5}}: now also J201.3 (SDA/GPIO2)
- net ~{SPI1_{LOAD}}: now also J201.37 (GPIO26); no longer J201.11 (GPIO17)
- net GPIO15: now reaches J201.10 (GPIO15/RXD)
- net GPIO15: now also J203.8 (Pin_8)
- net GPIO24: now reaches J201.18 (GPIO24)
- net GPIO24: now also J203.9 (Pin_9)
- net GPIO25: now reaches J201.22 (GPIO25)
- net GPIO25: now also J203.10 (Pin_10)
- net GPIO0: now reaches J201.27 (ID_SD/GPIO0)
- net GPIO0: now also J203.1 (Pin_1)
- net GPIO1: now reaches J201.28 (ID_SC/GPIO1)
- net GPIO1: now also J203.2 (Pin_2)
- net GPIO5: now reaches J201.29 (GCLK1/GPIO5)
- net GPIO5: now also J203.3 (Pin_3)
- net GPIO6: now reaches J201.31 (GCLK2/GPIO6)
- net GPIO6: now also J203.4 (Pin_4)
- net GPIO12: now reaches J201.32 (PWM0/GPIO12)
- net GPIO12: now also J203.5 (Pin_5)
- net GPIO13: now reaches J201.33 (PWM1/GPIO13)
- net GPIO13: now also J203.6 (Pin_6)
- net GPIO14: now reaches J201.8 (GPIO14/TXD)
- net GPIO14: now also J203.7 (Pin_7)
- no-connect marks 2 -> 18

Commit message: Fix U202
Parts:
- J203: footprint (none) -> Connector_PinHeader_2.54mm:PinHeader_1x10_P2.54mm_Vertical
Connections:
- net GND: now also U202.10 (A8), U202.3 (A1), U202.4 (A2), U202.5 (A3), U202.7 (A5), U202.8 (A6), U202.9 (A7); no longer U202.14 (B8), U202.15 (B7), U202.16 (B6), U202.17 (B5), U202.19 (B3), U202.20 (B2), U202.21 (B1)
Changed lines of the file:
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@@
   (junction (at 150.495 137.795) (diameter 0) (color 0 0 0 0)
   )
-  (junction (at 183.515 128.905) (diameter 0) (color 0 0 0 0)
+  (junction (at 149.225 128.905) (diameter 0) (color 0 0 0 0)
   )
   (junction (at 71.12 130.81) (diameter 0) (color 0 0 0 0)
@@
   (junction (at 74.93 130.81) (diameter 0) (color 0 0 0 0)
   )
-  (junction (at 183.515 113.665) (diameter 0) (color 0 0 0 0)
+  (junction (at 149.225 113.665) (diameter 0) (color 0 0 0 0)
   )
   (junction (at 76.2 130.81) (diameter 0) (color 0 0 0 0)
   )
-  (junction (at 180.975 113.665) (diameter 0) (color 0 0 0 0)
-  )
-  (junction (at 181.61 128.905) (diameter 0) (color 0 0 0 0)
-  )
-  (junction (at 179.705 128.905) (diameter 0) (color 0 0 0 0)
+  (junction (at 151.765 113.665) (diameter 0) (color 0 0 0 0)
+  )
+  (junction (at 151.13 128.905) (diameter 0) (color 0 0 0 0)
+  )
+  (junction (at 153.035 128.905) (diameter 0) (color 0 0 0 0)
   )
   (junction (at 229.87 128.27) (diameter 0) (color 0 0 0 0)
@@
   (junction (at 179.705 102.235) (diameter 0) (color 0 0 0 0)
   )
-  (no_connect (at 154.94 128.905))
   (no_connect (at 96.52 100.33))
-  (no_connect (at 154.94 113.665))
-  (no_connect (at 154.94 121.285))
-  (no_connect (at 154.94 123.825))
+  (no_connect (at 177.8 116.205))
+  (no_connect (at 177.8 121.285))
+  (no_connect (at 177.8 123.825))
+  (no_connect (at 177.8 113.665))
   (no_connect (at 55.88 100.33))
   (no_connect (at 234.315 50.8))
-  (no_connect (at 154.94 126.365))
   (no_connect (at 55.88 77.47))
   (no_connect (at 234.315 53.34))
-  (no_connect (at 154.94 111.125))
   (no_connect (at 55.88 80.01))
   (no_connect (at 234.315 48.26))
@@
   (no_connect (at 234.315 55.88))
   (no_connect (at 234.315 66.04))
-  (no_connect (at 154.94 116.205))
+  (no_connect (at 177.8 111.125))
   (no_connect (at 96.52 95.25))
+  (no_connect (at 177.8 128.905))
+  (no_connect (at 177.8 126.365))
   (bus_entry (at 144.145 53.975) (size 2.54 -2.54)
     (stroke (width 0) (type default) (color 0 0 0 0))
@@
     (stroke (width 0) (type default) (color 0 0 0 0))
   )
-  (wire (pts (xy 180.975 111.125) (xy 180.975 113.665))
+  (wire (pts (xy 151.765 111.125) (xy 151.765 113.665))
     (stroke (width 0) (type default) (color 0 0 0 0))
   )
@@
     (stroke (width 0) (type default) (color 0 0 0 0))
   )
-  (wire (pts (xy 177.8 113.665) (xy 180.975 113.665))
+  (wire (pts (xy 154.94 113.665) (xy 151.765 113.665))
     (stroke (width 0) (type default) (color 0 0 0 0))
   )
@@
     (stroke (width 0) (type default) (color 0 0 0 0))
   )
-  (wire (pts (xy 177.8 121.285) (xy 183.515 121.285))
+  (wire (pts (xy 154.94 121.285) (xy 149.225 121.285))
     (stroke (width 0) (type default) (color 0 0 0 0))
   )
@@
     (stroke (width 0) (type default) (color 0 0 0 0))
   )
-  (wire (pts (xy 180.975 113.665) (xy 183.515 113.665))
-    (stroke (width 0) (type default) (color 0 0 0 0))
-  )
-  (wire (pts (xy 181.61 123.825) (xy 181.61 128.905))
+  (wire (pts (xy 151.765 113.665) (xy 149.225 113.665))
+    (stroke (width 0) (type default) (color 0 0 0 0))
+  )
+  (wire (pts (xy 151.13 123.825) (xy 151.13 128.905))
     (stroke (width 0) (type default) (color 0 0 0 0))
   )
@@
     (stroke (width 0) (type default) (color 0 0 0 0))
   )
-  (wire (pts (xy 181.61 128.905) (xy 183.515 128.905))
+  (wire (pts (xy 151.13 128.905) (xy 149.225 128.905))
     (stroke (width 0) (type default) (color 0 0 0 0))
   )
@@
     (stroke (width 0) (type default) (color 0 0 0 0))
   )
-  (wire (pts (xy 183.515 128.905) (xy 186.69 128.905))
+  (wire (pts (xy 149.225 128.905) (xy 146.05 128.905))
     (stroke (width 0) (type default) (color 0 0 0 0))
   )
@@
     (stroke (width 0) (type default) (color 0 0 0 0))
   )
-  (wire (pts (xy 183.515 116.205) (xy 183.515 113.665))
+  (wire (pts (xy 149.225 116.205) (xy 149.225 113.665))
     (stroke (width 0) (type default) (color 0 0 0 0))
   )
@@
     (stroke (width 0) (type default) (color 0 0 0 0))
   )
-  (wire (pts (xy 179.705 126.365) (xy 179.705 128.905))
+  (wire (pts (xy 153.035 126.365) (xy 153.035 128.905))
     (stroke (width 0) (type default) (color 0 0 0 0))
   )
@@
     (stroke (width 0) (type default) (color 0 0 0 0))
   )
-  (wire (pts (xy 183.515 121.285) (xy 183.515 128.905))
+  (wire (pts (xy 149.225 121.285) (xy 149.225 128.905))
     (stroke (width 0) (type default) (color 0 0 0 0))
   )
@@
     (stroke (width 0) (type default) (color 0 0 0 0))
   )
-  (wire (pts (xy 177.8 123.825) (xy 181.61 123.825))
+  (wire (pts (xy 154.94 123.825) (xy 151.13 123.825))
     (stroke (width 0) (type default) (color 0 0 0 0))
   )
@@
     (stroke (width 0) (type default) (color 0 0 0 0))
   )
-  (wire (pts (xy 179.705 128.905) (xy 181.61 128.905))
-    (stroke (width 0) (type default) (color 0 0 0 0))
-  )
-  (wire (pts (xy 183.515 113.665) (xy 186.69 113.665))
+  (wire (pts (xy 153.035 128.905) (xy 151.13 128.905))
+    (stroke (width 0) (type default) (color 0 0 0 0))
+  )
+  (wire (pts (xy 149.225 113.665) (xy 146.05 113.665))
     (stroke (width 0) (type default) (color 0 0 0 0))
   )
@@
     (stroke (width 0) (type default) (color 0 0 0 0))
   )
-  (wire (pts (xy 177.8 116.205) (xy 183.515 116.205))
+  (wire (pts (xy 154.94 116.205) (xy 149.225 116.205))
     (stroke (width 0) (type default) (color 0 0 0 0))
   )
@@
     (stroke (width 0) (type default) (color 0 0 0 0))
   )
-  (wire (pts (xy 177.8 111.125) (xy 180.975 111.125))
+  (wire (pts (xy 154.94 111.125) (xy 151.765 111.125))
     (stroke (width 0) (type default) (color 0 0 0 0))
   )
@@
     (stroke (width 0) (type default) (color 0 0 0 0))
   )
-  (wire (pts (xy 177.8 128.905) (xy 179.705 128.905))
+  (wire (pts (xy 154.94 128.905) (xy 153.035 128.905))
     (stroke (width 0) (type default) (color 0 0 0 0))
   )
@@
     (stroke (width 0) (type default) (color 0 0 0 0))
   )
-  (wire (pts (xy 177.8 126.365) (xy 179.705 126.365))
+  (wire (pts (xy 154.94 126.365) (xy 153.035 126.365))
     (stroke (width 0) (type default) (color 0 0 0 0))
   )
@@
     (pin "1")
   )
-  (symbol (lib_id "power:GND") (at 186.69 113.665 90) (unit 1)
-    (in_bom yes) (on_board yes) (fields_autoplaced)
-    (property "Reference" "#PWR0223" (id 0) (at 193.04 113.665 0)
-      (effects (font (size 1.27 1.27)) hide)
-    )
-    (property "Value" "GND" (id 1) (at 190.5 113.6649 90)
+  (symbol (lib_id "power:GND") (at 146.05 113.665 270) (mirror x) (unit 1)
+    (in_bom yes) (on_board yes) (fields_autoplaced)
+    (property "Reference" "#PWR0223" (id 0) (at 139.7 113.665 0)
+      (effects (font (size 1.27 1.27)) hide)
+    )
+    (property "Value" "GND" (id 1) (at 142.24 113.6649 90)
       (effects (font (size 1.27 1.27)) (justify right))
     )
-    (property "Footprint" "" (id 2) (at 186.69 113.665 0)
-      (effects (font (size 1.27 1.27)) hide)
-    )
-    (property "Datasheet" "" (id 3) (at 186.69 113.665 0)
+    (property "Footprint" "" (id 2) (at 146.05 113.665 0)
+      (effects (font (size 1.27 1.27)) hide)
+    )
+    (property "Datasheet" "" (id 3) (at 146.05 113.665 0)
       (effects (font (size 1.27 1.27)) hide)
     )
@@
     (pin "4")
   )
-  (symbol (lib_id "power:GND") (at 186.69 128.905 90) (unit 1)
-    (in_bom yes) (on_board yes) (fields_autoplaced)
-    (property "Reference" "#PWR0224" (id 0) (at 193.04 128.905 0)
-      (effects (font (size 1.27 1.27)) hide)
-    )
-    (property "Value" "GND" (id 1) (at 190.5 128.9049 90)
+  (symbol (lib_id "power:GND") (at 146.05 128.905 270) (mirror x) (unit 1)
+    (in_bom yes) (on_board yes) (fields_autoplaced)
+    (property "Reference" "#PWR0224" (id 0) (at 139.7 128.905 0)
+      (effects (font (size 1.27 1.27)) hide)
+    )
+    (property "Value" "GND" (id 1) (at 142.24 128.9049 90)
       (effects (font (size 1.27 1.27)) (justify right))
     )
-    (property "Footprint" "" (id 2) (at 186.69 128.905 0)
-      (effects (font (size 1.27 1.27)) hide)
-    )
-    (property "Datasheet" "" (id 3) (at 186.69 128.905 0)
+    (property "Footprint" "" (id 2) (at 146.05 128.905 0)
+      (effects (font (size 1.27 1.27)) hide)
+    )
+    (property "Datasheet" "" (id 3) (at 146.05 128.905 0)
       (effects (font (size 1.27 1.27)) hide)
     )
@@
       (effects (font (size 1.27 1.27)) (justify left))
     )
-    (property "Footprint" "" (id 2) (at 140.335 166.37 0)
-      (effects (font (size 1.27 1.27)) hide)
-    )
+    (property "Footprint" "Connector_PinHeader_2.54mm:PinHeader_1x10_P2.54mm_Vertical" (id 2) (at 140.335 166.37 0)
+      (effects (font (size 1.27 1.27)) hide)
+    )
