File: pcbs/ALU Connector/ALU Connector.kicad_pcb (KiCad board)
At the start: 2 copper layers, 58.4 x 134.6 mm, 55 parts, among them J101 Conn_02x20_Odd_Even, J102 Conn_02x20_Odd_Even, J103 Conn_01x04, J104 Conn_02x20_Odd_Even, J105 Conn_01x10, J106 Conn_01x10, J107 Conn_01x10

Commit message: Finished draft
Parts:
- added D125: Yellow, LED_SMD:LED_0603_1608Metric, F.Cu at (76.2, 88.9)
- added D126: Yellow, LED_SMD:LED_0603_1608Metric, F.Cu at (76.2, 91.4)
- added D127: Yellow, LED_SMD:LED_0603_1608Metric, F.Cu at (76.2, 94.0)
- added D128: Yellow, LED_SMD:LED_0603_1608Metric, F.Cu at (76.2, 96.5)
- added D129: Yellow, LED_SMD:LED_0603_1608Metric, F.Cu at (76.2, 99.1)
- added D130: Yellow, LED_SMD:LED_0603_1608Metric, F.Cu at (76.2, 101.6)
- added D131: Yellow, LED_SMD:LED_0603_1608Metric, F.Cu at (76.2, 104.1)
- added D132: Yellow, LED_SMD:LED_0603_1608Metric, F.Cu at (76.2, 106.7)
- added D133: Yellow, LED_SMD:LED_0603_1608Metric, F.Cu at (76.2, 109.2)
- added R125: 4k7, Resistor_SMD:R_0603_1608Metric, F.Cu at (72.4, 88.9)
- added R126: 4k7, Resistor_SMD:R_0603_1608Metric, F.Cu at (72.4, 91.4)
- added R127: 4k7, Resistor_SMD:R_0603_1608Metric, F.Cu at (72.4, 94.0)
- added R128: 4k7, Resistor_SMD:R_0603_1608Metric, F.Cu at (72.4, 96.5)
- added R129: 4k7, Resistor_SMD:R_0603_1608Metric, F.Cu at (72.4, 99.1)
- added R130: 4k7, Resistor_SMD:R_0603_1608Metric, F.Cu at (72.4, 101.6)
- added R131: 4k7, Resistor_SMD:R_0603_1608Metric, F.Cu at (72.4, 104.1)
- added R132: 4k7, Resistor_SMD:R_0603_1608Metric, F.Cu at (72.4, 106.7)
- added R133: 4k7, Resistor_SMD:R_0603_1608Metric, F.Cu at (72.4, 109.2)
Connections:
- J102 pad 21: unconnected-(J102-Pad21) -> /In_{18}
- J102 pad 22: unconnected-(J102-Pad22) -> /In_{19}
- J102 pad 23: unconnected-(J102-Pad23) -> /In_{16}
- J102 pad 24: unconnected-(J102-Pad24) -> /In_{17}
- J102 pad 25: unconnected-(J102-Pad25) -> /In_{15}
- J102 pad 26: unconnected-(J102-Pad26) -> /In_{14}
- J102 pad 27: unconnected-(J102-Pad27) -> /In_{13}
- J102 pad 28: unconnected-(J102-Pad28) -> /In_{12}
- J102 pad 29: unconnected-(J102-Pad29) -> /In_{11}
- J102 pad 30: unconnected-(J102-Pad30) -> /In_{10}
- J102 pad 31: unconnected-(J102-Pad31) -> /In_{28}
- J102 pad 32: unconnected-(J102-Pad32) -> /In_{29}
- J102 pad 33: unconnected-(J102-Pad33) -> /In_{26}
- J102 pad 34: unconnected-(J102-Pad34) -> /In_{27}
- J102 pad 35: unconnected-(J102-Pad35) -> /In_{25}
- J102 pad 36: unconnected-(J102-Pad36) -> /In_{24}
- J102 pad 37: unconnected-(J102-Pad37) -> /In_{23}
- J102 pad 38: unconnected-(J102-Pad38) -> /In_{22}
- J102 pad 39: unconnected-(J102-Pad39) -> /In_{21}
- J102 pad 40: unconnected-(J102-Pad40) -> /In_{20}
- J106 pad 1: unconnected-(J106-Pad1) -> /In_{10}
- J106 pad 10: unconnected-(J106-Pad10) -> /In_{19}
- J106 pad 2: unconnected-(J106-Pad2) -> /In_{11}
- J106 pad 3: unconnected-(J106-Pad3) -> /In_{12}
- J106 pad 4: unconnected-(J106-Pad4) -> /In_{13}
- J106 pad 5: unconnected-(J106-Pad5) -> /In_{14}
- J106 pad 6: unconnected-(J106-Pad6) -> /In_{15}
- J106 pad 7: unconnected-(J106-Pad7) -> /In_{16}
- J106 pad 8: unconnected-(J106-Pad8) -> /In_{17}
- J106 pad 9: unconnected-(J106-Pad9) -> /In_{18}
- J107 pad 1: unconnected-(J107-Pad1) -> /In_{20}
- J107 pad 10: unconnected-(J107-Pad10) -> /In_{29}
- J107 pad 2: unconnected-(J107-Pad2) -> /In_{21}
- J107 pad 3: unconnected-(J107-Pad3) -> /In_{22}
- J107 pad 4: unconnected-(J107-Pad4) -> /In_{23}
- J107 pad 5: unconnected-(J107-Pad5) -> /In_{24}
- J107 pad 6: unconnected-(J107-Pad6) -> /In_{25}
- J107 pad 7: unconnected-(J107-Pad7) -> /In_{26}
- J107 pad 8: unconnected-(J107-Pad8) -> /In_{27}
- J107 pad 9: unconnected-(J107-Pad9) -> /In_{28}
Routing:
- net /In_{29}: track 0.00 -> 43.0 mm
- net /In_{19}: track 0.00 -> 43.0 mm
- net /In_{18}: track 0.00 -> 42.9 mm
- net /In_{28}: track 0.00 -> 42.9 mm
- net /In_{27}: track 0.00 -> 35.4 mm
- net /In_{17}: track 0.00 -> 35.4 mm
- net /In_{26}: track 0.00 -> 35.3 mm
- net /In_{16}: track 0.00 -> 35.3 mm
- net /In_{15}: track 0.00 -> 32.7 mm
- net /In_{25}: track 0.00 -> 32.7 mm
- net /In_{24}: track 0.00 -> 25.3 mm
- net /In_{14}: track 0.00 -> 25.3 mm
- net /In_{13}: track 0.00 -> 25.1 mm
- net /In_{23}: track 0.00 -> 25.1 mm
- net /In_{22}: track 0.00 -> 17.6 mm
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Other:
- board size 58.4 x 134.6 mm -> 52.1 x 129.5 mm
- board text added: "+5V"
- board text added: "ALU Connector"
- board text added: "A_{0}"
- board text added: "A_{7}"
- board text added: "B_{0}"
- board text added: "B_{7}"
- board text added: "C_{0}"
- board text added: "C_{7}"
- board text added: "Commit"
- board text added: "Decode"
- board text added: "Execute"
- board text added: "Flag"
- board text added: "GND"
- board text added: "I_{0}"
- board text added: "I_{3}"
- board text added: "In_{00}"
- board text added: "In_{09}"
- board text added: "In_{10}"
- board text added: "In_{19}"
- board text added: "In_{20}"
- board text added: "In_{29}"
- board text added: "Inputs"
- board text added: "JLCJLCJLCJLC"
- board text added: "Outputs"
- board text added: "RGE2023"
- board text added: "~{SELECT}"
