File: pcbs/SALU/decoder.kicad_sch (KiCad schematic)
At the start: 44 parts, among them U301 74HC138, U302 74HC138

Commit message: Some more functions
Parts:
- renumbered D304 to D302, D307 to D303, D309 to D304, D317 to D305, D319 to D306, D313 to D307, D315 to D308, D303 to D309, D306 to D310, D310 to D311, D318 to D313, D320 to D314, D302 to D315, D305 to D316, D308 to D317, D311 to D318, D314 to D319, D316 to D320, R304 to R302, R307 to R303, R309 to R304, R317 to R305, R319 to R306, R303 to R307, R306 to R308, R310 to R309, R312 to R310, R313 to R311, R315 to R312, R318 to R313, R320 to R314, R302 to R315, R305 to R316, R314 to R317, R316 to R318, R308 to R319, R311 to R320
