File: pcbs/SALU/incdec.kicad_sch (KiCad schematic)
At the start: 22 parts, among them U401 74HC283, U402 74HC245, U403 74HC245, U404 74HC86, U405 74HC283, U406 74HC245, U407 74HC08

Commit message: Some more functions
Parts:
- renumbered U403 to U401, U404 to U402, U407 to U403, U401 to U404, U402 to U406, U406 to U407
