File: pcbs/SALU/SALU.kicad_pcb (KiCad board)
At the start: 4 copper layers, 99 parts, among them J201 Conn_02x20_Odd_Even, U201 74HC245, U202 74HC245, U301 74HC138, U302 74HC138, U401 74HC245, U402 74HC86, U403 74HC08, U404 74HC283, U405 74HC283, U406 74HC245, U407 74HC245, U501 74HC00, U502 74HC00, U503 74HC245, U504 74HC245, U601 74HC245, U602 74HC245, U701 74HC08, U702 74HCT125, U703 74HC245, U704 74HC245

Commit message: Routing, routing, routing
Parts:
- moved U703 21.0 mm to (129.5, 52.1)
- moved U704 19.9 mm to (129.5, 67.3)
- moved C701 9.03 mm to (130.8, 24.1), turned to 90 degrees
- moved U701 8.13 mm to (128.3, 30.5)
- moved R405 7.62 mm to (67.3, 64.8)
- moved R408 7.62 mm to (59.7, 64.8)
- moved U501 3.82 mm to (83.8, 97.8)
- moved U502 3.82 mm to (83.8, 119.4)
- moved C501 3.81 mm to (95.2, 97.8), turned to 0 degrees
- moved C502 3.06 mm to (95.5, 119.4)
- moved R406 2.54 mm to (64.8, 64.8)
- moved R407 2.54 mm to (62.2, 64.8)
- moved C503 1.27 mm to (111.8, 94.0)
- moved U503 1.27 mm to (106.7, 102.9)
- moved U504 1.27 mm to (106.7, 144.8)
Connections:
- U503 pad 11: /Not-Copy/RESULT7 -> /Incrementer-Decrementer/RESULT7
- U503 pad 12: /Not-Copy/RESULT6 -> /Incrementer-Decrementer/RESULT6
- U503 pad 13: /Not-Copy/RESULT5 -> /Incrementer-Decrementer/RESULT5
- U503 pad 14: /Not-Copy/RESULT4 -> /Incrementer-Decrementer/RESULT4
- U503 pad 15: /Not-Copy/RESULT3 -> /Incrementer-Decrementer/RESULT3
- U503 pad 16: /Not-Copy/RESULT2 -> /Incrementer-Decrementer/RESULT2
- U503 pad 17: /Not-Copy/RESULT1 -> /Incrementer-Decrementer/RESULT1
- U503 pad 18: /Not-Copy/RESULT0 -> /Incrementer-Decrementer/RESULT0
- U504 pad 11: /Not-Copy/RESULT7 -> /Incrementer-Decrementer/RESULT7
- U504 pad 12: /Not-Copy/RESULT6 -> /Incrementer-Decrementer/RESULT6
- U504 pad 13: /Not-Copy/RESULT5 -> /Incrementer-Decrementer/RESULT5
- U504 pad 14: /Not-Copy/RESULT4 -> /Incrementer-Decrementer/RESULT4
- U504 pad 15: /Not-Copy/RESULT3 -> /Incrementer-Decrementer/RESULT3
- U504 pad 16: /Not-Copy/RESULT2 -> /Incrementer-Decrementer/RESULT2
- U504 pad 17: /Not-Copy/RESULT1 -> /Incrementer-Decrementer/RESULT1
- U504 pad 18: /Not-Copy/RESULT0 -> /Incrementer-Decrementer/RESULT0
Routing:
- net /Barrel Shifters/A1: track 79.2 -> 288.2 mm, vias 0 -> 8
- net /Barrel Shifters/A0: track 79.2 -> 287.7 mm, vias 0 -> 7
- net /Barrel Shifters/A5: track 79.2 -> 280.1 mm, vias 0 -> 7
- net /Barrel Shifters/A2: track 79.2 -> 275.5 mm, vias 0 -> 8
- net /Barrel Shifters/A6: track 79.2 -> 274.7 mm, vias 0 -> 7
- net /Barrel Shifters/A4: track 79.2 -> 274.5 mm, vias 0 -> 7
- net /Barrel Shifters/A3: track 79.2 -> 267.9 mm, vias 0 -> 8
- net /Barrel Shifters/A7: track 79.2 -> 253.8 mm, vias 0 -> 6
- net /Incrementer-Decrementer/RESULT0: track 0.00 -> 137.8 mm, vias 0 -> 4
- net /Incrementer-Decrementer/RESULT1: track 0.00 -> 135.0 mm, vias 0 -> 4
- net /Incrementer-Decrementer/RESULT2: track 0.00 -> 132.9 mm, vias 0 -> 4
- net /Incrementer-Decrementer/RESULT6: track 0.00 -> 131.2 mm, vias 0 -> 4
- net /Incrementer-Decrementer/RESULT3: track 0.00 -> 130.1 mm, vias 0 -> 4
- net /Incrementer-Decrementer/RESULT7: track 0.00 -> 127.6 mm, vias 0 -> 4
- net /Incrementer-Decrementer/RESULT4: track 0.00 -> 127.3 mm, vias 0 -> 4
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