File: pcbs/SALU/not_copy.kicad_sch (KiCad schematic)
At the start: 8 parts, among them U501 74HC00, U502 74HC00, U503 74HC245, U504 74HC245

Commit message: Routing, routing, routing
Changed lines of the file:
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@@
     (effects (font (size 1.27 1.27)) (justify right))
   )
-  (hierarchical_label "RESULT[0..7]" (shape output) (at 262.255 145.415 0)
+  (hierarchical_label "RESULT[0..7]" (shape tri_state) (at 262.255 145.415 0)
     (effects (font (size 1.27 1.27)) (justify left))
   )
