File: pcbs/SALU/barrel_shifters.kicad_sch (KiCad schematic)
At the start: 4 parts, among them U601 74HC245, U602 74HC245

Commit message: More routing
Changed lines of the file:
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@@
     (effects (font (size 1.27 1.27)) (justify right))
   )
-  (hierarchical_label "RESULT[0..7]" (shape output) (at 184.15 21.59 0)
+  (hierarchical_label "RESULT[0..7]" (shape tri_state) (at 184.15 21.59 0)
     (effects (font (size 1.27 1.27)) (justify left))
   )
