File: pcbs/SALU/shifters.kicad_sch (KiCad schematic)
At the start: 8 parts, among them U701 74HC08, U702 74HCT125, U703 74HC245, U704 74HC245

Commit message: More routing
Changed lines of the file:
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@@
     (effects (font (size 1.27 1.27)) (justify right))
   )
-  (hierarchical_label "RESULT[0..7]" (shape output) (at 199.39 29.845 0)
+  (hierarchical_label "RESULT[0..7]" (shape tri_state) (at 199.39 29.845 0)
     (effects (font (size 1.27 1.27)) (justify left))
   )

Commit message: Fiddling around with shifters
Connections:
- net A0: now also U702.2, U702.5; no longer U702.12, U702.9
- net A7: now also U702.12, U702.9; no longer U702.2, U702.5
- net GND: now also U701.1, U701.2; no longer U701.10, U701.9
- net ~{LSHIFT0}: now also U701.9, U702.10; no longer U701.1, U702.1
- net ~{LSHIFT1}: now also U701.10, U702.13; no longer U701.2, U702.4
- net ~{RSHIFT0}: now also U702.4; no longer U702.10
- net ~{RSHIFT1}: now also U702.1; no longer U702.13
- net at U703.19 (CE): now also U701.8; no longer U701.3
Other:
- moved on the sheet: U701A, U701C, U702A, U702B, U702C, U702D
