File: pcbs/Register File/Register File.kicad_pcb (KiCad board)
At the start: 4 copper layers, 208 parts, among them U201 74HCT574, U202 74HC245, U203 74HC245, U204 74HC245, U301 74HCT574, U302 74HC245, U303 74HC245, U304 74HC245, U401 74HCT574, U402 74HC245, U403 74HC245, U404 74HC245, U501 74HCT574, U502 74HC245, U503 74HC245, U504 74HC245, U601 74HCT574, U602 74HC245, U603 74HC245, U604 74HC245, U701 74HCT574, U702 74HC245, U703 74HC245, U704 74HC245, U801 74HCT574, U802 74HC245, U803 74HC245, U804 74HC245, U901 74HCT574, U902 74HC245, U903 74HC245, U904 74HC245

Commit message: Remember the control buses...
Parts:
- moved D910 112.2 mm to (250.9, 115.0)
- moved D909 112.2 mm to (250.9, 109.8)
- moved D911 112.2 mm to (250.9, 112.4)
- moved R909 112.2 mm to (255.0, 109.8)
- moved R911 112.2 mm to (255.0, 112.3)
- moved R910 112.2 mm to (255.0, 114.8)
- moved R809 78.3 mm to (226.0, 110.8)
- moved R811 78.3 mm to (226.0, 113.3)
- moved R810 78.3 mm to (226.0, 115.8)
- moved D809 78.3 mm to (222.0, 110.8)
- moved D810 78.3 mm to (222.0, 116.0)
- moved D811 78.3 mm to (222.0, 113.4)
- moved R611 58.4 mm to (175.7, 113.8)
- moved D609 58.4 mm to (171.7, 111.3)
- moved D611 58.4 mm to (171.7, 113.9)
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Connections:
- U202 pad 1: unconnected-(U202-A->B-Pad1) -> +5V
- U203 pad 1: unconnected-(U203-A->B-Pad1) -> +5V
- U204 pad 1: unconnected-(U204-A->B-Pad1) -> +5V
- U302 pad 1: unconnected-(U302-A->B-Pad1) -> +5V
- U303 pad 1: unconnected-(U303-A->B-Pad1) -> +5V
- U304 pad 1: unconnected-(U304-A->B-Pad1) -> +5V
- U402 pad 1: unconnected-(U402-A->B-Pad1) -> +5V
- U403 pad 1: unconnected-(U403-A->B-Pad1) -> +5V
- U404 pad 1: unconnected-(U404-A->B-Pad1) -> +5V
- U502 pad 1: unconnected-(U502-A->B-Pad1) -> +5V
- U503 pad 1: unconnected-(U503-A->B-Pad1) -> +5V
- U504 pad 1: unconnected-(U504-A->B-Pad1) -> +5V
- U602 pad 1: unconnected-(U602-A->B-Pad1) -> +5V
- U603 pad 1: unconnected-(U603-A->B-Pad1) -> +5V
- U604 pad 1: unconnected-(U604-A->B-Pad1) -> +5V
- U702 pad 1: unconnected-(U702-A->B-Pad1) -> +5V
- U703 pad 1: unconnected-(U703-A->B-Pad1) -> +5V
- U704 pad 1: unconnected-(U704-A->B-Pad1) -> +5V
- U802 pad 1: unconnected-(U802-A->B-Pad1) -> +5V
- U803 pad 1: unconnected-(U803-A->B-Pad1) -> +5V
- U804 pad 1: unconnected-(U804-A->B-Pad1) -> +5V
- U902 pad 1: unconnected-(U902-A->B-Pad1) -> +5V
- U903 pad 1: unconnected-(U903-A->B-Pad1) -> +5V
- U904 pad 1: unconnected-(U904-A->B-Pad1) -> +5V
Routing:
- net /Register 7/~{C_{Enable}}: track 0.00 -> 195.8 mm, vias 0 -> 1
- net /Register 7/~{B_{Enable}}: track 0.00 -> 195.3 mm, vias 0 -> 1
- net /Register 7/~{A_{Enable}}: track 0.00 -> 195.3 mm, vias 0 -> 1
- net /Register 6/~{C_{Enable}}: track 0.00 -> 169.9 mm, vias 0 -> 2
- net /Register 6/~{B_{Enable}}: track 0.00 -> 169.4 mm, vias 0 -> 1
- net /Register 6/~{A_{Enable}}: track 2.16 -> 169.4 mm, vias 0 -> 1
- net /Register 5/~{C_{Enable}}: track 0.00 -> 144.0 mm, vias 0 -> 1
- net /Register 5/~{B_{Enable}}: track 0.00 -> 143.5 mm, vias 0 -> 1
- net /Register 5/~{A_{Enable}}: track 0.00 -> 143.5 mm, vias 0 -> 1
- net /Register 4/~{C_{Enable}}: track 0.00 -> 118.1 mm, vias 0 -> 1
- net /Register 4/~{B_{Enable}}: track 0.00 -> 117.6 mm, vias 0 -> 1
- net /Register 4/~{A_{Enable}}: track 0.00 -> 117.6 mm, vias 0 -> 1
- net /Register 3/~{C_{Enable}}: track 0.00 -> 92.2 mm, vias 0 -> 1
- net /Register 3/~{B_{Enable}}: track 0.00 -> 91.7 mm, vias 0 -> 1
- net /Register 3/~{A_{Enable}}: track 0.00 -> 91.7 mm, vias 0 -> 1
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
Commit message: Yet more routing
Parts:
- added U1001: 74HC138, Package_DIP:DIP-16_W7.62mm_Socket, F.Cu at (43.2, 57.1)
Connections:
- net /Register 0/~{A_{Enable}} renamed /Selectors/~{A_{select}}0
- net /Register 1/~{A_{Enable}} renamed /Selectors/~{A_{select}}1
- net /Register 2/~{A_{Enable}} renamed /Selectors/~{A_{select}}2
- net /Register 3/~{A_{Enable}} renamed /Selectors/~{A_{select}}3
- net /Register 4/~{A_{Enable}} renamed /Selectors/~{A_{select}}4
- net /Register 5/~{A_{Enable}} renamed /Selectors/~{A_{select}}5
- net /Register 6/~{A_{Enable}} renamed /Selectors/~{A_{select}}6
- net /Register 7/~{A_{Enable}} renamed /Selectors/~{A_{select}}7
- U801 pad 2: /Register 6/C0 -> /Register 0/C0
- U801 pad 3: /Register 6/C1 -> /Register 0/C1
- U801 pad 4: /Register 6/C2 -> /Register 0/C2
- U801 pad 5: /Register 6/C3 -> /Register 0/C3
- U801 pad 6: /Register 6/C4 -> /Register 0/C4
- U801 pad 7: /Register 6/C5 -> /Register 0/C5
- U801 pad 8: /Register 6/C6 -> /Register 0/C6
- U801 pad 9: /Register 6/C7 -> /Register 0/C7
- U802 pad 11: /Register 6/A7 -> /Register 0/A7
- U802 pad 12: /Register 6/A6 -> /Register 0/A6
- U802 pad 13: /Register 6/A5 -> /Register 0/A5
- U802 pad 14: /Register 6/A4 -> /Register 0/A4
- U802 pad 15: /Register 6/A3 -> /Register 0/A3
- U802 pad 16: /Register 6/A2 -> /Register 0/A2
- U802 pad 17: /Register 6/A1 -> /Register 0/A1
- U802 pad 18: /Register 6/A0 -> /Register 0/A0
- U803 pad 11: /Register 6/B7 -> /Register 0/B7
- U803 pad 12: /Register 6/B6 -> /Register 0/B6
- U803 pad 13: /Register 6/B5 -> /Register 0/B5
- U803 pad 14: /Register 6/B4 -> /Register 0/B4
- U803 pad 15: /Register 6/B3 -> /Register 0/B3
- U803 pad 16: /Register 6/B2 -> /Register 0/B2
- U803 pad 17: /Register 6/B1 -> /Register 0/B1
- U803 pad 18: /Register 6/B0 -> /Register 0/B0
- U804 pad 11: /Register 6/C7 -> /Register 0/C7
- U804 pad 12: /Register 6/C6 -> /Register 0/C6
- U804 pad 13: /Register 6/C5 -> /Register 0/C5
- U804 pad 14: /Register 6/C4 -> /Register 0/C4
- U804 pad 15: /Register 6/C3 -> /Register 0/C3
- U804 pad 16: /Register 6/C2 -> /Register 0/C2
- U804 pad 17: /Register 6/C1 -> /Register 0/C1
- U804 pad 18: /Register 6/C0 -> /Register 0/C0
- U901 pad 2: /Register 7/C0 -> /Register 0/C0
- U901 pad 3: /Register 7/C1 -> /Register 0/C1
- U901 pad 4: /Register 7/C2 -> /Register 0/C2
- U901 pad 5: /Register 7/C3 -> /Register 0/C3
- U901 pad 6: /Register 7/C4 -> /Register 0/C4
- U901 pad 7: /Register 7/C5 -> /Register 0/C5
- U901 pad 8: /Register 7/C6 -> /Register 0/C6
- U901 pad 9: /Register 7/C7 -> /Register 0/C7
- U902 pad 11: /Register 7/A7 -> /Register 0/A7
- U902 pad 12: /Register 7/A6 -> /Register 0/A6
- U902 pad 13: /Register 7/A5 -> /Register 0/A5
- U902 pad 14: /Register 7/A4 -> /Register 0/A4
- U902 pad 15: /Register 7/A3 -> /Register 0/A3
- U902 pad 16: /Register 7/A2 -> /Register 0/A2
- U902 pad 17: /Register 7/A1 -> /Register 0/A1
- U902 pad 18: /Register 7/A0 -> /Register 0/A0
- U903 pad 11: /Register 7/B7 -> /Register 0/B7
- U903 pad 12: /Register 7/B6 -> /Register 0/B6
- U903 pad 13: /Register 7/B5 -> /Register 0/B5
- U903 pad 14: /Register 7/B4 -> /Register 0/B4
- U903 pad 15: /Register 7/B3 -> /Register 0/B3
- U903 pad 16: /Register 7/B2 -> /Register 0/B2
- U903 pad 17: /Register 7/B1 -> /Register 0/B1
- U903 pad 18: /Register 7/B0 -> /Register 0/B0
- U904 pad 11: /Register 7/C7 -> /Register 0/C7
- U904 pad 12: /Register 7/C6 -> /Register 0/C6
- U904 pad 13: /Register 7/C5 -> /Register 0/C5
- U904 pad 14: /Register 7/C4 -> /Register 0/C4
- U904 pad 15: /Register 7/C3 -> /Register 0/C3
- U904 pad 16: /Register 7/C2 -> /Register 0/C2
- U904 pad 17: /Register 7/C1 -> /Register 0/C1
- U904 pad 18: /Register 7/C0 -> /Register 0/C0
Routing:
- net /Register 0/C7: track 281.8 -> 386.8 mm, vias 6 -> 8
- net /Register 0/C6: track 281.8 -> 386.8 mm, vias 6 -> 8
- net /Register 0/C5: track 281.8 -> 386.8 mm, vias 6 -> 8
- net /Register 0/C4: track 281.8 -> 386.8 mm, vias 6 -> 8
- net /Register 0/C2: track 280.1 -> 384.9 mm, vias 6 -> 8
- net /Register 0/C3: track 279.8 -> 384.7 mm, vias 6 -> 8
- net /Register 0/C1: track 279.8 -> 384.7 mm, vias 6 -> 8
- net /Register 0/C0: track 279.8 -> 384.7 mm, vias 6 -> 8
- net /Register 0/B7: track 149.3 -> 201.6 mm, vias 6 -> 8
- net /Register 0/B6: track 149.3 -> 201.6 mm, vias 6 -> 8
- net /Register 0/B5: track 149.3 -> 201.6 mm, vias 6 -> 8
- net /Register 0/B4: track 149.3 -> 201.6 mm, vias 6 -> 8
- net /Register 0/B0: track 147.3 -> 199.5 mm, vias 6 -> 8
- net /Register 0/B3: track 147.3 -> 199.5 mm, vias 6 -> 8
- net /Register 0/B2: track 147.3 -> 199.5 mm, vias 6 -> 8
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