File: pcbs/Register File/Register File.kicad_pcb (KiCad board)
At the start: 4 copper layers, 251.5 x 116.8 mm, 215 parts, among them J101 Conn_02x20_Odd_Even, U1001 74HC138, U1002 74HC138, U1004 74HC138, U1007 74HC14, U201 74HCT574, U202 74HC245, U203 74HC245, U301 74HCT574, U302 74HC245, U303 74HC245, U401 74HCT574, U402 74HC245, U403 74HC245, U501 74HCT574, U502 74HC245, U503 74HC245, U601 74HCT574, U602 74HC245, U603 74HC245, U701 74HCT574, U702 74HC245, U703 74HC245, U801 74HCT574, U802 74HC245, U803 74HC245, U901 74HCT574, U902 74HC245, U903 74HC245

Commit message: Better routing
Parts:
- moved U1007 82.0 mm to (40.6, 31.8)
- moved U902 22.9 mm to (226.1, 63.5)
- moved U903 22.9 mm to (226.1, 83.8)
- moved U802 20.3 mm to (203.2, 63.5)
- moved U803 20.3 mm to (203.2, 83.8)
- moved D709 18.0 mm to (184.2, 55.4)
- moved D711 18.0 mm to (184.2, 75.7)
- moved R709 17.8 mm to (180.3, 55.4)
- moved R711 17.8 mm to (180.3, 75.7)
- moved U702 17.8 mm to (180.3, 63.5)
- moved U703 17.8 mm to (180.3, 83.8)
- moved D609 15.5 mm to (161.3, 55.4)
- moved D611 15.5 mm to (161.3, 75.7)
- moved R609 15.2 mm to (157.5, 55.4)
- moved R611 15.2 mm to (157.5, 75.7)
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Routing:
- net /Selectors/~{B_{select}}7: track 0.00 -> 202.5 mm
- net /Selectors/~{B_{select}}6: track 0.00 -> 179.9 mm
- net /Selectors/~{B_{select}}5: track 0.00 -> 174.1 mm, vias 0 -> 2
- net /Register 0/A0: track 0.00 -> 168.1 mm
- net /Selectors/~{A_{select}}6: track 19.9 -> 187.0 mm
- net /Selectors/~{A_{select}}5: track 16.9 -> 174.1 mm, vias 0 -> 2
- net /Selectors/~{B_{select}}4: track 0.00 -> 147.7 mm, vias 0 -> 2
- net /Register 0/A2: track 0.00 -> 144.0 mm
- net /Register 0/A7: track 0.00 -> 144.0 mm
- net /Register 0/A3: track 0.00 -> 144.0 mm
- net /Register 0/A1: track 0.00 -> 144.0 mm
- net /Register 0/A4: track 0.00 -> 144.0 mm
- net /Register 0/A6: track 0.00 -> 144.0 mm
- net /Register 0/A5: track 0.00 -> 144.0 mm
- net /Register 0/B6: track 0.00 -> 140.3 mm
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
Commit message: Working and routing
Parts:
- added U1001: 74HC14, Package_SO:SOIC-14_3.9x8.7mm_P1.27mm, F.Cu at (43.2, 17.7)
- moved J101 146.8 mm to (10.2, 33.0), turned to 0 degrees
- moved U1002 96.5 mm to (135.9, 16.6), turned to 90 degrees
- moved D909 23.1 mm to (229.9, 55.4)
- moved D910 23.1 mm to (229.9, 75.7)
- moved R909 22.9 mm to (226.1, 55.4)
- moved R910 22.9 mm to (226.1, 75.7)
- moved D809 20.6 mm to (207.0, 55.4)
- moved D810 20.6 mm to (207.0, 75.7)
- moved R809 20.3 mm to (203.2, 55.4)
- moved R810 20.3 mm to (203.2, 75.7)
- moved D1001 1.27 mm to (58.4, 21.6)
- moved D1002 1.27 mm to (81.3, 21.6)
- moved D1003 1.27 mm to (104.1, 21.6)
- moved D1004 1.27 mm to (127.0, 21.6)
- moved D1005 1.27 mm to (149.9, 21.6)
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- renumbered D211 to D210, D311 to D310, D411 to D410, D511 to D510, D611 to D610, D711 to D710, D811 to D810, D911 to D910, R1009 to R1001, R1010 to R1002, R1011 to R1003, R1012 to R1004, R1013 to R1005, R1014 to R1006, R1015 to R1007, R1016 to R1008, R211 to R210, R311 to R310, R411 to R410, R511 to R510, R611 to R610, R711 to R710, R811 to R810, R911 to R910, U1007 to U1002, U1004 to U1003, U1001 to U1004, U1002 to U1005
Connections:
- U1002 pad 1: GND -> /Selectors/W4
- U1002 pad 10: unconnected-(U1007-Pad10) -> /Selectors/C_{Write}7
- U1002 pad 11: unconnected-(U1007-Pad11) -> /Selectors/W7
- U1002 pad 12: unconnected-(U1007-Pad12) -> /Selectors/C_{Write}5
- U1002 pad 13: unconnected-(U1007-Pad13) -> /Selectors/W5
- U1002 pad 2: unconnected-(U1007-Pad2) -> /Selectors/C_{Write}4
- U1002 pad 3: GND -> /Selectors/W6
- U1002 pad 4: unconnected-(U1007-Pad4) -> /Selectors/C_{Write}6
- U1003 pad 8: unconnected-(U1004-GND-Pad8) -> GND
- U201 pad 11: /C_{Write}0 -> /Selectors/C_{Write}0
- U301 pad 11: /C_{Write}1 -> /Selectors/C_{Write}1
- U401 pad 11: /C_{Write}2 -> /Selectors/C_{Write}2
- U501 pad 11: /C_{Write}3 -> /Selectors/C_{Write}3
- U601 pad 11: /C_{Write}4 -> /Selectors/C_{Write}4
- U701 pad 11: /C_{Write}5 -> /Selectors/C_{Write}5
- U801 pad 11: /C_{Write}6 -> /Selectors/C_{Write}6
- U901 pad 11: /C_{Write}7 -> /Selectors/C_{Write}7
Routing:
- net /Register 7/r0: track 0.00 -> 86.0 mm, vias 0 -> 2
- net /Register 7/r2: track 0.00 -> 75.8 mm, vias 0 -> 2
- net /Register 7/r3: track 0.00 -> 70.8 mm, vias 0 -> 2
- net /Register 7/r4: track 0.00 -> 66.5 mm, vias 0 -> 2
- net /Register 7/r5: track 0.00 -> 62.8 mm, vias 0 -> 2
- net /Register 7/r1: track 22.7 -> 80.8 mm, vias 0 -> 2
- net /Register 7/r7: track 0.00 -> 55.8 mm, vias 0 -> 2
- net GND: track 132.3 -> 185.2 mm, vias 28 -> 49
- net /Register 7/r6: track 7.47 -> 59.2 mm, vias 0 -> 2
- net /Register 0/A7: track 144.0 -> 195.2 mm
- net /Register 0/A6: track 144.0 -> 194.5 mm
- net /Register 0/A5: track 144.0 -> 193.9 mm
- net /Register 0/A4: track 144.0 -> 193.3 mm
- net /Register 0/A3: track 144.0 -> 192.7 mm
- net /Register 0/A2: track 144.0 -> 192.0 mm
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Other:
- board size 251.5 x 116.8 mm -> 261.6 x 116.8 mm

Commit message: Finish board
Parts:
- added C1003: 100n, Capacitor_SMD:C_0603_1608Metric, F.Cu at (46.9, 76.2)
- added H101: MountingHole, MountingHole:MountingHole_2.7mm_M2.5, F.Cu at (10.2, 15.2)
- added H102: MountingHole, MountingHole:MountingHole_2.7mm_M2.5, F.Cu at (238.8, 15.2)
- added H103: MountingHole, MountingHole:MountingHole_2.7mm_M2.5, F.Cu at (10.2, 88.9)
- added H104: MountingHole, MountingHole:MountingHole_2.7mm_M2.5, F.Cu at (238.8, 88.9)
- moved C1002 45.1 mm to (47.0, 55.9)
- moved C1001 13.3 mm to (41.9, 33.0)
- moved U1003 12.7 mm to (38.1, 25.4), turned to -90 degrees
- moved U1002 2.03 mm to (136.4, 14.6), turned to 0 degrees
- moved U1001 0.70 mm to (43.2, 18.4), turned to 0 degrees
Connections:
- D1001 pad 2: +5V -> /Selectors/C_{Write}0
- D1002 pad 2: +5V -> /Selectors/C_{Write}1
- D1003 pad 2: +5V -> /Selectors/C_{Write}2
- D1004 pad 2: +5V -> /Selectors/C_{Write}3
- D1005 pad 2: +5V -> /Selectors/C_{Write}4
- D1006 pad 2: +5V -> /Selectors/C_{Write}5
- D1007 pad 2: +5V -> /Selectors/C_{Write}6
- D1008 pad 2: +5V -> /Selectors/C_{Write}7
- J101 pad 1: /Selectors/R_{A}0 -> GND
- J101 pad 10: /Register 0/A3 -> /Register 0/C4
- J101 pad 11: /Selectors/R_{B}2 -> /Register 0/C5
- J101 pad 12: /Register 0/A4 -> /Register 0/C6
- J101 pad 13: /Selectors/R_{C}0 -> /Register 0/C7
- J101 pad 14: /Register 0/A5 -> /Selectors/R_{A}0
- J101 pad 15: /Selectors/R_{C}1 -> /Selectors/R_{A}1
- J101 pad 16: /Register 0/A6 -> /Selectors/R_{A}2
- J101 pad 17: /Selectors/R_{C}2 -> /Register 0/A1
- J101 pad 18: /Register 0/A7 -> /Register 0/A0
- J101 pad 19: /De -> /Register 0/A3
- J101 pad 2: unconnected-(J101-Pin_2-Pad2) -> +5V
- J101 pad 20: /Co -> /Register 0/A2
- J101 pad 21: /Ex -> /Register 0/A5
- J101 pad 22: /PC -> /Register 0/A4
- J101 pad 23: /Register 0/C0 -> /Register 0/A7
- J101 pad 24: /Register 0/B0 -> /Register 0/A6
- J101 pad 25: /Register 0/C1 -> /Selectors/R_{B}1
- J101 pad 26: /Register 0/B1 -> /Selectors/R_{B}0
- J101 pad 27: /Register 0/C2 -> unconnected-(J101-Pin_27-Pad27)
- J101 pad 28: /Register 0/B2 -> /Selectors/R_{B}2
- J101 pad 29: /Register 0/C3 -> /W
- J101 pad 3: /Selectors/R_{A}1 -> /Selectors/R_{C}0
- J101 pad 30: /Register 0/B3 -> /~{Enable}
- J101 pad 31: /Register 0/C4 -> /Register 0/B1
- J101 pad 32: /Register 0/B4 -> /Register 0/B0
- J101 pad 33: /Register 0/C5 -> /Register 0/B3
- J101 pad 34: /Register 0/B5 -> /Register 0/B2
- J101 pad 35: /Register 0/C6 -> /Register 0/B5
- J101 pad 36: /Register 0/B6 -> /Register 0/B4
- J101 pad 37: /Register 0/C7 -> /Register 0/B7
- J101 pad 38: /Register 0/B7 -> /Register 0/B6
- J101 pad 4: /Register 0/A0 -> /Selectors/R_{C}1
- J101 pad 5: /Selectors/R_{A}2 -> /Selectors/R_{C}2
- J101 pad 6: /Register 0/A1 -> /Register 0/C0
- J101 pad 7: /Selectors/R_{B}0 -> /Register 0/C1
- J101 pad 8: /Register 0/A2 -> /Register 0/C2
- J101 pad 9: /Selectors/R_{B}1 -> /Register 0/C3
- R1001 pad 1: /Selectors/W0 -> GND
- R1002 pad 1: /Selectors/W1 -> GND
- R1003 pad 1: /Selectors/W2 -> GND
- R1004 pad 1: /Selectors/W3 -> GND
- R1005 pad 1: /Selectors/W4 -> GND
- R1006 pad 1: /Selectors/W5 -> GND
- R1007 pad 1: /Selectors/W6 -> GND
- R1008 pad 1: /Selectors/W7 -> GND
- U1001 pad 1: /Selectors/W0 -> Net-(U1003-~{Y3})
- U1001 pad 10: /Selectors/C_{Write}3 -> /Selectors/C_{Write}0
- U1001 pad 11: /Selectors/W3 -> Net-(U1003-~{Y0})
- U1001 pad 12: /Selectors/C_{Write}1 -> /Selectors/C_{Write}2
- U1001 pad 13: /Selectors/W1 -> Net-(U1003-~{Y2})
- U1001 pad 2: /Selectors/C_{Write}0 -> /Selectors/C_{Write}3
- U1001 pad 3: /Selectors/W2 -> Net-(U1003-~{Y1})
- U1001 pad 4: /Selectors/C_{Write}2 -> /Selectors/C_{Write}1
- U1002 pad 1: /Selectors/W4 -> Net-(U1003-~{Y7})
- U1002 pad 10: /Selectors/C_{Write}7 -> /Selectors/C_{Write}4
- U1002 pad 11: /Selectors/W7 -> Net-(U1003-~{Y4})
- U1002 pad 12: /Selectors/C_{Write}5 -> /Selectors/C_{Write}6
- U1002 pad 13: /Selectors/W5 -> Net-(U1003-~{Y6})
- U1002 pad 2: /Selectors/C_{Write}4 -> /Selectors/C_{Write}7
- U1002 pad 3: /Selectors/W6 -> Net-(U1003-~{Y5})
- U1002 pad 4: /Selectors/C_{Write}6 -> /Selectors/C_{Write}5
- U1003 pad 10: /Selectors/W5 -> Net-(U1003-~{Y5})
- U1003 pad 11: /Selectors/W4 -> Net-(U1003-~{Y4})
- U1003 pad 12: /Selectors/W3 -> Net-(U1003-~{Y3})
- U1003 pad 13: /Selectors/W2 -> Net-(U1003-~{Y2})
- U1003 pad 14: /Selectors/W1 -> Net-(U1003-~{Y1})
- U1003 pad 15: /Selectors/W0 -> Net-(U1003-~{Y0})
- U1003 pad 4: /Selectors/~{Active} -> /~{Enable}
- U1003 pad 6: /Selectors/C_{W}/~{C_{R}} -> /W
- U1003 pad 7: /Selectors/W7 -> Net-(U1003-~{Y7})
- U1003 pad 9: /Selectors/W6 -> Net-(U1003-~{Y6})
- U1004 pad 4: /Selectors/~{Active} -> /~{Enable}
- U1005 pad 4: /Selectors/~{Active} -> /~{Enable}
Routing:
- net Net-(U1003-~{Y6}): track 0.00 -> 140.2 mm, vias 0 -> 1
- net Net-(U1003-~{Y4}): track 0.00 -> 134.4 mm, vias 0 -> 1
- net Net-(U1003-~{Y5}): track 0.00 -> 131.8 mm, vias 0 -> 1
- net Net-(U1003-~{Y7}): track 0.00 -> 126.6 mm, vias 0 -> 1
- net +5V: track 25.8 -> 143.2 mm, vias 0 -> 50
- net /Selectors/C_{Write}7: track 27.8 -> 127.5 mm, vias 0 -> 2
- net /Selectors/C_{Write}3: track 26.8 -> 125.9 mm, vias 0 -> 2
- net /~{Enable}: track 0.00 -> 73.7 mm, vias 0 -> 2
- net /Register 0/B5: track 163.7 -> 233.9 mm, vias 0 -> 2
- net /Register 0/B1: track 163.7 -> 233.9 mm, vias 0 -> 2
- net /Register 0/B7: track 163.7 -> 233.9 mm, vias 0 -> 2
- net /Register 0/B3: track 163.7 -> 233.9 mm, vias 0 -> 2
- net /Selectors/C_{Write}6: track 27.8 -> 97.9 mm, vias 0 -> 2
- net /W: track 0.00 -> 68.2 mm, vias 0 -> 2
- net /Selectors/C_{Write}2: track 27.8 -> 95.9 mm, vias 0 -> 2
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- removed copper zone on In1.Cu, net GND
- removed copper zone on In2.Cu, net GND
Other:
- board size 261.6 x 116.8 mm -> 243.8 x 88.9 mm
- copper layers 4 -> 2
- board text removed: "(out)"
- board text removed: "+5V"
- board text removed: "A0"
- board text removed: "A7"
- board text removed: "B0"
- board text removed: "B7"
- board text removed: "C Bus"
- board text removed: "C0"
- board text removed: "C7"
- board text removed: "C_{W}/~{C_{R}}"
- board text removed: "Commit"
- board text removed: "Decode"
- board text removed: "Execute"
- board text removed: "GND"
- board text removed: "PC Update"
- board text removed: "R_{A}"
- board text removed: "R_{B}"
- board text removed: "R_{C}"
