File: pcbs/Register File/Register File.kicad_sch (KiCad schematic)
At the start: 1 part, among them J101 Conn_02x20_Odd_Even

Commit message: Lots of rethinking
Connections:
- net Selectors/C_{W}/~{C_{R}}: no longer names the net of J101.2 (Pin_2)
Other:
- sheet Register 0 ports: added none; removed ~{C_{Enable}}
- sheet Register 1 ports: added none; removed ~{C_{Enable}}
- sheet Register 2 ports: added none; removed ~{C_{Enable}}
- sheet Register 3 ports: added none; removed ~{C_{Enable}}
- sheet Register 4 ports: added none; removed ~{C_{Enable}}
- sheet Register 5 ports: added none; removed ~{C_{Enable}}
- sheet Register 6 ports: added none; removed ~{C_{Enable}}
- sheet Register 7 ports: added none; removed ~{C_{Enable}}
- sheet Selectors ports: added none; removed C_{W}/~{C_{R}}, {De, Ex, Co, PC}, ~{C_{select}}[0..7]

Commit message: Finish board
Parts:
- added H101, H102, H103, H104: MountingHole, MountingHole:MountingHole_2.7mm_M2.5, symbol Mechanical:MountingHole
Connections:
- net Co is gone; now on net A2: J101.20 (Pin_20)
- net De is gone; now on net A3: J101.19 (Pin_19)
- net Ex is gone; now on net A5: J101.21 (Pin_21)
- net PC is gone; now on net A4: J101.22 (Pin_22)
- net +5V: now also J101.2 (Pin_2)
- net A0: now also J101.18 (Pin_18); no longer J101.4 (Pin_4)
- net A1: now also J101.17 (Pin_17); no longer J101.6 (Pin_6)
- net A2: no longer J101.8 (Pin_8)
- net A3: no longer J101.10 (Pin_10)
- net A4: no longer J101.12 (Pin_12)
- net A5: no longer J101.14 (Pin_14)
- net A6: now also J101.24 (Pin_24); no longer J101.16 (Pin_16)
- net A7: now also J101.23 (Pin_23); no longer J101.18 (Pin_18)
- net B0: now also J101.32 (Pin_32); no longer J101.24 (Pin_24)
- net B1: now also J101.31 (Pin_31); no longer J101.26 (Pin_26)
- net B2: now also J101.34 (Pin_34); no longer J101.28 (Pin_28)
- net B3: now also J101.33 (Pin_33); no longer J101.30 (Pin_30)
- net B4: now also J101.36 (Pin_36); no longer J101.32 (Pin_32)
- net B5: now also J101.35 (Pin_35); no longer J101.34 (Pin_34)
- net B6: now also J101.38 (Pin_38); no longer J101.36 (Pin_36)
- net B7: now also J101.37 (Pin_37); no longer J101.38 (Pin_38)
- net C0: now also J101.6 (Pin_6); no longer J101.23 (Pin_23)
- net C1: now also J101.7 (Pin_7); no longer J101.25 (Pin_25)
- net C2: now also J101.8 (Pin_8); no longer J101.27 (Pin_27)
- net C3: now also J101.9 (Pin_9); no longer J101.29 (Pin_29)
- net C4: now also J101.10 (Pin_10); no longer J101.31 (Pin_31)
- net C5: now also J101.11 (Pin_11); no longer J101.33 (Pin_33)
- net C6: now also J101.12 (Pin_12); no longer J101.35 (Pin_35)
- net C7: now also J101.13 (Pin_13); no longer J101.37 (Pin_37)
- net GND: now also J101.1 (Pin_1)
- net R_{A}0: now also J101.14 (Pin_14); no longer J101.1 (Pin_1)
- net R_{A}1: now also J101.15 (Pin_15); no longer J101.3 (Pin_3)
- net R_{A}2: now also J101.16 (Pin_16); no longer J101.5 (Pin_5)
- net R_{B}0: now also J101.26 (Pin_26); no longer J101.7 (Pin_7)
- net R_{B}1: now also J101.25 (Pin_25); no longer J101.9 (Pin_9)
- net R_{B}2: now also J101.28 (Pin_28); no longer J101.11 (Pin_11)
- net R_{C}0: now also J101.3 (Pin_3); no longer J101.13 (Pin_13)
- net R_{C}1: now also J101.4 (Pin_4); no longer J101.15 (Pin_15)
- net R_{C}2: now also J101.5 (Pin_5); no longer J101.17 (Pin_17)
- new net W: J101.29 (Pin_29)
- new net ~{Enable}: J101.30 (Pin_30)
- no-connect marks 0 -> 1
Other:
- sheet Register 0 ports: added C_{Write}; removed C_{write}
- sheet Register 1 ports: added C_{Write}; removed C_{write}
- sheet Register 2 ports: added C_{Write}; removed C_{write}
- sheet Register 3 ports: added C_{Write}; removed C_{write}
- sheet Register 4 ports: added C_{Write}; removed C_{write}
- sheet Register 5 ports: added C_{Write}; removed C_{write}
- sheet Register 6 ports: added C_{Write}; removed C_{write}
- sheet Register 7 ports: added C_{Write}; removed C_{write}
- sheet Selectors ports: added C_{W}, ~{Active}; removed none
- moved on the sheet: J101
