File: pcbs/Register File/register.kicad_sch (KiCad schematic)
At the start: 27 parts, among them U201 74HCT574, U203 74HC245

Commit message: Lots of rethinking
Parts:
- removed D108: Blue, LED_SMD:LED_0603_1608Metric, symbol Device:LED
- removed R809: 4k7, Resistor_SMD:R_0603_1608Metric, symbol Device:R
- removed U203: 74HC245, Package_SO:SOIC-20W_7.5x12.8mm_P1.27mm, symbol 74xx:74HC245

Commit message: Finish board
Connections:
- net C_{write} renamed C_{Write}
Changed lines of the file:
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@@
+    (stroke (width 0) (type default))
+  )
+  (wire (pts (xy 43.18 104.14) (xy 50.8 104.14))
+    (stroke (width 0) (type default))
+  )
+  (bus (pts (xy 228.6 92.71) (xy 228.6 95.25))
+    (stroke (width 0) (type default))
+  )
+  (bus (pts (xy 48.26 35.56) (xy 48.26 38.1))
+    (stroke (width 0) (type default))
+  )
+  (wire (pts (xy 195.58 71.12) (xy 195.58 72.39))
+    (stroke (width 0) (type default))
+  )
+  (wire (pts (xy 123.19 82.55) (xy 182.88 82.55))
+    (stroke (width 0) (type default))
+  )
+  (wire (pts (xy 71.12 114.3) (xy 76.2 114.3))
+    (stroke (width 0) (type default))
+  )
+  (wire (pts (xy 176.53 102.87) (xy 182.88 102.87))
+    (stroke (width 0) (type default))
+  )
+  (wire (pts (xy 208.28 87.63) (xy 226.06 87.63))
+    (stroke (width 0) (type default))
+  )
+  (wire (pts (xy 76.2 144.78) (xy 76.2 134.62))
+    (stroke (width 0) (type default))
+  )
+  (wire (pts (xy 43.18 134.62) (xy 50.8 134.62))
+    (stroke (width 0) (type default))
+  )
+  (bus (pts (xy 228.6 87.63) (xy 228.6 90.17))
+    (stroke (width 0) (type default))
+  )
+  (bus (pts (xy 48.26 43.18) (xy 48.26 45.72))
+    (stroke (width 0) (type default))
+  )
+  (wire (pts (xy 71.12 154.94) (xy 76.2 154.94))
+    (stroke (width 0) (type default))
+  )
+  (wire (pts (xy 90.17 50.8) (xy 138.43 50.8))
+    (stroke (width 0) (type default))
+  )
+  (wire (pts (xy 58.42 114.3) (xy 63.5 114.3))
+    (stroke (width 0) (type default))
+  )
+  (wire (pts (xy 71.12 134.62) (xy 76.2 134.62))
+    (stroke (width 0) (type default))
+  )
+  (bus (pts (xy 228.6 30.48) (xy 228.6 33.02))
+    (stroke (width 0) (type default))
+  )
+  (wire (pts (xy 71.12 104.14) (xy 76.2 104.14))
+    (stroke (width 0) (type default))
+  )
+  (wire (pts (xy 76.2 154.94) (xy 76.2 144.78))
+    (stroke (width 0) (type default))
+  )
+  (wire (pts (xy 176.53 55.88) (xy 182.88 55.88))
+    (stroke (width 0) (type default))
+  )
+  (bus (pts (xy 228.6 82.55) (xy 228.6 85.09))
+    (stroke (width 0) (type default))
+  )
+  (wire (pts (xy 200.66 115.57) (xy 195.58 115.57))
+    (stroke (width 0) (type default))
+  )
+  (wire (pts (xy 130.81 90.17) (xy 130.81 43.18))
+    (stroke (width 0) (type default))
+  )
+  (wire (pts (xy 76.2 104.14) (xy 76.2 93.98))
+    (stroke (width 0) (type default))
+  )
+  (wire (pts (xy 208.28 50.8) (xy 226.06 50.8))
+    (stroke (width 0) (type default))
+  )
+  (wire (pts (xy 58.42 144.78) (xy 63.5 144.78))
+    (stroke (width 0) (type default))
+  )
+  (wire (pts (xy 133.35 45.72) (xy 133.35 92.71))
+    (stroke (width 0) (type default))
+  )
+  (wire (pts (xy 64.77 58.42) (xy 60.96 58.42))
+    (stroke (width 0) (type default))
+  )
+  (wire (pts (xy 154.94 68.58) (xy 158.75 68.58))
+    (stroke (width 0) (type default))
+  )
+  (wire (pts (xy 43.18 165.1) (xy 50.8 165.1))
+    (stroke (width 0) (type default))
+  )
+  (bus (pts (xy 228.6 38.1) (xy 228.6 40.64))
+    (stroke (width 0) (type default))
+  )
+  (wire (pts (xy 76.2 114.3) (xy 76.2 104.14))
+    (stroke (width 0) (type default))
+  )
+  (wire (pts (xy 208.28 90.17) (xy 226.06 90.17))
+    (stroke (width 0) (type default))
+  )
+  (wire (pts (xy 176.53 68.58) (xy 182.88 68.58))
+    (stroke (width 0) (type default))
+  )
+  (wire (pts (xy 58.42 154.94) (xy 63.5 154.94))
+    (stroke (width 0) (type default))
+  )
+  (wire (pts (xy 180.34 116.84) (xy 182.88 116.84))
+    (stroke (width 0) (type default))
+  )
+  (wire (pts (xy 90.17 48.26) (xy 135.89 48.26))
+    (stroke (width 0) (type default))
+  )
+  (wire (pts (xy 123.19 35.56) (xy 182.88 35.56))
+    (stroke (width 0) (type default))
+  )
+  (bus (pts (xy 228.6 45.72) (xy 228.6 48.26))
+    (stroke (width 0) (type default))
+  )
+  (wire (pts (xy 182.88 80.01) (xy 120.65 80.01))
+    (stroke (width 0) (type default))
+  )
+  (bus (pts (xy 228.6 40.64) (xy 228.6 43.18))
+    (stroke (width 0) (type default))
+  )
+  (wire (pts (xy 58.42 165.1) (xy 63.5 165.1))
+    (stroke (width 0) (type default))
+  )
+  (wire (pts (xy 90.17 38.1) (xy 125.73 38.1))
+    (stroke (width 0) (type default))
+  )
+  (wire (pts (xy 43.18 93.98) (xy 50.8 93.98))
+    (stroke (width 0) (type default))
+  )
+  (wire (pts (xy 208.28 40.64) (xy 226.06 40.64))
+    (stroke (width 0) (type default))
+  )
+  (wire (pts (xy 208.28 97.79) (xy 226.06 97.79))
+    (stroke (width 0) (type default))
+  )
+  (wire (pts (xy 201.93 67.31) (xy 195.58 67.31))
+    (stroke (width 0) (type default))
+  )
+  (wire (pts (xy 195.58 67.31) (xy 195.58 66.04))
+    (stroke (width 0) (type default))
+  )
+  (wire (pts (xy 138.43 97.79) (xy 182.88 97.79))
+    (stroke (width 0) (type default))
+  )
+  (wire (pts (xy 190.5 71.12) (xy 195.58 71.12))
+    (stroke (width 0) (type default))
+  )
+  (bus (pts (xy 228.6 25.4) (xy 228.6 30.48))
     (stroke (width 0) (type default))
   )
   (wire (pts (xy 50.8 55.88) (xy 64.77 55.88))
-    (stroke (width 0) (type default))
-  )
-  (wire (pts (xy 43.18 104.14) (xy 50.8 104.14))
-    (stroke (width 0) (type default))
-  )
-  (bus (pts (xy 228.6 92.71) (xy 228.6 95.25))
-    (stroke (width 0) (type default))
-  )
-  (bus (pts (xy 48.26 35.56) (xy 48.26 38.1))
-    (stroke (width 0) (type default))
-  )
-  (wire (pts (xy 195.58 71.12) (xy 195.58 72.39))
-    (stroke (width 0) (type default))
-  )
-  (wire (pts (xy 123.19 82.55) (xy 182.88 82.55))
-    (stroke (width 0) (type default))
-  )
-  (wire (pts (xy 71.12 114.3) (xy 76.2 114.3))
-    (stroke (width 0) (type default))
-  )
-  (wire (pts (xy 176.53 102.87) (xy 182.88 102.87))
-    (stroke (width 0) (type default))
-  )
-  (wire (pts (xy 208.28 87.63) (xy 226.06 87.63))
-    (stroke (width 0) (type default))
-  )
-  (wire (pts (xy 76.2 144.78) (xy 76.2 134.62))
-    (stroke (width 0) (type default))
-  )
-  (wire (pts (xy 43.18 134.62) (xy 50.8 134.62))
-    (stroke (width 0) (type default))
-  )
-  (bus (pts (xy 228.6 87.63) (xy 228.6 90.17))
-    (stroke (width 0) (type default))
-  )
-  (bus (pts (xy 48.26 43.18) (xy 48.26 45.72))
-    (stroke (width 0) (type default))
-  )
-  (wire (pts (xy 71.12 154.94) (xy 76.2 154.94))
-    (stroke (width 0) (type default))
-  )
-  (wire (pts (xy 90.17 50.8) (xy 138.43 50.8))
-    (stroke (width 0) (type default))
-  )
-  (wire (pts (xy 58.42 114.3) (xy 63.5 114.3))
-    (stroke (width 0) (type default))
-  )
-  (wire (pts (xy 71.12 134.62) (xy 76.2 134.62))
-    (stroke (width 0) (type default))
-  )
-  (bus (pts (xy 228.6 30.48) (xy 228.6 33.02))
-    (stroke (width 0) (type default))
-  )
-  (wire (pts (xy 71.12 104.14) (xy 76.2 104.14))
-    (stroke (width 0) (type default))
-  )
-  (wire (pts (xy 76.2 154.94) (xy 76.2 144.78))
-    (stroke (width 0) (type default))
-  )
-  (wire (pts (xy 176.53 55.88) (xy 182.88 55.88))
-    (stroke (width 0) (type default))
-  )
-  (bus (pts (xy 228.6 82.55) (xy 228.6 85.09))
-    (stroke (width 0) (type default))
-  )
-  (wire (pts (xy 200.66 115.57) (xy 195.58 115.57))
-    (stroke (width 0) (type default))
-  )
-  (wire (pts (xy 130.81 90.17) (xy 130.81 43.18))
-    (stroke (width 0) (type default))
-  )
-  (wire (pts (xy 76.2 104.14) (xy 76.2 93.98))
-    (stroke (width 0) (type default))
-  )
-  (wire (pts (xy 208.28 50.8) (xy 226.06 50.8))
-    (stroke (width 0) (type default))
-  )
-  (wire (pts (xy 58.42 144.78) (xy 63.5 144.78))
-    (stroke (width 0) (type default))
-  )
-  (wire (pts (xy 133.35 45.72) (xy 133.35 92.71))
-    (stroke (width 0) (type default))
-  )
-  (wire (pts (xy 64.77 58.42) (xy 60.96 58.42))
-    (stroke (width 0) (type default))
-  )
-  (wire (pts (xy 154.94 68.58) (xy 158.75 68.58))
-    (stroke (width 0) (type default))
-  )
-  (wire (pts (xy 43.18 165.1) (xy 50.8 165.1))
-    (stroke (width 0) (type default))
-  )
-  (bus (pts (xy 228.6 38.1) (xy 228.6 40.64))
-    (stroke (width 0) (type default))
-  )
-  (wire (pts (xy 76.2 114.3) (xy 76.2 104.14))
-    (stroke (width 0) (type default))
-  )
-  (wire (pts (xy 208.28 90.17) (xy 226.06 90.17))
-    (stroke (width 0) (type default))
-  )
-  (wire (pts (xy 176.53 68.58) (xy 182.88 68.58))
-    (stroke (width 0) (type default))
-  )
-  (wire (pts (xy 58.42 154.94) (xy 63.5 154.94))
-    (stroke (width 0) (type default))
-  )
-  (wire (pts (xy 180.34 116.84) (xy 182.88 116.84))
-    (stroke (width 0) (type default))
-  )
-  (wire (pts (xy 90.17 48.26) (xy 135.89 48.26))
-    (stroke (width 0) (type default))
-  )
-  (wire (pts (xy 123.19 35.56) (xy 182.88 35.56))
-    (stroke (width 0) (type default))
-  )
-  (bus (pts (xy 228.6 45.72) (xy 228.6 48.26))
-    (stroke (width 0) (type default))
-  )
-  (wire (pts (xy 182.88 80.01) (xy 120.65 80.01))
-    (stroke (width 0) (type default))
-  )
-  (bus (pts (xy 228.6 40.64) (xy 228.6 43.18))
-    (stroke (width 0) (type default))
-  )
-  (wire (pts (xy 58.42 165.1) (xy 63.5 165.1))
-    (stroke (width 0) (type default))
-  )
-  (wire (pts (xy 90.17 38.1) (xy 125.73 38.1))
-    (stroke (width 0) (type default))
-  )
-  (wire (pts (xy 43.18 93.98) (xy 50.8 93.98))
-    (stroke (width 0) (type default))
-  )
-  (wire (pts (xy 208.28 40.64) (xy 226.06 40.64))
-    (stroke (width 0) (type default))
-  )
-  (wire (pts (xy 208.28 97.79) (xy 226.06 97.79))
-    (stroke (width 0) (type default))
-  )
-  (wire (pts (xy 201.93 67.31) (xy 195.58 67.31))
-    (stroke (width 0) (type default))
-  )
-  (wire (pts (xy 195.58 67.31) (xy 195.58 66.04))
-    (stroke (width 0) (type default))
-  )
-  (wire (pts (xy 138.43 97.79) (xy 182.88 97.79))
-    (stroke (width 0) (type default))
-  )
-  (wire (pts (xy 190.5 71.12) (xy 195.58 71.12))
-    (stroke (width 0) (type default))
-  )
-  (bus (pts (xy 228.6 25.4) (xy 228.6 30.48))
     (stroke (width 0) (type default))
   )
@@
     (effects (font (size 1.27 1.27)) (justify left))
   )
-  (hierarchical_label "C_{write}" (shape input) (at 50.8 55.88 180) (fields_autoplaced)
+  (hierarchical_label "C_{Write}" (shape input) (at 50.8 55.88 180) (fields_autoplaced)
     (effects (font (size 1.27 1.27)) (justify right))
   )
