File: pcbs/Register File/selectors.kicad_sch (KiCad schematic)
At the start: 33 parts, among them U1001 74HC138, U1002 74HC138, U1003 74HC138, U1004 74HC138, U1005 74HC540, U1006 74HC32, U1007 74HC14

Commit message: Lots of rethinking
Parts:
- removed R401 (x8): 220k, Resistor_SMD:R_0603_1608Metric, symbol Device:R
- removed U1003: 74HC138, Package_DIP:DIP-16_W7.62mm_Socket, symbol 74xx:74HC138
- removed U1005: 74HC540, Package_DIP:DIP-20_W7.62mm_Socket, symbol 74xx:74LS540
- removed U1006: 74HC32, Package_DIP:DIP-14_W7.62mm_Socket, symbol 74xx:74LS32
Connections:
- net GND: no longer U1004.8 (GND)
- net ~{Active}: no longer U1007.12
- net Ex: no longer names the net of U1007.11
- net ~{Execute}: no longer names the net of U1007.10
- no-connect marks 5 -> 4

Commit message: Working and routing
Parts:
- added U1001: 74HC14, Package_SO:SOIC-14_3.9x8.7mm_P1.27mm, symbol 74xx:74HC14
- U1002: renamed from U1007; LCSC (none) -> C5605
- renumbered U1004 to U1003, U1001 to U1004, U1002 to U1005
Connections:
- net +5V: now also U1001.14 (VCC)
- net GND: now also U1003.8 (GND), U1001.5, U1001.7 (GND), U1001.9; no longer U1002.1, U1002.3
- net W0: now also U1001.1
- net W1: now also U1001.13
- net W2: now also U1001.3
- net W3: now also U1001.11
- net W4: now also U1002.1
- net W5: now also U1002.13
- net W6: now also U1002.3
- net W7: now also U1002.11
- net C_{Write}7: now reaches U1002.10
- net C_{Write}6: now reaches U1002.4
- net C_{Write}4: now reaches U1002.2
- net C_{Write}5: now reaches U1002.12
- new net C_{Write}0: U1001.2
- new net C_{Write}1: U1001.12
- new net C_{Write}2: U1001.4
- new net C_{Write}3: U1001.10
Other:
- moved on the sheet: D801, R809, R810, R811, R812, R813, R814, R815, R816, U1002A, U1002B, U1002E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

Commit message: Finish board
Parts:
- added C302: 100n, Capacitor_SMD:C_0603_1608Metric, symbol Device:C
Connections:
- net +5V: now also C302.1; no longer D801.2 (A), D801.2 (A), D801.2 (A), D801.2 (A), D801.2 (A), D801.2 (A), D801.2 (A), D801.2 (A)
- net C_{Write}0: now also D801.2 (A), U1001.10; no longer U1001.2
- net C_{Write}1: now also D801.2 (A), U1001.4; no longer U1001.12
- net C_{Write}2: now also D801.2 (A), U1001.12; no longer U1001.4
- net C_{Write}3: now also D801.2 (A), U1001.2; no longer U1001.10
- net C_{Write}4: now also D801.2 (A), U1002.10; no longer U1002.2
- net C_{Write}5: now also D801.2 (A), U1002.4; no longer U1002.12
- net C_{Write}6: now also D801.2 (A), U1002.12; no longer U1002.4
- net C_{Write}7: now also D801.2 (A), U1002.2; no longer U1002.10
- net GND: now also R809.1, R810.1, R811.1, R812.1, R813.1, R814.1, R815.1, R816.1, C302.2
- net C_{W}/~{C_{R}} renamed C_{W}
- removed net W0: R809.1, U1001.1, U1003.15 (~{Y0})
- removed net W1: R810.1, U1001.13, U1003.14 (~{Y1})
- removed net W2: R811.1, U1001.3, U1003.13 (~{Y2})
- removed net W3: R812.1, U1001.11, U1003.12 (~{Y3})
- removed net W4: R813.1, U1002.1, U1003.11 (~{Y4})
- removed net W5: R814.1, U1002.13, U1003.10 (~{Y5})
- removed net W6: R815.1, U1002.3, U1003.9 (~{Y6})
- removed net W7: R816.1, U1002.11, U1003.7 (~{Y7})
- new net: U1002.3, U1003.10 (~{Y5})
- new net: U1002.11, U1003.11 (~{Y4})
- new net: U1001.1, U1003.12 (~{Y3})
- new net: U1001.13, U1003.13 (~{Y2})
- new net: U1001.3, U1003.14 (~{Y1})
- new net: U1001.11, U1003.15 (~{Y0})
- new net: U1002.1, U1003.7 (~{Y7})
- new net: U1002.13, U1003.9 (~{Y6})
Other:
- moved on the sheet: U1001A, U1001B, U1001E, U1001F, U1002A, U1002B, U1002E, U1002F
