File: pcbs/Simple Program Counter/incrementer.kicad_sch (KiCad schematic)
At the start: 2 parts, among them U404 74HC283, U405 74HC283

Commit message: Getting close
Connections:
- net PC_{next}0 renamed PC_{inc}0
- net PC_{next}1 renamed PC_{inc}1
- net PC_{next}2 renamed PC_{inc}2
- net PC_{next}3 renamed PC_{inc}3
- net PC_{next}4 renamed PC_{inc}4
- net PC_{next}5 renamed PC_{inc}5
- net PC_{next}6 renamed PC_{inc}6
- net PC_{next}7 renamed PC_{inc}7
Changed lines of the file:
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@@
     (effects (font (size 1.27 1.27)) (justify left top))
   )
-  (label "PC_{next}5" (at 97.79 95.25 0) (fields_autoplaced)
+  (label "PC_{inc}5" (at 97.79 95.25 0) (fields_autoplaced)
     (effects (font (size 1.27 1.27)) (justify left bottom))
   )
-  (label "PC_{next}4" (at 97.79 92.71 0) (fields_autoplaced)
+  (label "PC_{inc}4" (at 97.79 92.71 0) (fields_autoplaced)
     (effects (font (size 1.27 1.27)) (justify left bottom))
   )
@@
     (effects (font (size 1.27 1.27)) (justify left bottom))
   )
-  (label "PC_{next}0" (at 97.79 43.18 0) (fields_autoplaced)
+  (label "PC_{inc}0" (at 97.79 43.18 0) (fields_autoplaced)
     (effects (font (size 1.27 1.27)) (justify left bottom))
   )
@@
     (effects (font (size 1.27 1.27)) (justify left bottom))
   )
-  (label "PC_{next}7" (at 97.79 100.33 0) (fields_autoplaced)
+  (label "PC_{inc}7" (at 97.79 100.33 0) (fields_autoplaced)
     (effects (font (size 1.27 1.27)) (justify left bottom))
   )
@@
     (effects (font (size 1.27 1.27)) (justify left bottom))
   )
-  (label "PC_{next}2" (at 97.79 48.26 0) (fields_autoplaced)
+  (label "PC_{inc}2" (at 97.79 48.26 0) (fields_autoplaced)
     (effects (font (size 1.27 1.27)) (justify left bottom))
   )
-  (label "PC_{next}6" (at 97.79 97.79 0) (fields_autoplaced)
+  (label "PC_{inc}6" (at 97.79 97.79 0) (fields_autoplaced)
     (effects (font (size 1.27 1.27)) (justify left bottom))
   )
@@
     (effects (font (size 1.27 1.27)) (justify left bottom))
   )
-  (label "PC_{next}1" (at 97.79 45.72 0) (fields_autoplaced)
+  (label "PC_{inc}1" (at 97.79 45.72 0) (fields_autoplaced)
     (effects (font (size 1.27 1.27)) (justify left bottom))
   )
-  (label "PC_{next}3" (at 97.79 50.8 0) (fields_autoplaced)
+  (label "PC_{inc}3" (at 97.79 50.8 0) (fields_autoplaced)
     (effects (font (size 1.27 1.27)) (justify left bottom))
   )
-  (hierarchical_label "PC_{next}[0..7]" (shape output) (at 121.92 35.56 0) (fields_autoplaced)
+  (hierarchical_label "PC_{inc}[0..7]" (shape output) (at 121.92 35.56 0) (fields_autoplaced)
     (effects (font (size 1.27 1.27)) (justify left))
   )
