File: pcbs/Simple Program Counter/instructions.kicad_sch (KiCad schematic)
At the start: 22 parts, among them U202 74HC245, U401 74HC138

Commit message: Getting close
Other:
- added sheet PC Update (pcupdate.kicad_sch)
Changed lines of the file:
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@@
+    (stroke (width 0) (type default))
+  )
+  (wire (pts (xy 50.8 38.1) (xy 57.15 38.1))
     (stroke (width 0) (type default))
   )
@@
     (stroke (width 0) (type default))
   )
+  (wire (pts (xy 50.8 48.26) (xy 57.15 48.26))
+    (stroke (width 0) (type default))
+  )
   (wire (pts (xy 69.85 182.88) (xy 69.85 185.42))
     (stroke (width 0) (type default))
@@
     (stroke (width 0) (type default))
   )
+  (wire (pts (xy 50.8 43.18) (xy 57.15 43.18))
+    (stroke (width 0) (type default))
+  )
   (wire (pts (xy 143.51 129.54) (xy 154.94 129.54))
     (stroke (width 0) (type default))
@@
     (stroke (width 0) (type default))
   )
+  (bus (pts (xy 104.14 34.29) (xy 111.76 34.29))
+    (stroke (width 0) (type default))
+  )
   (wire (pts (xy 143.51 121.92) (xy 154.94 121.92))
     (stroke (width 0) (type default))
@@
     (stroke (width 0) (type default))
   )
+  (wire (pts (xy 50.8 33.02) (xy 57.15 33.02))
+    (stroke (width 0) (type default))
+  )
   (wire (pts (xy 167.64 102.87) (xy 167.64 106.68))
     (stroke (width 0) (type default))
@@
     (effects (font (size 1.27 1.27)) (justify left bottom))
   )
-  (label "PC_{curr}2" (at 143.51 119.38 0)
+  (label "PC_{curr}2" (at 143.51 119.38 0) (fields_autoplaced)
     (effects (font (size 1.27 1.27)) (justify left bottom))
   )
@@
     (effects (font (size 1.27 1.27)) (justify left bottom))
   )
-  (label "PC_{curr}7" (at 143.51 132.08 0)
-    (effects (font (size 1.27 1.27)) (justify left bottom))
-  )
-  (label "PC_{curr}4" (at 143.51 124.46 0)
-    (effects (font (size 1.27 1.27)) (justify left bottom))
-  )
-  (label "C1" (at 180.34 116.84 0)
-    (effects (font (size 1.27 1.27)) (justify left bottom))
-  )
-  (label "C6" (at 180.34 129.54 0)
-    (effects (font (size 1.27 1.27)) (justify left bottom))
-  )
-  (label "~{Decoded}3" (at 240.03 110.49 0)
-    (effects (font (size 1.27 1.27)) (justify left bottom))
-  )
-  (label "C2" (at 180.34 119.38 0)
-    (effects (font (size 1.27 1.27)) (justify left bottom))
-  )
-  (label "~{Decoded}4" (at 240.03 120.65 0)
+  (label "PC_{curr}7" (at 143.51 132.08 0) (fields_autoplaced)
+    (effects (font (size 1.27 1.27)) (justify left bottom))
+  )
+  (label "PC_{curr}4" (at 143.51 124.46 0) (fields_autoplaced)
+    (effects (font (size 1.27 1.27)) (justify left bottom))
+  )
+  (label "C1" (at 180.34 116.84 0) (fields_autoplaced)
+    (effects (font (size 1.27 1.27)) (justify left bottom))
+  )
+  (label "~{BranchZ}" (at 50.8 48.26 180) (fields_autoplaced)
+    (effects (font (size 1.27 1.27)) (justify right bottom))
+  )
+  (label "C6" (at 180.34 129.54 0) (fields_autoplaced)
+    (effects (font (size 1.27 1.27)) (justify left bottom))
+  )
+  (label "~{Decoded}3" (at 240.03 110.49 0) (fields_autoplaced)
+    (effects (font (size 1.27 1.27)) (justify left bottom))
+  )
+  (label "C2" (at 180.34 119.38 0) (fields_autoplaced)
+    (effects (font (size 1.27 1.27)) (justify left bottom))
+  )
+  (label "~{Decoded}4" (at 240.03 120.65 0) (fields_autoplaced)
     (effects (font (size 1.27 1.27)) (justify left bottom))
   )
@@
     (effects (font (size 1.27 1.27)) (justify left bottom))
   )
-  (label "C7" (at 180.34 132.08 0)
-    (effects (font (size 1.27 1.27)) (justify left bottom))
-  )
-  (label "C4" (at 180.34 124.46 0)
+  (label "C7" (at 180.34 132.08 0) (fields_autoplaced)
+    (effects (font (size 1.27 1.27)) (justify left bottom))
+  )
+  (label "C4" (at 180.34 124.46 0) (fields_autoplaced)
     (effects (font (size 1.27 1.27)) (justify left bottom))
   )
@@
     (effects (font (size 1.27 1.27)) (justify left bottom))
   )
-  (label "~{Decoded}5" (at 240.03 130.81 0)
-    (effects (font (size 1.27 1.27)) (justify left bottom))
-  )
-  (label "~{Decoded}0" (at 240.03 80.01 0)
-    (effects (font (size 1.27 1.27)) (justify left bottom))
-  )
-  (label "~{Decoded}6" (at 240.03 140.97 0)
+  (label "~{Decoded}5" (at 240.03 130.81 0) (fields_autoplaced)
+    (effects (font (size 1.27 1.27)) (justify left bottom))
+  )
+  (label "~{Decoded}0" (at 240.03 80.01 0) (fields_autoplaced)
+    (effects (font (size 1.27 1.27)) (justify left bottom))
+  )
+  (label "~{Decoded}6" (at 240.03 140.97 0) (fields_autoplaced)
     (effects (font (size 1.27 1.27)) (justify left bottom))
   )
@@
     (effects (font (size 1.27 1.27)) (justify left bottom))
   )
-  (label "C0" (at 180.34 114.3 0)
-    (effects (font (size 1.27 1.27)) (justify left bottom))
-  )
-  (label "PC_{curr}6" (at 143.51 129.54 0)
-    (effects (font (size 1.27 1.27)) (justify left bottom))
-  )
-  (label "C5" (at 180.34 127 0)
+  (label "C0" (at 180.34 114.3 0) (fields_autoplaced)
+    (effects (font (size 1.27 1.27)) (justify left bottom))
+  )
+  (label "PC_{curr}6" (at 143.51 129.54 0) (fields_autoplaced)
+    (effects (font (size 1.27 1.27)) (justify left bottom))
+  )
+  (label "C5" (at 180.34 127 0) (fields_autoplaced)
     (effects (font (size 1.27 1.27)) (justify left bottom))
   )
@@
     (effects (font (size 1.27 1.27)) (justify left bottom))
   )
-  (label "PC_{curr}5" (at 143.51 127 0)
-    (effects (font (size 1.27 1.27)) (justify left bottom))
-  )
-  (label "~{Decoded}1" (at 240.03 90.17 0)
+  (label "PC_{curr}5" (at 143.51 127 0) (fields_autoplaced)
+    (effects (font (size 1.27 1.27)) (justify left bottom))
+  )
+  (label "~{Decoded}1" (at 240.03 90.17 0) (fields_autoplaced)
     (effects (font (size 1.27 1.27)) (justify left bottom))
   )
@@
     (effects (font (size 1.27 1.27)) (justify left bottom))
   )
-  (label "PC_{curr}1" (at 143.51 116.84 0)
-    (effects (font (size 1.27 1.27)) (justify left bottom))
-  )
-  (label "PC_{curr}0" (at 143.51 114.3 0)
+  (label "PC_{curr}1" (at 143.51 116.84 0) (fields_autoplaced)
+    (effects (font (size 1.27 1.27)) (justify left bottom))
+  )
+  (label "PC_{curr}0" (at 143.51 114.3 0) (fields_autoplaced)
     (effects (font (size 1.27 1.27)) (justify left bottom))
   )
@@
     (effects (font (size 1.27 1.27)) (justify left bottom))
   )
-  (label "~{Decoded}7" (at 240.03 151.13 0)
-    (effects (font (size 1.27 1.27)) (justify left bottom))
-  )
-  (label "~{Decoded}2" (at 240.03 100.33 0)
-    (effects (font (size 1.27 1.27)) (justify left bottom))
-  )
-  (label "PC_{curr}3" (at 143.51 121.92 0)
-    (effects (font (size 1.27 1.27)) (justify left bottom))
-  )
-  (label "C3" (at 180.34 121.92 0)
+  (label "~{Decoded}7" (at 240.03 151.13 0) (fields_autoplaced)
+    (effects (font (size 1.27 1.27)) (justify left bottom))
+  )
+  (label "~{Decoded}2" (at 240.03 100.33 0) (fields_autoplaced)
+    (effects (font (size 1.27 1.27)) (justify left bottom))
+  )
+  (label "PC_{curr}3" (at 143.51 121.92 0) (fields_autoplaced)
+    (effects (font (size 1.27 1.27)) (justify left bottom))
+  )
+  (label "C3" (at 180.34 121.92 0) (fields_autoplaced)
     (effects (font (size 1.27 1.27)) (justify left bottom))
   )
@@
     (effects (font (size 1.27 1.27)) (justify left))
   )
-  (hierarchical_label "A[0..7]" (shape input) (at 30.48 38.1 180) (fields_autoplaced)
+  (hierarchical_label "A[0..7]" (shape input) (at 50.8 38.1 180) (fields_autoplaced)
     (effects (font (size 1.27 1.27)) (justify right))
   )
-  (hierarchical_label "PC_{next}[0..7]" (shape input) (at 30.48 31.75 180) (fields_autoplaced)
+  (hierarchical_label "PC_{inc}[0..7]" (shape input) (at 50.8 33.02 180) (fields_autoplaced)
     (effects (font (size 1.27 1.27)) (justify right))
   )
@@
     (effects (font (size 1.27 1.27)) (justify right))
   )
-  (hierarchical_label "B[0..7]" (shape input) (at 30.48 44.45 180) (fields_autoplaced)
+  (hierarchical_label "PC_{next}[0..7]" (shape tri_state) (at 111.76 34.29 0) (fields_autoplaced)
+    (effects (font (size 1.27 1.27)) (justify left))
+  )
+  (hierarchical_label "B[0..7]" (shape input) (at 50.8 43.18 180) (fields_autoplaced)
     (effects (font (size 1.27 1.27)) (justify right))
   )
@@
       )
     )
+  )
+  (sheet (at 57.15 25.4) (size 46.99 36.83) (fields_autoplaced)
+    (stroke (width 0.1524) (type solid))
+    (fill (color 0 0 0 0.0000))
+    (property "Sheetname" "PC Update" (at 57.15 24.6884 0)
+      (effects (font (size 1.27 1.27)) (justify left bottom))
+    )
+    (property "Sheetfile" "pcupdate.kicad_sch" (at 57.15 62.8146 0)
+      (effects (font (size 1.27 1.27)) (justify left top))
+    )
+    (pin "PC_{inc}[0..7]" input (at 57.15 33.02 180)
+      (effects (font (size 1.27 1.27)) (justify left))
+    )
+    (pin "PC_{next}[0..7]" tri_state (at 104.14 34.29 0)
+      (effects (font (size 1.27 1.27)) (justify right))
+    )
+    (pin "A[0..7]" input (at 57.15 38.1 180)
+      (effects (font (size 1.27 1.27)) (justify left))
+    )
+    (pin "B[0..7]" input (at 57.15 43.18 180)
+      (effects (font (size 1.27 1.27)) (justify left))
+    )
+    (pin "~{BRANCHZERO}" input (at 57.15 48.26 180)
+      (effects (font (size 1.27 1.27)) (justify left))
+    )
+    (instances
+      (project "Simple Program Counter"
+        (path "/4f63efd2-c13f-4abc-af18-011a9cace63e/f2f3ce6f-4aba-4b71-8d92-5a32ab3e29dc" (page "5"))
+      )
+    )
